File: KiCad/GPS Hardware/MCU.sch (KiCad schematic (older format))
At the start: 0 parts

Commit message: Update
Parts:
- added C? (x3): C, symbol Device:C
- added J?: Conn_2Rows-07Pins, symbol Connector_Generic:Conn_2Rows-07Pins
- added R? (x4): R, symbol Device:R
- added R? (x2): 0, symbol Device:R
- added U?: ATmega328-AU, Package_QFP:TQFP-32_7x7mm_P0.8mm, symbol MCU_Microchip_ATmega:ATmega328-AU
- added U?: SN74AVC4T774PW, SOP65P640X120-16N, symbol GPS~Hardware:SN74AVC4T774PW
- added Y?: Crystal_GND24, symbol Device:Crystal_GND24
Connections:
- net labels added: +1V8, +3V3, AVR_VCC, CTS, CTS_Cellular, GND, INT_Power, MISO, MOSI, RESET, RTS, RTS_Cellular, RX, RX_Cellular, SCK, SCL_Power, SDA_Power, TX, TX_Cellular
- wire segments 0 -> 17
Other:
- note added: "Disconnect 0 ohm resistor depending on the input supply."
