File: KiCad/GPS Hardware/MCU.sch (KiCad schematic (older format))
At the start: 13 parts

Commit message: Finished adding components, need to add values
Parts:
- removed R? (x2): 0, symbol Device:R
- added C? (x5): C, symbol Device:C
Connections:
- net labels added: PWR_Cellular, RESET_Cellular
- net labels removed: AVR_VCC
- wire segments 17 -> 26
Other:
- note removed: "Disconnect 0 ohm resistor depending on the input supply."
- moved on the sheet: C?, J?, R?

Commit message: Update, 21st August
Parts:
- C? (x6): value C -> 0u1; footprint (none) -> Capacitor_SMD:C_0603_1608Metric_Pad1.08x0.95mm_HandSolder
- C? (x2): value C -> 22p; footprint (none) -> Capacitor_SMD:C_0603_1608Metric_Pad1.08x0.95mm_HandSolder
- J?: footprint (none) -> Connector_PinHeader_1.00mm:PinHeader_2x03_P1.00mm_Vertical_SMD
- R?: value R -> 10k; footprint (none) -> Resistor_SMD:R_0603_1608Metric_Pad0.98x0.95mm_HandSolder
- R? (x3): value R -> 2k2; footprint (none) -> Resistor_SMD:R_0603_1608Metric_Pad0.98x0.95mm_HandSolder
- Y?: footprint (none) -> Crystal:Crystal_SMD_HC49-SD_HandSoldering
Connections:
- no-connect marks 0 -> 10
Changed lines of the file:
@@
 P 1950 2200
 F 0 "C?" H 2065 2246 50  0000 L CNN
-F 1 "C" H 2065 2155 50  0000 L CNN
-F 2 "" H 1988 2050 50  0001 C CNN
+F 1 "0u1" H 2065 2155 50  0000 L CNN
+F 2 "Capacitor_SMD:C_0603_1608Metric_Pad1.08x0.95mm_HandSolder" H 1988 2050 50  0001 C CNN
 F 3 "~" H 1950 2200 50  0001 C CNN
 	1    1950 2200
@@
 P 4400 2350
 F 0 "C?" H 4515 2396 50  0000 L CNN
-F 1 "C" H 4515 2305 50  0000 L CNN
-F 2 "" H 4438 2200 50  0001 C CNN
-F 3 "~" H 4400 2350 50  0001 C CNN
+F 1 "22p" H 4515 2305 50  0000 L CNN
+F 2 "Capacitor_SMD:C_0603_1608Metric_Pad1.08x0.95mm_HandSolder" H 4438 2200 50  0001 C CNN
+F 3 "https://www.mouser.co.uk/ProductDetail/KEMET/C0603C220J1HACTU?qs=W0yvOO0ixfF6hDt%252BXfnhnA%3D%3D" H 4400 2350 50  0001 C CNN
 	1    4400 2350
 	1    0    0    -1
@@
 P 4400 2950
 F 0 "C?" H 4515 2996 50  0000 L CNN
-F 1 "C" H 4515 2905 50  0000 L CNN
-F 2 "" H 4438 2800 50  0001 C CNN
-F 3 "~" H 4400 2950 50  0001 C CNN
+F 1 "22p" H 4515 2905 50  0000 L CNN
+F 2 "Capacitor_SMD:C_0603_1608Metric_Pad1.08x0.95mm_HandSolder" H 4438 2800 50  0001 C CNN
+F 3 "https://www.mouser.co.uk/ProductDetail/KEMET/C0603C220J1HACTU?qs=W0yvOO0ixfF6hDt%252BXfnhnA%3D%3D" H 4400 2950 50  0001 C CNN
 	1    4400 2950
 	1    0    0    -1
@@
 F 0 "Y?" V 4354 2894 50  0000 L CNN
 F 1 "Crystal_GND24" V 4445 2894 50  0000 L CNN
-F 2 "" H 4400 2650 50  0001 C CNN
-F 3 "~" H 4400 2650 50  0001 C CNN
+F 2 "Crystal:Crystal_SMD_HC49-SD_HandSoldering" H 4400 2650 50  0001 C CNN
+F 3 "https://www.mouser.co.uk/ProductDetail/IQD/LFXTAL030234Reel?qs=e4%2FAndAAwgKRGsJIO2WnVQ%3D%3D" H 4400 2650 50  0001 C CNN
 	1    4400 2650
 	0    1    1    0
@@
 P 4000 3750
 F 0 "R?" H 4070 3796 50  0000 L CNN
-F 1 "R" H 4070 3705 50  0000 L CNN
-F 2 "" V 3930 3750 50  0001 C CNN
+F 1 "10k" V 4000 3700 50  0000 L CNN
+F 2 "Resistor_SMD:R_0603_1608Metric_Pad0.98x0.95mm_HandSolder" V 3930 3750 50  0001 C CNN
 F 3 "~" H 4000 3750 50  0001 C CNN
 	1    4000 3750
@@
 F 0 "J?" H 4400 1517 50  0000 C CNN
 F 1 "Conn_2Rows-07Pins" H 4400 1426 50  0000 C CNN
-F 2 "" H 4350 1200 50  0001 C CNN
+F 2 "Connector_PinHeader_1.00mm:PinHeader_2x03_P1.00mm_Vertical_SMD" H 4350 1200 50  0001 C CNN
 F 3 "~" H 4350 1200 50  0001 C CNN
 	1    4350 1200
@@
 U 1 1 614D403D
 P 3700 2300
-F 0 "R?" V 3493 2300 50  0000 C CNN
-F 1 "R" V 3584 2300 50  0000 C CNN
-F 2 "" V 3630 2300 50  0001 C CNN
+F 0 "R?" V 3650 2150 50  0000 C CNN
+F 1 "2k2" V 3700 2300 50  0000 C CNN
+F 2 "Resistor_SMD:R_0603_1608Metric_Pad0.98x0.95mm_HandSolder" V 3630 2300 50  0001 C CNN
 F 3 "~" H 3700 2300 50  0001 C CNN
 	1    3700 2300
@@
 U 1 1 614D4D77
 P 3700 2400
-F 0 "R?" V 3493 2400 50  0000 C CNN
-F 1 "R" V 3584 2400 50  0000 C CNN
-F 2 "" V 3630 2400 50  0001 C CNN
+F 0 "R?" V 3650 2250 50  0000 C CNN
+F 1 "2k2" V 3700 2400 50  0000 C CNN
+F 2 "Resistor_SMD:R_0603_1608Metric_Pad0.98x0.95mm_HandSolder" V 3630 2400 50  0001 C CNN
 F 3 "~" H 3700 2400 50  0001 C CNN
 	1    3700 2400
@@
 U 1 1 614D58E3
 P 3700 2500
-F 0 "R?" V 3493 2500 50  0000 C CNN
-F 1 "R" V 3584 2500 50  0000 C CNN
-F 2 "" V 3630 2500 50  0001 C CNN
+F 0 "R?" V 3650 2350 50  0000 C CNN
+F 1 "2k2" V 3700 2500 50  0000 C CNN
+F 2 "Resistor_SMD:R_0603_1608Metric_Pad0.98x0.95mm_HandSolder" V 3630 2500 50  0001 C CNN
 F 3 "~" H 3700 2500 50  0001 C CNN
 	1    3700 2500
@@
 P 2550 1050
 F 0 "C?" H 2665 1096 50  0000 L CNN
-F 1 "C" H 2665 1005 50  0000 L CNN
-F 2 "" H 2588 900 50  0001 C CNN
+F 1 "0u1" H 2665 1005 50  0000 L CNN
+F 2 "Capacitor_SMD:C_0603_1608Metric_Pad1.08x0.95mm_HandSolder" H 2588 900 50  0001 C CNN
 F 3 "~" H 2550 1050 50  0001 C CNN
 	1    2550 1050
@@
 P 2900 1050
 F 0 "C?" H 3015 1096 50  0000 L CNN
-F 1 "C" H 3015 1005 50  0000 L CNN
-F 2 "" H 2938 900 50  0001 C CNN
+F 1 "0u1" H 3015 1005 50  0000 L CNN
+F 2 "Capacitor_SMD:C_0603_1608Metric_Pad1.08x0.95mm_HandSolder" H 2938 900 50  0001 C CNN
 F 3 "~" H 2900 1050 50  0001 C CNN
 	1    2900 1050
@@
 P 3250 1050
 F 0 "C?" H 3365 1096 50  0000 L CNN
-F 1 "C" H 3365 1005 50  0000 L CNN
-F 2 "" H 3288 900 50  0001 C CNN
+F 1 "0u1" H 3365 1005 50  0000 L CNN
+F 2 "Capacitor_SMD:C_0603_1608Metric_Pad1.08x0.95mm_HandSolder" H 3288 900 50  0001 C CNN
 F 3 "~" H 3250 1050 50  0001 C CNN
 	1    3250 1050
@@
 P 7600 2100
 F 0 "C?" H 7715 2146 50  0000 L CNN
-F 1 "C" H 7715 2055 50  0000 L CNN
-F 2 "" H 7638 1950 50  0001 C CNN
+F 1 "0u1" H 7715 2055 50  0000 L CNN
+F 2 "Capacitor_SMD:C_0603_1608Metric_Pad1.08x0.95mm_HandSolder" H 7638 1950 50  0001 C CNN
 F 3 "~" H 7600 2100 50  0001 C CNN
 	1    7600 2100
@@
 P 7050 2200
 F 0 "C?" H 7165 2246 50  0000 L CNN
-F 1 "C" H 7165 2155 50  0000 L CNN
-F 2 "" H 7088 2050 50  0001 C CNN
+F 1 "0u1" H 7165 2155 50  0000 L CNN
+F 2 "Capacitor_SMD:C_0603_1608Metric_Pad1.08x0.95mm_HandSolder" H 7088 2050 50  0001 C CNN
 F 3 "~" H 7050 2200 50  0001 C CNN
 	1    7050 2200
@@
 Text GLabel 3450 3200 2    50   Input ~ 0
 RESET_Cellular
+NoConn ~ 2250 2200
+NoConn ~ 2250 2300
+NoConn ~ 3450 2000
+NoConn ~ 3450 2100
+NoConn ~ 3450 2200
+NoConn ~ 3450 2900
+NoConn ~ 3450 3000
+NoConn ~ 3450 4100
+NoConn ~ 3450 4300
+NoConn ~ 3450 4400
 $EndSCHEMATC

Commit message: Added footprints to most components
Parts:
- gave numbers to parts that had none: 16
Changed lines of the file:
@@
 $EndDescr
 $Comp
-L MCU_Microchip_ATmega:ATmega328-AU U?
+L MCU_Microchip_ATmega:ATmega328-AU U5
 U 1 1 61474832
 P 2850 3200
-F 0 "U?" H 2850 1611 50  0000 C CNN
+F 0 "U5" H 2850 1611 50  0000 C CNN
 F 1 "ATmega328-AU" H 2850 1520 50  0000 C CNN
 F 2 "Package_QFP:TQFP-32_7x7mm_P0.8mm" H 2850 3200 50  0001 C CIN
@@
 $EndComp
 $Comp
-L Device:C C?
+L Device:C C10
 U 1 1 6147650D
 P 1950 2200
-F 0 "C?" H 2065 2246 50  0000 L CNN
+F 0 "C10" H 2065 2246 50  0000 L CNN
 F 1 "0u1" H 2065 2155 50  0000 L CNN
 F 2 "Capacitor_SMD:C_0603_1608Metric_Pad1.08x0.95mm_HandSolder" H 1988 2050 50  0001 C CNN
@@
 	3450 2700 3950 2700
 $Comp
-L Device:C C?
+L Device:C C14
 U 1 1 6147B129
 P 4400 2350
-F 0 "C?" H 4515 2396 50  0000 L CNN
+F 0 "C14" H 4515 2396 50  0000 L CNN
 F 1 "22p" H 4515 2305 50  0000 L CNN
 F 2 "Capacitor_SMD:C_0603_1608Metric_Pad1.08x0.95mm_HandSolder" H 4438 2200 50  0001 C CNN
@@
 Connection ~ 4400 2500
 $Comp
-L Device:C C?
+L Device:C C15
 U 1 1 6147BAE8
 P 4400 2950
-F 0 "C?" H 4515 2996 50  0000 L CNN
+F 0 "C15" H 4515 2996 50  0000 L CNN
 F 1 "22p" H 4515 2905 50  0000 L CNN
 F 2 "Capacitor_SMD:C_0603_1608Metric_Pad1.08x0.95mm_HandSolder" H 4438 2800 50  0001 C CNN
@@
 $EndComp
 $Comp
-L Device:Crystal_GND24 Y?
+L Device:Crystal_GND24 Y1
 U 1 1 614775D6
 P 4400 2650
-F 0 "Y?" V 4354 2894 50  0000 L CNN
+F 0 "Y1" V 4354 2894 50  0000 L CNN
 F 1 "Crystal_GND24" V 4445 2894 50  0000 L CNN
 F 2 "Crystal:Crystal_SMD_HC49-SD_HandSoldering" H 4400 2650 50  0001 C CNN
@@
 SCK
 $Comp
-L Device:R R?
+L Device:R R15
 U 1 1 614B0F0F
 P 4000 3750
-F 0 "R?" H 4070 3796 50  0000 L CNN
+F 0 "R15" H 4070 3796 50  0000 L CNN
 F 1 "10k" V 4000 3700 50  0000 L CNN
 F 2 "Resistor_SMD:R_0603_1608Metric_Pad0.98x0.95mm_HandSolder" V 3930 3750 50  0001 C CNN
@@
 $EndComp
 $Comp
-L Connector_Generic:Conn_2Rows-07Pins J?
+L Connector_Generic:Conn_2Rows-07Pins J2
 U 1 1 614C8DA4
 P 4350 1200
-F 0 "J?" H 4400 1517 50  0000 C CNN
+F 0 "J2" H 4400 1517 50  0000 C CNN
 F 1 "Conn_2Rows-07Pins" H 4400 1426 50  0000 C CNN
 F 2 "Connector_PinHeader_1.00mm:PinHeader_2x03_P1.00mm_Vertical_SMD" H 4350 1200 50  0001 C CNN
@@
 $EndComp
 $Comp
-L Device:R R?
+L Device:R R12
 U 1 1 614D403D
 P 3700 2300
-F 0 "R?" V 3650 2150 50  0000 C CNN
+F 0 "R12" V 3650 2150 50  0000 C CNN
 F 1 "2k2" V 3700 2300 50  0000 C CNN
 F 2 "Resistor_SMD:R_0603_1608Metric_Pad0.98x0.95mm_HandSolder" V 3630 2300 50  0001 C CNN
@@
 $EndComp
 $Comp
-L Device:R R?
+L Device:R R13
 U 1 1 614D4D77
 P 3700 2400
-F 0 "R?" V 3650 2250 50  0000 C CNN
+F 0 "R13" V 3650 2250 50  0000 C CNN
 F 1 "2k2" V 3700 2400 50  0000 C CNN
 F 2 "Resistor_SMD:R_0603_1608Metric_Pad0.98x0.95mm_HandSolder" V 3630 2400 50  0001 C CNN
@@
 $EndComp
 $Comp
-L Device:R R?
+L Device:R R14
 U 1 1 614D58E3
 P 3700 2500
-F 0 "R?" V 3650 2350 50  0000 C CNN
+F 0 "R14" V 3650 2350 50  0000 C CNN
 F 1 "2k2" V 3700 2500 50  0000 C CNN
 F 2 "Resistor_SMD:R_0603_1608Metric_Pad0.98x0.95mm_HandSolder" V 3630 2500 50  0001 C CNN
@@
 Connection ~ 2850 1700
 $Comp
-L Device:C C?
+L Device:C C11
 U 1 1 6121D0CD
 P 2550 1050
-F 0 "C?" H 2665 1096 50  0000 L CNN
+F 0 "C11" H 2665 1096 50  0000 L CNN
 F 1 "0u1" H 2665 1005 50  0000 L CNN
 F 2 "Capacitor_SMD:C_0603_1608Metric_Pad1.08x0.95mm_HandSolder" H 2588 900 50  0001 C CNN
@@
 $EndComp
 $Comp
-L Device:C C?
+L Device:C C12
 U 1 1 6121E29B
 P 2900 1050
-F 0 "C?" H 3015 1096 50  0000 L CNN
+F 0 "C12" H 3015 1096 50  0000 L CNN
 F 1 "0u1" H 3015 1005 50  0000 L CNN
 F 2 "Capacitor_SMD:C_0603_1608Metric_Pad1.08x0.95mm_HandSolder" H 2938 900 50  0001 C CNN
@@
 $EndComp
 $Comp
-L Device:C C?
+L Device:C C13
 U 1 1 6121E902
 P 3250 1050
-F 0 "C?" H 3365 1096 50  0000 L CNN
+F 0 "C13" H 3365 1096 50  0000 L CNN
 F 1 "0u1" H 3365 1005 50  0000 L CNN
 F 2 "Capacitor_SMD:C_0603_1608Metric_Pad1.08x0.95mm_HandSolder" H 3288 900 50  0001 C CNN
@@
 RX
 $Comp
-L GPS~Hardware:SN74AVC4T774PW U?
+L GPS~Hardware:SN74AVC4T774PW U6
 U 1 1 61491FC4
 P 6250 2750
-F 0 "U?" H 6250 3820 50  0000 C CNN
+F 0 "U6" H 6250 3820 50  0000 C CNN
 F 1 "SN74AVC4T774PW" H 6250 3729 50  0000 C CNN
 F 2 "SOP65P640X120-16N" H 6250 2750 50  0001 L BNN
@@
 $EndComp
 $Comp
-L Device:C C?
+L Device:C C17
 U 1 1 612AD4B1
 P 7600 2100
-F 0 "C?" H 7715 2146 50  0000 L CNN
+F 0 "C17" H 7715 2146 50  0000 L CNN
 F 1 "0u1" H 7715 2055 50  0000 L CNN
 F 2 "Capacitor_SMD:C_0603_1608Metric_Pad1.08x0.95mm_HandSolder" H 7638 1950 50  0001 C CNN
@@
 $EndComp
 $Comp
-L Device:C C?
+L Device:C C16
 U 1 1 612AE26D
 P 7050 2200
-F 0 "C?" H 7165 2246 50  0000 L CNN
+F 0 "C16" H 7165 2246 50  0000 L CNN
 F 1 "0u1" H 7165 2155 50  0000 L CNN
 F 2 "Capacitor_SMD:C_0603_1608Metric_Pad1.08x0.95mm_HandSolder" H 7088 2050 50  0001 C CNN
@@
 	7050 2050 6950 2050
 $Comp
-L power:GND #PWR?
+L power:GND #PWR0110
 U 1 1 612DF9B5
 P 7050 2350
-F 0 "#PWR?" H 7050 2100 50  0001 C CNN
+F 0 "#PWR0110" H 7050 2100 50  0001 C CNN
 F 1 "GND" H 7055 2177 50  0000 C CNN
 F 2 "" H 7050 2350 50  0001 C CNN
@@
 $EndComp
 $Comp
-L power:GND #PWR?
+L power:GND #PWR0149
 U 1 1 612E15CE
 P 7600 2250
-F 0 "#PWR?" H 7600 2000 50  0001 C CNN
+F 0 "#PWR0149" H 7600 2000 50  0001 C CNN
 F 1 "GND" H 7605 2077 50  0000 C CNN
 F 2 "" H 7600 2250 50  0001 C CNN

Commit message: Added all footprints
Hopefully they are correct :)
Parts:
- U6: footprint SOP65P640X120-16N -> GPS Hardware:SOP65P640X120-16N
Changed lines of the file:
@@
 F 0 "U6" H 6250 3820 50  0000 C CNN
 F 1 "SN74AVC4T774PW" H 6250 3729 50  0000 C CNN
-F 2 "SOP65P640X120-16N" H 6250 2750 50  0001 L BNN
+F 2 "GPS Hardware:SOP65P640X120-16N" H 6250 2750 50  0001 L BNN
 F 3 "" H 6250 2750 50  0001 L BNN
 	1    6250 2750

Commit message: Update
Parts:
- removed J2: Conn_2Rows-07Pins, Connector_PinHeader_1.00mm:PinHeader_2x03_P1.00mm_Vertical_SMD, symbol Connector_Generic:Conn_2Rows-07Pins
- removed Y1: Crystal_GND24, Crystal:Crystal_SMD_HC49-SD_HandSoldering, symbol Device:Crystal_GND24
- added J2: Conn_01x06_Male, Connector_PinHeader_1.00mm:PinHeader_2x03_P1.00mm_Vertical_SMD, symbol Connector:Conn_01x06_Male
- added Y1: Crystal, Crystal:Crystal_SMD_HC49-SD, symbol Device:Crystal
Changed lines of the file:
@@
 Connection ~ 4400 2800
-$Comp
-L power:GND #PWR0128
-U 1 1 6147C141
-P 4200 2650
-F 0 "#PWR0128" H 4200 2400 50  0001 C CNN
-F 1 "GND" V 4205 2522 50  0000 R CNN
-F 2 "" H 4200 2650 50  0001 C CNN
-F 3 "" H 4200 2650 50  0001 C CNN
-	1    4200 2650
-	0    1    1    0
-$EndComp
-$Comp
-L Device:Crystal_GND24 Y1
-U 1 1 614775D6
-P 4400 2650
-F 0 "Y1" V 4354 2894 50  0000 L CNN
-F 1 "Crystal_GND24" V 4445 2894 50  0000 L CNN
-F 2 "Crystal:Crystal_SMD_HC49-SD_HandSoldering" H 4400 2650 50  0001 C CNN
-F 3 "https://www.mouser.co.uk/ProductDetail/IQD/LFXTAL030234Reel?qs=e4%2FAndAAwgKRGsJIO2WnVQ%3D%3D" H 4400 2650 50  0001 C CNN
-	1    4400 2650
-	0    1    1    0
-$EndComp
-$Comp
-L power:GND #PWR0129
-U 1 1 6147C5EB
-P 4600 2650
-F 0 "#PWR0129" H 4600 2400 50  0001 C CNN
-F 1 "GND" H 4605 2477 50  0000 C CNN
-F 2 "" H 4600 2650 50  0001 C CNN
-F 3 "" H 4600 2650 50  0001 C CNN
-	1    4600 2650
-	1    0    0    -1
-$EndComp
 $Comp
 L power:GND #PWR0130
@@
 $EndComp
 $Comp
-L Connector_Generic:Conn_2Rows-07Pins J2
-U 1 1 614C8DA4
-P 4350 1200
-F 0 "J2" H 4400 1517 50  0000 C CNN
-F 1 "Conn_2Rows-07Pins" H 4400 1426 50  0000 C CNN
-F 2 "Connector_PinHeader_1.00mm:PinHeader_2x03_P1.00mm_Vertical_SMD" H 4350 1200 50  0001 C CNN
-F 3 "~" H 4350 1200 50  0001 C CNN
-	1    4350 1200
-	1    0    0    -1
-$EndComp
-$Comp
 L Device:R R12
 U 1 1 614D403D
@@
 Wire Wire Line
 	3450 2500 3550 2500
-Text GLabel 4150 1100 0    50   Output ~ 0
-MISO
-Text GLabel 4150 1200 0    50   Output ~ 0
-SCK
-Text GLabel 4150 1300 0    50   Output ~ 0
-RESET
 Text GLabel 4050 3500 2    50   Input ~ 0
 RESET
-Text GLabel 4650 1200 2    50   Output ~ 0
-MOSI
-$Comp
-L power:GND #PWR0132
-U 1 1 611EA8CA
-P 4650 1300
-F 0 "#PWR0132" H 4650 1050 50  0001 C CNN
-F 1 "GND" V 4655 1172 50  0000 R CNN
-F 2 "" H 4650 1300 50  0001 C CNN
-F 3 "" H 4650 1300 50  0001 C CNN
-	1    4650 1300
-	0    -1   -1   0
-$EndComp
-$Comp
-L power:GND #PWR0133
-U 1 1 611EB810
-P 4150 1400
-F 0 "#PWR0133" H 4150 1150 50  0001 C CNN
-F 1 "GND" V 4155 1272 50  0000 R CNN
-F 2 "" H 4150 1400 50  0001 C CNN
-F 3 "" H 4150 1400 50  0001 C CNN
-	1    4150 1400
-	0    1    1    0
-$EndComp
 Wire Wire Line
 	3450 3500 4000 3500
@@
 	1    2850 4700
 	1    0    0    -1
-$EndComp
-$Comp
-L power:+3V3 #PWR0135
-U 1 1 61218E15
-P 4650 1100
-F 0 "#PWR0135" H 4650 950 50  0001 C CNN
-F 1 "+3V3" V 4665 1228 50  0000 L CNN
-F 2 "" H 4650 1100 50  0001 C CNN
-F 3 "" H 4650 1100 50  0001 C CNN
-	1    4650 1100
-	0    1    1    0
 $EndComp
 $Comp
@@
 NoConn ~ 3450 4300
 NoConn ~ 3450 4400
+$Comp
+L Device:Crystal Y1
+U 1 1 6124749D
+P 4400 2650
+F 0 "Y1" V 4354 2781 50  0000 L CNN
+F 1 "Crystal" V 4445 2781 50  0000 L CNN
+F 2 "Crystal:Crystal_SMD_HC49-SD" H 4400 2650 50  0001 C CNN
+F 3 "https://www.mouser.co.uk/ProductDetail/IQD/LFXTAL030234Reel?qs=e4%2FAndAAwgKRGsJIO2WnVQ%3D%3D" H 4400 2650 50  0001 C CNN
+	1    4400 2650
+	0    1    1    0
+$EndComp
+$Comp
+L Connector:Conn_01x06_Male J2
+U 1 1 612547C1
+P 4150 1300
+F 0 "J2" H 4258 1681 50  0000 C CNN
+F 1 "Conn_01x06_Male" H 4258 1590 50  0000 C CNN
+F 2 "Connector_PinHeader_1.00mm:PinHeader_2x03_P1.00mm_Vertical_SMD" H 4150 1300 50  0001 C CNN
+F 3 "~" H 4150 1300 50  0001 C CNN
+	1    4150 1300
+	1    0    0    -1
+$EndComp
+$Comp
+L power:+3V3 #PWR0135
+U 1 1 61218E15
+P 4350 1200
+F 0 "#PWR0135" H 4350 1050 50  0001 C CNN
+F 1 "+3V3" V 4365 1328 50  0000 L CNN
+F 2 "" H 4350 1200 50  0001 C CNN
+F 3 "" H 4350 1200 50  0001 C CNN
+	1    4350 1200
+	0    1    1    0
+$EndComp
+$Comp
+L power:GND #PWR0132
+U 1 1 611EA8CA
+P 4350 1600
+F 0 "#PWR0132" H 4350 1350 50  0001 C CNN
+F 1 "GND" V 4355 1472 50  0000 R CNN
+F 2 "" H 4350 1600 50  0001 C CNN
+F 3 "" H 4350 1600 50  0001 C CNN
+	1    4350 1600
+	0    -1   -1   0
+$EndComp
+Text GLabel 4350 1400 2    50   Output ~ 0
+MOSI
+Text GLabel 4350 1500 2    50   Output ~ 0
+RESET
+Text GLabel 4350 1300 2    50   Output ~ 0
+SCK
+Text GLabel 4350 1100 2    50   Output ~ 0
+MISO
 $EndSCHEMATC

Commit message: Update for PC
Parts:
- C11, C12, C13: footprint Capacitor_SMD:C_0603_1608Metric_Pad1.08x0.95mm_HandSolder -> Capacitor_SMD:C_0402_1005Metric_Pad0.74x0.62mm_HandSolder
Changed lines of the file:
@@
 F 0 "C11" H 2665 1096 50  0000 L CNN
 F 1 "0u1" H 2665 1005 50  0000 L CNN
-F 2 "Capacitor_SMD:C_0603_1608Metric_Pad1.08x0.95mm_HandSolder" H 2588 900 50  0001 C CNN
+F 2 "Capacitor_SMD:C_0402_1005Metric_Pad0.74x0.62mm_HandSolder" H 2588 900 50  0001 C CNN
 F 3 "~" H 2550 1050 50  0001 C CNN
 	1    2550 1050
@@
 F 0 "C12" H 3015 1096 50  0000 L CNN
 F 1 "0u1" H 3015 1005 50  0000 L CNN
-F 2 "Capacitor_SMD:C_0603_1608Metric_Pad1.08x0.95mm_HandSolder" H 2938 900 50  0001 C CNN
+F 2 "Capacitor_SMD:C_0402_1005Metric_Pad0.74x0.62mm_HandSolder" H 2938 900 50  0001 C CNN
 F 3 "~" H 2900 1050 50  0001 C CNN
 	1    2900 1050
@@
 F 0 "C13" H 3365 1096 50  0000 L CNN
 F 1 "0u1" H 3365 1005 50  0000 L CNN
-F 2 "Capacitor_SMD:C_0603_1608Metric_Pad1.08x0.95mm_HandSolder" H 3288 900 50  0001 C CNN
+F 2 "Capacitor_SMD:C_0402_1005Metric_Pad0.74x0.62mm_HandSolder" H 3288 900 50  0001 C CNN
 F 3 "~" H 3250 1050 50  0001 C CNN
 	1    3250 1050

Commit message: Update once again
Changed lines of the file:
@@
 L power:GND #PWR0145
 U 1 1 6149C4AF
-P 5550 2650
-F 0 "#PWR0145" H 5550 2400 50  0001 C CNN
-F 1 "GND" V 5555 2522 50  0000 R CNN
-F 2 "" H 5550 2650 50  0001 C CNN
-F 3 "" H 5550 2650 50  0001 C CNN
-	1    5550 2650
+P 5550 2250
+F 0 "#PWR0145" H 5550 2000 50  0001 C CNN
+F 1 "GND" V 5555 2122 50  0000 R CNN
+F 2 "" H 5550 2250 50  0001 C CNN
+F 3 "" H 5550 2250 50  0001 C CNN
+	1    5550 2250
 	0    1    1    0
 $EndComp
@@
 L power:GND #PWR0147
 U 1 1 6149B341
-P 5550 2250
-F 0 "#PWR0147" H 5550 2000 50  0001 C CNN
-F 1 "GND" V 5555 2122 50  0000 R CNN
-F 2 "" H 5550 2250 50  0001 C CNN
-F 3 "" H 5550 2250 50  0001 C CNN
-	1    5550 2250
-	0    1    1    0
-$EndComp
-Connection ~ 5200 2450
-Wire Wire Line
-	5200 2550 5200 2450
-Wire Wire Line
-	5550 2550 5200 2550
-Wire Wire Line
-	5200 2450 5200 2250
-Wire Wire Line
-	5550 2450 5200 2450
+P 5550 2550
+F 0 "#PWR0147" H 5550 2300 50  0001 C CNN
+F 1 "GND" V 5555 2422 50  0000 R CNN
+F 2 "" H 5550 2550 50  0001 C CNN
+F 3 "" H 5550 2550 50  0001 C CNN
+	1    5550 2550
+	0    1    1    0
+$EndComp
+Wire Wire Line
+	5550 2650 5200 2650
 $Comp
 L power:+3V3 #PWR0148
@@
 	1    0    0    -1
 $EndComp
-Text GLabel 6950 3250 2    50   Input ~ 0
-RTS_Cellular
-Text GLabel 6950 3150 2    50   Output ~ 0
-CTS_Cellular
-Text GLabel 5550 3250 0    50   Output ~ 0
+Text GLabel 6950 3250 2    50   Output ~ 0
 RX_Cellular
-Text GLabel 5550 3150 0    50   Input ~ 0
+Text GLabel 6950 3150 2    50   Input ~ 0
 TX_Cellular
-Text GLabel 6950 2950 2    50   Output ~ 0
-CTS
-Text GLabel 6950 2850 2    50   Input ~ 0
-RTS
-Text GLabel 5550 2950 0    50   Input ~ 0
+Text GLabel 6950 2950 2    50   Input ~ 0
 TX
-Text GLabel 5550 2850 0    50   Output ~ 0
+Text GLabel 6950 2850 2    50   Output ~ 0
 RX
-$Comp
-L GPS~Hardware:SN74AVC4T774PW U6
-U 1 1 61491FC4
-P 6250 2750
-F 0 "U6" H 6250 3820 50  0000 C CNN
-F 1 "SN74AVC4T774PW" H 6250 3729 50  0000 C CNN
-F 2 "GPS Hardware:SOP65P640X120-16N" H 6250 2750 50  0001 L BNN
-F 3 "" H 6250 2750 50  0001 L BNN
-	1    6250 2750
-	1    0    0    -1
-$EndComp
 $Comp
 L Device:C C17
@@
 Text GLabel 4350 1100 2    50   Output ~ 0
 MISO
+$Comp
+L GPS~Hardware:SN74AVC4T774PW U6
+U 1 1 61491FC4
+P 6250 2750
+F 0 "U6" H 6250 3820 50  0000 C CNN
+F 1 "SN74AVC4T774PW" H 6250 3729 50  0000 C CNN
+F 2 "GPS Hardware:SOP65P640X120-16N" H 6250 2750 50  0001 L BNN
+F 3 "" H 6250 2750 50  0001 L BNN
+	1    6250 2750
+	1    0    0    -1
+$EndComp
+Text GLabel 5550 2950 0    50   Input ~ 0
+RTS
+Text GLabel 5550 2850 0    50   Output ~ 0
+CTS
+Text GLabel 5550 3250 0    50   Output ~ 0
+CTS_Cellular
+Text GLabel 5550 3150 0    50   Input ~ 0
+RTS_Cellular
+Connection ~ 5200 2450
+Wire Wire Line
+	5200 2450 5200 2250
+Wire Wire Line
+	5550 2450 5200 2450
+Wire Wire Line
+	5200 2450 5200 2650
 $EndSCHEMATC

Commit message: Update (again :+1:  )
Parts:
- C16, C17: footprint Capacitor_SMD:C_0603_1608Metric_Pad1.08x0.95mm_HandSolder -> Capacitor_SMD:C_0402_1005Metric_Pad0.74x0.62mm_HandSolder
- R15: footprint Resistor_SMD:R_0603_1608Metric_Pad0.98x0.95mm_HandSolder -> Resistor_SMD:R_0402_1005Metric_Pad0.72x0.64mm_HandSolder
Changed lines of the file:
@@
 F 0 "R15" H 4070 3796 50  0000 L CNN
 F 1 "10k" V 4000 3700 50  0000 L CNN
-F 2 "Resistor_SMD:R_0603_1608Metric_Pad0.98x0.95mm_HandSolder" V 3930 3750 50  0001 C CNN
+F 2 "Resistor_SMD:R_0402_1005Metric_Pad0.72x0.64mm_HandSolder" V 3930 3750 50  0001 C CNN
 F 3 "~" H 4000 3750 50  0001 C CNN
 	1    4000 3750
@@
 F 0 "C17" H 7715 2146 50  0000 L CNN
 F 1 "0u1" H 7715 2055 50  0000 L CNN
-F 2 "Capacitor_SMD:C_0603_1608Metric_Pad1.08x0.95mm_HandSolder" H 7638 1950 50  0001 C CNN
+F 2 "Capacitor_SMD:C_0402_1005Metric_Pad0.74x0.62mm_HandSolder" H 7638 1950 50  0001 C CNN
 F 3 "~" H 7600 2100 50  0001 C CNN
 	1    7600 2100
@@
 F 0 "C16" H 7165 2246 50  0000 L CNN
 F 1 "0u1" H 7165 2155 50  0000 L CNN
-F 2 "Capacitor_SMD:C_0603_1608Metric_Pad1.08x0.95mm_HandSolder" H 7088 2050 50  0001 C CNN
+F 2 "Capacitor_SMD:C_0402_1005Metric_Pad0.74x0.62mm_HandSolder" H 7088 2050 50  0001 C CNN
 F 3 "~" H 7050 2200 50  0001 C CNN
 	1    7050 2200
