File: KiCad/GPS Hardware/MCU.sch (KiCad schematic (older format))
At the start: 16 parts, among them J2 Conn_01x06_Male, U5 ATmega328-AU, U6 SN74AVC4T774PW, Y1 Crystal

Commit message: Update to PC
Changed lines of the file:
@@
 	1    0    0    -1
 $EndComp
-Text GLabel 3450 3100 2    50   Output ~ 0
+Text GLabel 3450 3200 2    50   Output ~ 0
 PWR_Cellular
-Text GLabel 3450 3200 2    50   Input ~ 0
+Text GLabel 3450 3100 2    50   Input ~ 0
 RESET_Cellular
 NoConn ~ 2250 2200

Commit message: Update PC
Parts:
- R12, R13, R14: value 2k2 -> 330; footprint Resistor_SMD:R_0603_1608Metric_Pad0.98x0.95mm_HandSolder -> Resistor_SMD:R_0402_1005Metric_Pad0.72x0.64mm_HandSolder
Changed lines of the file:
@@
 P 3700 2300
 F 0 "R12" V 3650 2150 50  0000 C CNN
-F 1 "2k2" V 3700 2300 50  0000 C CNN
-F 2 "Resistor_SMD:R_0603_1608Metric_Pad0.98x0.95mm_HandSolder" V 3630 2300 50  0001 C CNN
+F 1 "330" V 3700 2300 50  0000 C CNN
+F 2 "Resistor_SMD:R_0402_1005Metric_Pad0.72x0.64mm_HandSolder" V 3630 2300 50  0001 C CNN
 F 3 "~" H 3700 2300 50  0001 C CNN
 	1    3700 2300
@@
 P 3700 2400
 F 0 "R13" V 3650 2250 50  0000 C CNN
-F 1 "2k2" V 3700 2400 50  0000 C CNN
-F 2 "Resistor_SMD:R_0603_1608Metric_Pad0.98x0.95mm_HandSolder" V 3630 2400 50  0001 C CNN
+F 1 "330" V 3700 2400 50  0000 C CNN
+F 2 "Resistor_SMD:R_0402_1005Metric_Pad0.72x0.64mm_HandSolder" V 3630 2400 50  0001 C CNN
 F 3 "~" H 3700 2400 50  0001 C CNN
 	1    3700 2400
@@
 P 3700 2500
 F 0 "R14" V 3650 2350 50  0000 C CNN
-F 1 "2k2" V 3700 2500 50  0000 C CNN
-F 2 "Resistor_SMD:R_0603_1608Metric_Pad0.98x0.95mm_HandSolder" V 3630 2500 50  0001 C CNN
+F 1 "330" V 3700 2500 50  0000 C CNN
+F 2 "Resistor_SMD:R_0402_1005Metric_Pad0.72x0.64mm_HandSolder" V 3630 2500 50  0001 C CNN
 F 3 "~" H 3700 2500 50  0001 C CNN
 	1    3700 2500
@@
 L power:GND #PWR0132
 U 1 1 611EA8CA
-P 4350 1600
-F 0 "#PWR0132" H 4350 1350 50  0001 C CNN
-F 1 "GND" V 4355 1472 50  0000 R CNN
-F 2 "" H 4350 1600 50  0001 C CNN
-F 3 "" H 4350 1600 50  0001 C CNN
-	1    4350 1600
+P 4350 1400
+F 0 "#PWR0132" H 4350 1150 50  0001 C CNN
+F 1 "GND" V 4355 1272 50  0000 R CNN
+F 2 "" H 4350 1400 50  0001 C CNN
+F 3 "" H 4350 1400 50  0001 C CNN
+	1    4350 1400
 	0    -1   -1   0
 $EndComp
-Text GLabel 4350 1400 2    50   Output ~ 0
+Text GLabel 4350 1500 2    50   Output ~ 0
 MOSI
-Text GLabel 4350 1500 2    50   Output ~ 0
+Text GLabel 4350 1600 2    50   Output ~ 0
 RESET
+Text GLabel 4350 1100 2    50   Output ~ 0
+SCK
 Text GLabel 4350 1300 2    50   Output ~ 0
-SCK
-Text GLabel 4350 1100 2    50   Output ~ 0
 MISO
 $Comp

Commit message: Update to PC
Parts:
- C10: footprint Capacitor_SMD:C_0603_1608Metric_Pad1.08x0.95mm_HandSolder -> Capacitor_SMD:C_0402_1005Metric_Pad0.74x0.62mm_HandSolder
Changed lines of the file:
@@
 F 0 "C10" H 2065 2246 50  0000 L CNN
 F 1 "0u1" H 2065 2155 50  0000 L CNN
-F 2 "Capacitor_SMD:C_0603_1608Metric_Pad1.08x0.95mm_HandSolder" H 1988 2050 50  0001 C CNN
+F 2 "Capacitor_SMD:C_0402_1005Metric_Pad0.74x0.62mm_HandSolder" H 1988 2050 50  0001 C CNN
 F 3 "~" H 1950 2200 50  0001 C CNN
 	1    1950 2200

Commit message: Updated the sim choice to a push-push type, and generated the final gerber files
Parts:
- C10, C11, C12, C13, C14, C15, C16, C17: symbol Device:C -> GPS-Hardware-rescue:C-Device
- J2: symbol Connector:Conn_01x06_Male -> GPS-Hardware-rescue:Conn_01x06_Male-Connector
- R12, R13, R14, R15: symbol Device:R -> GPS-Hardware-rescue:R-Device
- U5: symbol MCU_Microchip_ATmega:ATmega328-AU -> GPS-Hardware-rescue:ATmega328-AU-MCU_Microchip_ATmega
- Y1: symbol Device:Crystal -> GPS-Hardware-rescue:Crystal-Device
Changed lines of the file:
@@
 $EndDescr
 $Comp
-L MCU_Microchip_ATmega:ATmega328-AU U5
+L GPS-Hardware-rescue:ATmega328-AU-MCU_Microchip_ATmega U5
 U 1 1 61474832
 P 2850 3200
@@
 $EndComp
 $Comp
-L Device:C C10
+L GPS-Hardware-rescue:C-Device C10
 U 1 1 6147650D
 P 1950 2200
@@
 $EndComp
 $Comp
-L power:GND #PWR0127
+L GPS-Hardware-rescue:GND-power #PWR0127
 U 1 1 61476BD2
 P 1950 2350
@@
 	3450 2700 3950 2700
 $Comp
-L Device:C C14
+L GPS-Hardware-rescue:C-Device C14
 U 1 1 6147B129
 P 4400 2350
@@
 Connection ~ 4400 2500
 $Comp
-L Device:C C15
+L GPS-Hardware-rescue:C-Device C15
 U 1 1 6147BAE8
 P 4400 2950
@@
 Connection ~ 4400 2800
 $Comp
-L power:GND #PWR0130
+L GPS-Hardware-rescue:GND-power #PWR0130
 U 1 1 6147CE24
 P 4400 2200
@@
 $EndComp
 $Comp
-L power:GND #PWR0131
+L GPS-Hardware-rescue:GND-power #PWR0131
 U 1 1 6147D183
 P 4400 3100
@@
 SCK
 $Comp
-L Device:R R15
+L GPS-Hardware-rescue:R-Device R15
 U 1 1 614B0F0F
 P 4000 3750
@@
 $EndComp
 $Comp
-L Device:R R12
+L GPS-Hardware-rescue:R-Device R12
 U 1 1 614D403D
 P 3700 2300
@@
 $EndComp
 $Comp
-L Device:R R13
+L GPS-Hardware-rescue:R-Device R13
 U 1 1 614D4D77
 P 3700 2400
@@
 $EndComp
 $Comp
-L Device:R R14
+L GPS-Hardware-rescue:R-Device R14
 U 1 1 614D58E3
 P 3700 2500
@@
 	4000 3900 4000 3950
 $Comp
-L power:GND #PWR0134
+L GPS-Hardware-rescue:GND-power #PWR0134
 U 1 1 61218305
 P 2850 4700
@@
 $EndComp
 $Comp
-L power:+3V3 #PWR0136
+L GPS-Hardware-rescue:+3V3-power #PWR0136
 U 1 1 6121A2B1
 P 4000 3950
@@
 	2850 1700 2950 1700
 $Comp
-L power:+3V3 #PWR0137
+L GPS-Hardware-rescue:+3V3-power #PWR0137
 U 1 1 6121C704
 P 2850 1700
@@
 Connection ~ 2850 1700
 $Comp
-L Device:C C11
+L GPS-Hardware-rescue:C-Device C11
 U 1 1 6121D0CD
 P 2550 1050
@@
 $EndComp
 $Comp
-L Device:C C12
+L GPS-Hardware-rescue:C-Device C12
 U 1 1 6121E29B
 P 2900 1050
@@
 $EndComp
 $Comp
-L Device:C C13
+L GPS-Hardware-rescue:C-Device C13
 U 1 1 6121E902
 P 3250 1050
@@
 	2900 900  3250 900
 $Comp
-L power:+3V3 #PWR0138
+L GPS-Hardware-rescue:+3V3-power #PWR0138
 U 1 1 6121FA8B
 P 2900 900
@@
 $EndComp
 $Comp
-L power:GND #PWR0139
+L GPS-Hardware-rescue:GND-power #PWR0139
 U 1 1 612206D8
 P 2550 1200
@@
 $EndComp
 $Comp
-L power:GND #PWR0140
+L GPS-Hardware-rescue:GND-power #PWR0140
 U 1 1 61220D84
 P 2900 1200
@@
 $EndComp
 $Comp
-L power:GND #PWR0141
+L GPS-Hardware-rescue:GND-power #PWR0141
 U 1 1 612213CA
 P 3250 1200
@@
 	2250 2000 1950 2000
 $Comp
-L power:+1V8 #PWR0142
+L GPS-Hardware-rescue:+1V8-power #PWR0142
 U 1 1 6149F6C9
 P 7150 2050
@@
 $EndComp
 $Comp
-L power:+3V3 #PWR0143
+L GPS-Hardware-rescue:+3V3-power #PWR0143
 U 1 1 6149E56B
 P 7700 1950
@@
 $EndComp
 $Comp
-L power:GND #PWR0144
+L GPS-Hardware-rescue:GND-power #PWR0144
 U 1 1 6149DEBA
 P 6950 3450
@@
 $EndComp
 $Comp
-L power:GND #PWR0145
+L GPS-Hardware-rescue:GND-power #PWR0145
 U 1 1 6149C4AF
 P 5550 2250
@@
 $EndComp
 $Comp
-L power:GND #PWR0146
+L GPS-Hardware-rescue:GND-power #PWR0146
 U 1 1 6149BDCB
 P 5550 2350
@@
 $EndComp
 $Comp
-L power:GND #PWR0147
+L GPS-Hardware-rescue:GND-power #PWR0147
 U 1 1 6149B341
 P 5550 2550
@@
 	5550 2650 5200 2650
 $Comp
-L power:+3V3 #PWR0148
+L GPS-Hardware-rescue:+3V3-power #PWR0148
 U 1 1 6149A2FD
 P 5200 2250
@@
 RX
 $Comp
-L Device:C C17
+L GPS-Hardware-rescue:C-Device C17
 U 1 1 612AD4B1
 P 7600 2100
@@
 $EndComp
 $Comp
-L Device:C C16
+L GPS-Hardware-rescue:C-Device C16
 U 1 1 612AE26D
 P 7050 2200
@@
 	7050 2050 6950 2050
 $Comp
-L power:GND #PWR0110
+L GPS-Hardware-rescue:GND-power #PWR0110
 U 1 1 612DF9B5
 P 7050 2350
@@
 $EndComp
 $Comp
-L power:GND #PWR0149
+L GPS-Hardware-rescue:GND-power #PWR0149
 U 1 1 612E15CE
 P 7600 2250
@@
 NoConn ~ 3450 4400
 $Comp
-L Device:Crystal Y1
+L GPS-Hardware-rescue:Crystal-Device Y1
 U 1 1 6124749D
 P 4400 2650
@@
 $EndComp
 $Comp
-L Connector:Conn_01x06_Male J2
+L GPS-Hardware-rescue:Conn_01x06_Male-Connector J2
 U 1 1 612547C1
 P 4150 1300
+AR Path="/612547C1" Ref="J2"  Part="1"
+AR Path="/613BCFBA/612547C1" Ref="J2"  Part="1"
 F 0 "J2" H 4258 1681 50  0000 C CNN
 F 1 "Conn_01x06_Male" H 4258 1590 50  0000 C CNN
@@
 $EndComp
 $Comp
-L power:+3V3 #PWR0135
+L GPS-Hardware-rescue:+3V3-power #PWR0135
 U 1 1 61218E15
 P 4350 1200
@@
 $EndComp
 $Comp
-L power:GND #PWR0132
+L GPS-Hardware-rescue:GND-power #PWR0132
 U 1 1 611EA8CA
 P 4350 1400
