File: KiCad/GPS Hardware/Cellular and GPS.sch (KiCad schematic (older format))
At the start: 0 parts

Commit message: Finished adding components, need to add values
Parts:
- added C? (x14): C, symbol Device:C
- added D? (x4): D_TVS, symbol Device:D_TVS
- added D?: LED, symbol Device:LED
- added J?: Conn_Coaxial, symbol Connector:Conn_Coaxial
- added J?: SIM7050-6-0-00-X_REVC, GCT_SIM7050-6-0-00-X_REVC, symbol GPS~Hardware:SIM7050-6-0-00-X_REVC
- added Q?: BC847, Package_TO_SOT_SMD:SOT-23, symbol Transistor_BJT:BC847
- added R? (x5): R, symbol Device:R
- added U?: SARA-U201, RF_GSM:ublox_SARA-G3_LGA-96, symbol RF_GSM:SARA-U201
- added U?: ublox_SAM-M8Q, RF_GPS:ublox_SAM-M8Q, symbol RF_GPS:ublox_SAM-M8Q
- added U?: NCP662SQ33T1G, symbol GPS~Hardware:NCP662SQ33T1G
- added U?: 74AVC2T245GU-Q100X, symbol GPS~Hardware:74AVC2T245GU-Q100X
Connections:
- net labels added: +1V8, +3V3, CLK, CTS_Cellular, EXTINT, GND, GPIO2, GPIO3, GPIO4, IO, PWR_Cellular, RESET_Cellular, RST, RTS_Cellular, RX_Cellular, TX_Cellular, TX_GPS, VCC, VCC_GPS, VSIM
- wire segments 0 -> 42
- no-connect marks 0 -> 23
