File: KiCad/GPS Hardware/Cellular and GPS.sch (KiCad schematic (older format))
At the start: 31 parts

Commit message: Added footprints to most components
Parts:
- C18: renamed from C?; value C -> 10n; footprint (none) -> Capacitor_SMD:C_0402_1005Metric_Pad0.74x0.62mm_HandSolder
- C19, C22, C23, C24, C26, C27: renamed from C?; value C -> 0u1; footprint (none) -> Capacitor_SMD:C_0603_1608Metric_Pad1.08x0.95mm_HandSolder
- C20: renamed from C?; value C -> 56p; footprint (none) -> Capacitor_SMD:C_0402_1005Metric_Pad0.74x0.62mm_HandSolder
- C21: renamed from C?; value C -> 15p; footprint (none) -> Capacitor_SMD:C_0402_1005Metric_Pad0.74x0.62mm_HandSolder
- C25: renamed from C?; value C -> 4u7; footprint (none) -> Capacitor_SMD:C_0603_1608Metric_Pad1.08x0.95mm_HandSolder
- C28, C29, C30, C31: renamed from C?; value C -> 47p; footprint (none) -> Capacitor_SMD:C_0402_1005Metric_Pad0.74x0.62mm_HandSolder
- D2: renamed from D?; footprint (none) -> LED_SMD:LED_0603_1608Metric_Pad1.05x0.95mm_HandSolder
- D3, D4, D5, D6: renamed from D?; value D_TVS -> PESD0402; footprint (none) -> Capacitor_SMD:C_0402_1005Metric_Pad0.74x0.62mm_HandSolder
- J3: renamed from J?; footprint (none) -> GPS Hardware:RFSOLUTIONS_CON-SMA-EDGE-S
- R16: renamed from R?; value R -> 100k; footprint (none) -> Resistor_SMD:R_0603_1608Metric_Pad0.98x0.95mm_HandSolder
- R17: renamed from R?; value R -> 10k; footprint (none) -> Resistor_SMD:R_0603_1608Metric_Pad0.98x0.95mm_HandSolder
- R18, R20: renamed from R?; value R -> 47k; footprint (none) -> Resistor_SMD:R_0603_1608Metric_Pad0.98x0.95mm_HandSolder
- R19: renamed from R?; value R -> 820; footprint (none) -> Resistor_SMD:R_0603_1608Metric_Pad0.98x0.95mm_HandSolder
- gave numbers to parts that had none: 6

Commit message: Added all footprints
Hopefully they are correct :)
Parts:
- J4: footprint GCT_SIM7050-6-0-00-X_REVC -> GPS Hardware:GCT_SIM7050-6-0-00-X_REVC
- U7: footprint (none) -> GPS Hardware:QFN40P140X180X50-10N
- U9: footprint (none) -> GPS Hardware:SOT95P240X120-3N
Changed lines of the file:
@@
 F 0 "J4" H 9200 1767 50  0000 C CNN
 F 1 "SIM7050-6-0-00-X_REVC" H 9200 1676 50  0000 C CNN
-F 2 "GCT_SIM7050-6-0-00-X_REVC" H 9200 1400 50  0001 L BNN
+F 2 "GPS Hardware:GCT_SIM7050-6-0-00-X_REVC" H 9200 1400 50  0001 L BNN
 F 3 "" H 9200 1400 50  0001 L BNN
 F 4 "GCT" H 9200 1400 50  0001 L BNN "MANUFACTURER"
@@
 F 0 "U9" H 5500 4625 50  0000 C CNN
 F 1 "NCP662SQ33T1G" H 5500 4534 50  0000 C CNN
-F 2 "" H 5500 4300 50  0001 C CNN
+F 2 "GPS Hardware:SOT95P240X120-3N" H 5500 4300 50  0001 C CNN
 F 3 "" H 5500 4300 50  0001 C CNN
 	1    5500 4300
@@
 F 0 "U7" H 2750 6415 50  0000 C CNN
 F 1 "74AVC2T245GU-Q100X" H 2750 6324 50  0000 C CNN
-F 2 "" H 2750 5850 50  0001 C CNN
+F 2 "GPS Hardware:QFN40P140X180X50-10N" H 2750 5850 50  0001 C CNN
 F 3 "" H 2750 5850 50  0001 C CNN
 	1    2750 5850
@@
 Text GLabel 7850 1400 0    50   Input ~ 0
 VSIM
+$Comp
+L power:GND #PWR0113
+U 1 1 61244203
+P 3900 1750
+F 0 "#PWR0113" H 3900 1500 50  0001 C CNN
+F 1 "GND" H 3905 1577 50  0000 C CNN
+F 2 "" H 3900 1750 50  0001 C CNN
+F 3 "" H 3900 1750 50  0001 C CNN
+	1    3900 1750
+	-1   0    0    1
+$EndComp
 $EndSCHEMATC

Commit message: Update
Parts:
- removed J4: SIM7050-6-0-00-X_REVC, GPS Hardware:GCT_SIM7050-6-0-00-X_REVC, symbol GPS~Hardware:SIM7050-6-0-00-X_REVC
- added J4: SIM8051-6-0-14-01-X-REVD, GCT_SIM8051-6-0-14-01-X-REVD, symbol GPS~Hardware:SIM8051-6-0-14-01-X-REVD
- C27: value 0u1 -> 47p; footprint Capacitor_SMD:C_0603_1608Metric_Pad1.08x0.95mm_HandSolder -> Capacitor_SMD:C_0402_1005Metric_Pad0.74x0.62mm_HandSolder
- C31: value 47p -> 0u1; footprint Capacitor_SMD:C_0402_1005Metric_Pad0.74x0.62mm_HandSolder -> Capacitor_SMD:C_0603_1608Metric_Pad1.08x0.95mm_HandSolder

Commit message: Update to laptop
Parts:
- J4: footprint GCT_SIM8051-6-0-14-01-X-REVD -> GPS Hardware:GCT_SIM8051-6-0-14-01-X-REVD
Changed lines of the file:
@@
 F 0 "J4" H 9200 2917 50  0000 C CNN
 F 1 "SIM8051-6-0-14-01-X-REVD" H 9200 2826 50  0000 C CNN
-F 2 "GCT_SIM8051-6-0-14-01-X-REVD" H 9100 2550 50  0001 L BNN
+F 2 "GPS Hardware:GCT_SIM8051-6-0-14-01-X-REVD" H 9100 2550 50  0001 L BNN
 F 3 "" H 9100 2550 50  0001 L BNN
 F 4 "GCT" H 9100 2550 50  0001 L BNN "MANUFACTURER"

Commit message: Update (again :+1:  )
Parts:
- R16: footprint Resistor_SMD:R_0603_1608Metric_Pad0.98x0.95mm_HandSolder -> Resistor_SMD:R_0402_1005Metric_Pad0.72x0.64mm_HandSolder
Changed lines of the file:
@@
 F 0 "R16" H 1770 2746 50  0000 L CNN
 F 1 "100k" H 1770 2655 50  0000 L CNN
-F 2 "Resistor_SMD:R_0603_1608Metric_Pad0.98x0.95mm_HandSolder" V 1630 2700 50  0001 C CNN
+F 2 "Resistor_SMD:R_0402_1005Metric_Pad0.72x0.64mm_HandSolder" V 1630 2700 50  0001 C CNN
 F 3 "~" H 1700 2700 50  0001 C CNN
 	1    1700 2700

Commit message: Update
Parts:
- C19: footprint Capacitor_SMD:C_0603_1608Metric_Pad1.08x0.95mm_HandSolder -> Capacitor_SMD:C_0402_1005Metric_Pad0.74x0.62mm_HandSolder
Changed lines of the file:
@@
 F 0 "C19" H 2265 1396 50  0000 L CNN
 F 1 "0u1" H 2265 1305 50  0000 L CNN
-F 2 "Capacitor_SMD:C_0603_1608Metric_Pad1.08x0.95mm_HandSolder" H 2188 1200 50  0001 C CNN
+F 2 "Capacitor_SMD:C_0402_1005Metric_Pad0.74x0.62mm_HandSolder" H 2188 1200 50  0001 C CNN
 F 3 "~" H 2150 1350 50  0001 C CNN
 	1    2150 1350

Commit message: Update to PC
Parts:
- removed C24, C26: 0u1, Capacitor_SMD:C_0603_1608Metric_Pad1.08x0.95mm_HandSolder, symbol Device:C
- removed U9: NCP662SQ33T1G, GPS Hardware:SOT95P240X120-3N, symbol GPS~Hardware:NCP662SQ33T1G
- added Q2: BC847, Package_TO_SOT_SMD:SOT-23, symbol Transistor_BJT:BC847
- added Q3: BSS84, Package_TO_SOT_SMD:SOT-323_SC-70, symbol Transistor_FET:BSS84
- C22, C23, C25: footprint Capacitor_SMD:C_0603_1608Metric_Pad1.08x0.95mm_HandSolder -> Capacitor_SMD:C_0402_1005Metric_Pad0.74x0.62mm_HandSolder
- R20: footprint Resistor_SMD:R_0603_1608Metric_Pad0.98x0.95mm_HandSolder -> Resistor_SMD:R_0402_1005Metric_Pad0.72x0.64mm_HandSolder
Connections:
- wire segments 42 -> 45
Other:
- note added: "GPIO2 Pin has a 1ma output, no need for a resistor"
Changed lines of the file:
@@
 	1    0    0    -1
 $EndComp
-$Comp
-L GPS~Hardware:NCP662SQ33T1G U9
-U 1 1 614F6EC1
-P 5500 4300
-F 0 "U9" H 5500 4625 50  0000 C CNN
-F 1 "NCP662SQ33T1G" H 5500 4534 50  0000 C CNN
-F 2 "GPS Hardware:SOT95P240X120-3N" H 5500 4300 50  0001 C CNN
-F 3 "" H 5500 4300 50  0001 C CNN
-	1    5500 4300
-	1    0    0    -1
-$EndComp
-Text GLabel 4700 4400 0    50   Input ~ 0
-VCC
-$Comp
-L Device:C C24
-U 1 1 61505EC5
-P 4850 4550
-F 0 "C24" H 4965 4596 50  0000 L CNN
-F 1 "0u1" H 4965 4505 50  0000 L CNN
-F 2 "Capacitor_SMD:C_0603_1608Metric_Pad1.08x0.95mm_HandSolder" H 4888 4400 50  0001 C CNN
-F 3 "~" H 4850 4550 50  0001 C CNN
-	1    4850 4550
-	1    0    0    -1
-$EndComp
-$Comp
-L power:GND #PWR0167
-U 1 1 6150A428
-P 4850 4700
-F 0 "#PWR0167" H 4850 4450 50  0001 C CNN
-F 1 "GND" H 4855 4527 50  0000 C CNN
-F 2 "" H 4850 4700 50  0001 C CNN
-F 3 "" H 4850 4700 50  0001 C CNN
-	1    4850 4700
-	1    0    0    -1
-$EndComp
-Wire Wire Line
-	4850 4400 4700 4400
-Wire Wire Line
-	4850 4400 5000 4400
-Connection ~ 4850 4400
-$Comp
-L power:GND #PWR0168
-U 1 1 6151004E
-P 5000 4200
-F 0 "#PWR0168" H 5000 3950 50  0001 C CNN
-F 1 "GND" V 5005 4072 50  0000 R CNN
-F 2 "" H 5000 4200 50  0001 C CNN
-F 3 "" H 5000 4200 50  0001 C CNN
-	1    5000 4200
-	0    1    1    0
-$EndComp
-$Comp
-L Device:C C26
-U 1 1 61510928
-P 6050 4550
-F 0 "C26" H 6165 4596 50  0000 L CNN
-F 1 "0u1" H 6165 4505 50  0000 L CNN
-F 2 "Capacitor_SMD:C_0603_1608Metric_Pad1.08x0.95mm_HandSolder" H 6088 4400 50  0001 C CNN
-F 3 "~" H 6050 4550 50  0001 C CNN
-	1    6050 4550
-	1    0    0    -1
-$EndComp
-$Comp
-L power:GND #PWR0169
-U 1 1 615113AB
-P 6050 4700
-F 0 "#PWR0169" H 6050 4450 50  0001 C CNN
-F 1 "GND" H 6055 4527 50  0000 C CNN
-F 2 "" H 6050 4700 50  0001 C CNN
-F 3 "" H 6050 4700 50  0001 C CNN
-	1    6050 4700
-	1    0    0    -1
-$EndComp
-Wire Wire Line
-	6000 4400 6050 4400
-Text GLabel 6300 4400 2    50   Output ~ 0
-VCC_GPS
-Wire Wire Line
-	6050 4400 6300 4400
-Connection ~ 6050 4400
-$Comp
-L Device:R R?
-U 1 1 6151C5E7
-P 6100 4050
-AR Path="/613BCFBA/6151C5E7" Ref="R?"  Part="1"
-AR Path="/613BCFF5/6151C5E7" Ref="R20"  Part="1"
-F 0 "R20" H 6170 4096 50  0000 L CNN
-F 1 "47k" V 6100 4000 50  0000 L CNN
-F 2 "Resistor_SMD:R_0603_1608Metric_Pad0.98x0.95mm_HandSolder" V 6030 4050 50  0001 C CNN
-F 3 "~" H 6100 4050 50  0001 C CNN
-	1    6100 4050
-	1    0    0    -1
-$EndComp
-Wire Wire Line
-	6000 4200 6100 4200
-$Comp
-L power:GND #PWR0170
-U 1 1 6151E09F
-P 6100 3900
-F 0 "#PWR0170" H 6100 3650 50  0001 C CNN
-F 1 "GND" H 6105 3727 50  0000 C CNN
-F 2 "" H 6100 3900 50  0001 C CNN
-F 3 "" H 6100 3900 50  0001 C CNN
-	1    6100 3900
-	-1   0    0    1
-$EndComp
-Text GLabel 6300 4200 2    50   Input ~ 0
-GPIO2
-Wire Wire Line
-	6300 4200 6100 4200
-Connection ~ 6100 4200
 Text GLabel 3700 2950 2    50   Output ~ 0
 GPIO2
@@
 F 0 "C22" H 3415 5896 50  0000 L CNN
 F 1 "0u1" H 3415 5805 50  0000 L CNN
-F 2 "Capacitor_SMD:C_0603_1608Metric_Pad1.08x0.95mm_HandSolder" H 3338 5700 50  0001 C CNN
+F 2 "Capacitor_SMD:C_0402_1005Metric_Pad0.74x0.62mm_HandSolder" H 3338 5700 50  0001 C CNN
 F 3 "~" H 3300 5850 50  0001 C CNN
 	1    3300 5850
@@
 F 0 "C23" H 4065 5796 50  0000 L CNN
 F 1 "0u1" H 4065 5705 50  0000 L CNN
-F 2 "Capacitor_SMD:C_0603_1608Metric_Pad1.08x0.95mm_HandSolder" H 3988 5600 50  0001 C CNN
+F 2 "Capacitor_SMD:C_0402_1005Metric_Pad0.74x0.62mm_HandSolder" H 3988 5600 50  0001 C CNN
 F 3 "~" H 3950 5750 50  0001 C CNN
 	1    3950 5750
@@
 F 0 "C25" V 5498 5700 50  0000 C CNN
 F 1 "4u7" V 5589 5700 50  0000 C CNN
-F 2 "Capacitor_SMD:C_0603_1608Metric_Pad1.08x0.95mm_HandSolder" H 5788 5550 50  0001 C CNN
+F 2 "Capacitor_SMD:C_0402_1005Metric_Pad0.74x0.62mm_HandSolder" H 5788 5550 50  0001 C CNN
 F 3 "~" H 5750 5700 50  0001 C CNN
 	1    5750 5700
@@
 F 1 "BC847" H 4541 2805 50  0000 L CNN
 F 2 "Package_TO_SOT_SMD:SOT-23" H 4550 2775 50  0001 L CIN
-F 3 "http://www.infineon.com/dgdl/Infineon-BC847SERIES_BC848SERIES_BC849SERIES_BC850SERIES-DS-v01_01-en.pdf?fileId=db3a304314dca389011541d4630a1657" H 4350 2850 50  0001 L CNN
+F 3 "https://www.mouser.co.uk/datasheet/2/308/1/BC846ALT1_D-2310268.pdf" H 4350 2850 50  0001 L CNN
 	1    4350 2850
 	1    0    0    -1
@@
 $EndComp
 NoConn ~ 9600 2550
+$Comp
+L Transistor_BJT:BC847 Q2
+U 1 1 613C6B7F
+P 5050 4050
+F 0 "Q2" H 5241 4096 50  0000 L CNN
+F 1 "BC847" H 5241 4005 50  0000 L CNN
+F 2 "Package_TO_SOT_SMD:SOT-23" H 5250 3975 50  0001 L CIN
+F 3 "https://www.mouser.co.uk/datasheet/2/308/1/BC846ALT1_D-2310268.pdf" H 5050 4050 50  0001 L CNN
+	1    5050 4050
+	1    0    0    -1
+$EndComp
+Text GLabel 4750 4050 0    50   Input ~ 0
+GPIO2
+Wire Wire Line
+	4750 4050 4850 4050
+$Comp
+L power:GND #PWR0104
+U 1 1 613D3752
+P 5150 4350
+F 0 "#PWR0104" H 5150 4100 50  0001 C CNN
+F 1 "GND" H 5155 4177 50  0000 C CNN
+F 2 "" H 5150 4350 50  0001 C CNN
+F 3 "" H 5150 4350 50  0001 C CNN
+	1    5150 4350
+	1    0    0    -1
+$EndComp
+Wire Wire Line
+	5150 4250 5150 4350
+$Comp
+L Device:R R20
+U 1 1 613D777A
+P 5150 3600
+F 0 "R20" H 5220 3646 50  0000 L CNN
+F 1 "47k" H 5220 3555 50  0000 L CNN
+F 2 "Resistor_SMD:R_0402_1005Metric_Pad0.72x0.64mm_HandSolder" V 5080 3600 50  0001 C CNN
+F 3 "~" H 5150 3600 50  0001 C CNN
+	1    5150 3600
+	1    0    0    -1
+$EndComp
+Wire Wire Line
+	5150 3750 5150 3800
+$Comp
+L power:+3V3 #PWR0163
+U 1 1 613DE378
+P 5150 3350
+F 0 "#PWR0163" H 5150 3200 50  0001 C CNN
+F 1 "+3V3" H 5165 3523 50  0000 C CNN
+F 2 "" H 5150 3350 50  0001 C CNN
+F 3 "" H 5150 3350 50  0001 C CNN
+	1    5150 3350
+	1    0    0    -1
+$EndComp
+Wire Wire Line
+	5150 3450 5150 3350
+$Comp
+L Transistor_FET:BSS84 Q3
+U 1 1 613E1FB9
+P 5650 3800
+F 0 "Q3" H 5854 3754 50  0000 L CNN
+F 1 "BSS84" H 5854 3845 50  0000 L CNN
+F 2 "Package_TO_SOT_SMD:SOT-323_SC-70" H 5850 3725 50  0001 L CIN
+F 3 "http://assets.nexperia.com/documents/data-sheet/BSS84.pdf" H 5650 3800 50  0001 L CNN
+	1    5650 3800
+	1    0    0    1
+$EndComp
+Wire Wire Line
+	5450 3800 5150 3800
+Connection ~ 5150 3800
+Wire Wire Line
+	5150 3800 5150 3850
+Wire Wire Line
+	5150 3450 5750 3450
+Wire Wire Line
+	5750 3450 5750 3600
+Connection ~ 5150 3450
+Text GLabel 5750 4050 3    50   Output ~ 0
+VCC_GPS
+Wire Wire Line
+	5750 4000 5750 4050
+Text Notes 4200 4700 0    50   ~ 0
+GPIO2 Pin has a 1ma output, no need for a resistor
 $EndSCHEMATC

Commit message: Updated the sim choice to a push-push type, and generated the final gerber files
Parts:
- removed J4: SIM8051-6-0-14-01-X-REVD, GPS Hardware:GCT_SIM8051-6-0-14-01-X-REVD, symbol GPS~Hardware:SIM8051-6-0-14-01-X-REVD
- added J?: SIM8065-6-1-14-01-A_REVA1, GCT_SIM8065-6-1-14-01-A_REVA1, symbol GPS~Hardware:SIM8065-6-1-14-01-A_REVA1
- C18, C19, C20, C21, C22, C23, C25, C27, C28, C29, C30, C31: symbol Device:C -> GPS-Hardware-rescue:C-Device
- D2: symbol Device:LED -> GPS-Hardware-rescue:LED-Device
- D3, D4, D5, D6: symbol Device:D_TVS -> GPS-Hardware-rescue:D_TVS-Device
- J3: symbol Connector:Conn_Coaxial -> GPS-Hardware-rescue:Conn_Coaxial-Connector
- Q1, Q2: symbol Transistor_BJT:BC847 -> GPS-Hardware-rescue:BC847-Transistor_BJT
- Q3: symbol Transistor_FET:BSS84 -> GPS-Hardware-rescue:BSS84-Transistor_FET
- R16, R17, R18, R19, R20: symbol Device:R -> GPS-Hardware-rescue:R-Device
- U10: symbol RF_GPS:ublox_SAM-M8Q -> GPS-Hardware-rescue:ublox_SAM-M8Q-RF_GPS
- U8: symbol RF_GSM:SARA-U201 -> GPS-Hardware-rescue:SARA-U201-RF_GSM
Connections:
- wire segments 45 -> 50
- no-connect marks 23 -> 24
Other:
- moved on the sheet: C27, C28, C29, C30, C31, D3, D4, D5, D6
