File: KiCad/GPS Hardware/Power.sch (KiCad schematic (older format))
At the start: 27 parts

Commit message: Update
Parts:
- removed U?: SARA-U201, RF_GSM:ublox_SARA-G3_LGA-96, symbol RF_GSM:SARA-U201
- added C? (x2): C, symbol Device:C
- added U?: LM3480-3.3, Package_TO_SOT_SMD:SOT-23, symbol Regulator_Linear:LM3480-3.3
Connections:
- net labels added: +3V3
- wire segments 41 -> 46
Changed lines of the file:
@@
 Text GLabel 1750 950  2    50   Output ~ 0
 VBUS
-Text GLabel 3850 950  0    50   Input ~ 0
+Text GLabel 3750 950  0    50   Input ~ 0
 VBUS
 Text GLabel 1800 1700 2    50   Output ~ 0
@@
 P 1150 2450
 AR Path="/613BC25E" Ref="#PWR?"  Part="1"
-AR Path="/613B204B/613BC25E" Ref="#PWR?"  Part="1"
-F 0 "#PWR?" H 1150 2200 50  0001 C CNN
+AR Path="/613B204B/613BC25E" Ref="#PWR0101"  Part="1"
+F 0 "#PWR0101" H 1150 2200 50  0001 C CNN
 F 1 "GND" H 1155 2277 50  0000 C CNN
 F 2 "" H 1150 2450 50  0001 C CNN
@@
 P 5150 3050
 AR Path="/613BC264" Ref="#PWR?"  Part="1"
-AR Path="/613B204B/613BC264" Ref="#PWR?"  Part="1"
-F 0 "#PWR?" H 5150 2800 50  0001 C CNN
+AR Path="/613B204B/613BC264" Ref="#PWR0102"  Part="1"
+F 0 "#PWR0102" H 5150 2800 50  0001 C CNN
 F 1 "GND" H 5155 2877 50  0000 C CNN
 F 2 "" H 5150 3050 50  0001 C CNN
@@
 P 3200 1250
 AR Path="/613BC26A" Ref="#PWR?"  Part="1"
-AR Path="/613B204B/613BC26A" Ref="#PWR?"  Part="1"
-F 0 "#PWR?" H 3200 1000 50  0001 C CNN
+AR Path="/613B204B/613BC26A" Ref="#PWR0103"  Part="1"
+F 0 "#PWR0103" H 3200 1000 50  0001 C CNN
 F 1 "GND" H 3205 1077 50  0000 C CNN
 F 2 "" H 3200 1250 50  0001 C CNN
@@
 P 3200 1950
 AR Path="/613BC270" Ref="#PWR?"  Part="1"
-AR Path="/613B204B/613BC270" Ref="#PWR?"  Part="1"
-F 0 "#PWR?" H 3200 1700 50  0001 C CNN
+AR Path="/613B204B/613BC270" Ref="#PWR0104"  Part="1"
+F 0 "#PWR0104" H 3200 1700 50  0001 C CNN
 F 1 "GND" H 3205 1777 50  0000 C CNN
 F 2 "" H 3200 1950 50  0001 C CNN
@@
 P 3950 2100
 AR Path="/613BC27C" Ref="#PWR?"  Part="1"
-AR Path="/613B204B/613BC27C" Ref="#PWR?"  Part="1"
-F 0 "#PWR?" H 3950 1850 50  0001 C CNN
+AR Path="/613B204B/613BC27C" Ref="#PWR0105"  Part="1"
+F 0 "#PWR0105" H 3950 1850 50  0001 C CNN
 F 1 "GND" V 3955 1972 50  0000 R CNN
 F 2 "" H 3950 2100 50  0001 C CNN
@@
 P 3950 2200
 AR Path="/613BC288" Ref="#PWR?"  Part="1"
-AR Path="/613B204B/613BC288" Ref="#PWR?"  Part="1"
-F 0 "#PWR?" H 3950 1950 50  0001 C CNN
+AR Path="/613B204B/613BC288" Ref="#PWR0106"  Part="1"
+F 0 "#PWR0106" H 3950 1950 50  0001 C CNN
 F 1 "GND" V 3955 2072 50  0000 R CNN
 F 2 "" H 3950 2200 50  0001 C CNN
@@
 P 3800 2450
 AR Path="/613BC2B4" Ref="#PWR?"  Part="1"
-AR Path="/613B204B/613BC2B4" Ref="#PWR?"  Part="1"
-F 0 "#PWR?" H 3800 2300 50  0001 C CNN
+AR Path="/613B204B/613BC2B4" Ref="#PWR0107"  Part="1"
+F 0 "#PWR0107" H 3800 2300 50  0001 C CNN
 F 1 "+3.3V" H 3815 2623 50  0000 C CNN
 F 2 "" H 3800 2450 50  0001 C CNN
@@
 P 2050 1150
 AR Path="/613BC2BA" Ref="#PWR?"  Part="1"
-AR Path="/613B204B/613BC2BA" Ref="#PWR?"  Part="1"
-F 0 "#PWR?" H 2050 900 50  0001 C CNN
+AR Path="/613B204B/613BC2BA" Ref="#PWR0108"  Part="1"
+F 0 "#PWR0108" H 2050 900 50  0001 C CNN
 F 1 "GND" V 2055 1022 50  0000 R CNN
 F 2 "" H 2050 1150 50  0001 C CNN
@@
 P 2050 1250
 AR Path="/613BC2C0" Ref="#PWR?"  Part="1"
-AR Path="/613B204B/613BC2C0" Ref="#PWR?"  Part="1"
-F 0 "#PWR?" H 2050 1000 50  0001 C CNN
+AR Path="/613B204B/613BC2C0" Ref="#PWR0109"  Part="1"
+F 0 "#PWR0109" H 2050 1000 50  0001 C CNN
 F 1 "GND" V 2055 1122 50  0000 R CNN
 F 2 "" H 2050 1250 50  0001 C CNN
@@
 P 6050 1250
 AR Path="/613BC2EA" Ref="#PWR?"  Part="1"
-AR Path="/613B204B/613BC2EA" Ref="#PWR?"  Part="1"
-F 0 "#PWR?" H 6050 1000 50  0001 C CNN
+AR Path="/613B204B/613BC2EA" Ref="#PWR0110"  Part="1"
+F 0 "#PWR0110" H 6050 1000 50  0001 C CNN
 F 1 "GND" H 6055 1077 50  0000 C CNN
 F 2 "" H 6050 1250 50  0001 C CNN
@@
 P 6500 1250
 AR Path="/613BC2F0" Ref="#PWR?"  Part="1"
-AR Path="/613B204B/613BC2F0" Ref="#PWR?"  Part="1"
-F 0 "#PWR?" H 6500 1000 50  0001 C CNN
+AR Path="/613B204B/613BC2F0" Ref="#PWR0111"  Part="1"
+F 0 "#PWR0111" H 6500 1000 50  0001 C CNN
 F 1 "GND" H 6505 1077 50  0000 C CNN
 F 2 "" H 6500 1250 50  0001 C CNN
@@
 P 850 2450
 AR Path="/613BC2F9" Ref="#PWR?"  Part="1"
-AR Path="/613B204B/613BC2F9" Ref="#PWR?"  Part="1"
-F 0 "#PWR?" H 850 2200 50  0001 C CNN
+AR Path="/613B204B/613BC2F9" Ref="#PWR0112"  Part="1"
+F 0 "#PWR0112" H 850 2200 50  0001 C CNN
 F 1 "GND" H 855 2277 50  0000 C CNN
 F 2 "" H 850 2450 50  0001 C CNN
@@
 P 6100 2250
 AR Path="/613BC316" Ref="#PWR?"  Part="1"
-AR Path="/613B204B/613BC316" Ref="#PWR?"  Part="1"
-F 0 "#PWR?" H 6100 2100 50  0001 C CNN
+AR Path="/613B204B/613BC316" Ref="#PWR0113"  Part="1"
+F 0 "#PWR0113" H 6100 2100 50  0001 C CNN
 F 1 "+BATT" V 6115 2378 50  0000 L CNN
 F 2 "" H 6100 2250 50  0001 C CNN
@@
 P 6100 2550
 AR Path="/613BC31C" Ref="#PWR?"  Part="1"
-AR Path="/613B204B/613BC31C" Ref="#PWR?"  Part="1"
-F 0 "#PWR?" H 6100 2400 50  0001 C CNN
+AR Path="/613B204B/613BC31C" Ref="#PWR0114"  Part="1"
+F 0 "#PWR0114" H 6100 2400 50  0001 C CNN
 F 1 "-BATT" V 6115 2678 50  0000 L CNN
 F 2 "" H 6100 2550 50  0001 C CNN
@@
 P 6100 2550
 AR Path="/613BC322" Ref="#PWR?"  Part="1"
-AR Path="/613B204B/613BC322" Ref="#PWR?"  Part="1"
-F 0 "#PWR?" H 6100 2300 50  0001 C CNN
+AR Path="/613B204B/613BC322" Ref="#PWR0115"  Part="1"
+F 0 "#PWR0115" H 6100 2300 50  0001 C CNN
 F 1 "GND" H 6105 2377 50  0000 C CNN
 F 2 "" H 6100 2550 50  0001 C CNN
@@
 P 5850 2550
 AR Path="/613BC331" Ref="#PWR?"  Part="1"
-AR Path="/613B204B/613BC331" Ref="#PWR?"  Part="1"
-F 0 "#PWR?" H 5850 2300 50  0001 C CNN
+AR Path="/613B204B/613BC331" Ref="#PWR0116"  Part="1"
+F 0 "#PWR0116" H 5850 2300 50  0001 C CNN
 F 1 "GND" H 5855 2377 50  0000 C CNN
 F 2 "" H 5850 2550 50  0001 C CNN
@@
 P 5250 2650
 AR Path="/613BC33D" Ref="#PWR?"  Part="1"
-AR Path="/613B204B/613BC33D" Ref="#PWR?"  Part="1"
-F 0 "#PWR?" H 5250 2400 50  0001 C CNN
+AR Path="/613B204B/613BC33D" Ref="#PWR0117"  Part="1"
+F 0 "#PWR0117" H 5250 2400 50  0001 C CNN
 F 1 "GND" H 5255 2477 50  0000 C CNN
 F 2 "" H 5250 2650 50  0001 C CNN
@@
 P 5600 3250
 AR Path="/613BC35C" Ref="#PWR?"  Part="1"
-AR Path="/613B204B/613BC35C" Ref="#PWR?"  Part="1"
-F 0 "#PWR?" H 5600 3000 50  0001 C CNN
+AR Path="/613B204B/613BC35C" Ref="#PWR0118"  Part="1"
+F 0 "#PWR0118" H 5600 3000 50  0001 C CNN
 F 1 "GND" H 5605 3077 50  0000 C CNN
 F 2 "" H 5600 3250 50  0001 C CNN
@@
 P 6000 3250
 AR Path="/613BC362" Ref="#PWR?"  Part="1"
-AR Path="/613B204B/613BC362" Ref="#PWR?"  Part="1"
-F 0 "#PWR?" H 6000 3000 50  0001 C CNN
+AR Path="/613B204B/613BC362" Ref="#PWR0119"  Part="1"
+F 0 "#PWR0119" H 6000 3000 50  0001 C CNN
 F 1 "GND" H 6005 3077 50  0000 C CNN
 F 2 "" H 6000 3250 50  0001 C CNN
@@
 $EndComp
 $Comp
-L power:GND #PWR?
+L power:GND #PWR0120
 U 1 1 61411635
 P 3850 1700
-F 0 "#PWR?" H 3850 1450 50  0001 C CNN
+F 0 "#PWR0120" H 3850 1450 50  0001 C CNN
 F 1 "GND" H 3855 1527 50  0000 C CNN
 F 2 "" H 3850 1700 50  0001 C CNN
@@
 $EndComp
 $Comp
-L power:GND #PWR?
+L power:GND #PWR0121
 U 1 1 614120E2
 P 3850 1250
-F 0 "#PWR?" H 3850 1000 50  0001 C CNN
+F 0 "#PWR0121" H 3850 1000 50  0001 C CNN
 F 1 "GND" H 3855 1077 50  0000 C CNN
 F 2 "" H 3850 1250 50  0001 C CNN
@@
 $EndComp
 $Comp
-L power:GND #PWR?
+L power:GND #PWR0122
 U 1 1 6142CFD4
 P 6950 1250
-F 0 "#PWR?" H 6950 1000 50  0001 C CNN
+F 0 "#PWR0122" H 6950 1000 50  0001 C CNN
 F 1 "GND" H 6955 1077 50  0000 C CNN
 F 2 "" H 6950 1250 50  0001 C CNN
@@
 Different capacitor values for low impedance at a range of frequencies
 $Comp
-L RF_GSM:SARA-U201 U?
-U 1 1 6144695D
-P 9000 3750
-F 0 "U?" H 9000 2561 50  0000 C CNN
-F 1 "SARA-U201" H 9000 2470 50  0000 C CNN
-F 2 "RF_GSM:ublox_SARA-G3_LGA-96" H 9700 2700 50  0001 C CNN
-F 3 "https://www.u-blox.com/sites/default/files/SARA-U2_DataSheet_(UBX-13005287).pdf" H 9000 3750 50  0001 C CNN
-	1    9000 3750
-	1    0    0    -1
-$EndComp
+L Regulator_Linear:LM3480-3.3 U?
+U 1 1 6145B119
+P 8600 1750
+F 0 "U?" H 8600 1992 50  0000 C CNN
+F 1 "LM3480-3.3" H 8600 1901 50  0000 C CNN
+F 2 "Package_TO_SOT_SMD:SOT-23" H 8600 1975 50  0001 C CIN
+F 3 "http://www.ti.com/lit/ds/symlink/lm3480.pdf" H 8600 1750 50  0001 C CNN
+	1    8600 1750
+	1    0    0    -1
+$EndComp
+$Comp
+L Device:C C?
+U 1 1 6146363C
+P 8150 1900
+F 0 "C?" H 8265 1946 50  0000 L CNN
+F 1 "C" H 8265 1855 50  0000 L CNN
+F 2 "" H 8188 1750 50  0001 C CNN
+F 3 "~" H 8150 1900 50  0001 C CNN
+	1    8150 1900
+	1    0    0    -1
+$EndComp
+$Comp
+L Device:C C?
+U 1 1 614640B3
+P 9050 1900
+F 0 "C?" H 9165 1946 50  0000 L CNN
+F 1 "C" H 9165 1855 50  0000 L CNN
+F 2 "" H 9088 1750 50  0001 C CNN
+F 3 "~" H 9050 1900 50  0001 C CNN
+	1    9050 1900
+	1    0    0    -1
+$EndComp
+Wire Wire Line
+	8150 1750 8300 1750
+Wire Wire Line
+	8900 1750 9050 1750
+Text GLabel 8000 1750 0    50   Input ~ 0
+VCC
+Wire Wire Line
+	8000 1750 8150 1750
+Connection ~ 8150 1750
+$Comp
+L power:+3V3 #PWR?
+U 1 1 6146807E
+P 9250 1750
+F 0 "#PWR?" H 9250 1600 50  0001 C CNN
+F 1 "+3V3" V 9265 1878 50  0000 L CNN
+F 2 "" H 9250 1750 50  0001 C CNN
+F 3 "" H 9250 1750 50  0001 C CNN
+	1    9250 1750
+	0    1    1    0
+$EndComp
+Wire Wire Line
+	9050 1750 9250 1750
+Connection ~ 9050 1750
+$Comp
+L power:GND #PWR?
+U 1 1 6146B115
+P 8150 2050
+F 0 "#PWR?" H 8150 1800 50  0001 C CNN
+F 1 "GND" H 8155 1877 50  0000 C CNN
+F 2 "" H 8150 2050 50  0001 C CNN
+F 3 "" H 8150 2050 50  0001 C CNN
+	1    8150 2050
+	1    0    0    -1
+$EndComp
+$Comp
+L power:GND #PWR?
+U 1 1 6146BB0D
+P 9050 2050
+F 0 "#PWR?" H 9050 1800 50  0001 C CNN
+F 1 "GND" H 9055 1877 50  0000 C CNN
+F 2 "" H 9050 2050 50  0001 C CNN
+F 3 "" H 9050 2050 50  0001 C CNN
+	1    9050 2050
+	1    0    0    -1
+$EndComp
+$Comp
+L power:GND #PWR?
+U 1 1 6146F41C
+P 8600 2050
+F 0 "#PWR?" H 8600 1800 50  0001 C CNN
+F 1 "GND" H 8605 1877 50  0000 C CNN
+F 2 "" H 8600 2050 50  0001 C CNN
+F 3 "" H 8600 2050 50  0001 C CNN
+	1    8600 2050
+	1    0    0    -1
+$EndComp
+Wire Wire Line
+	3750 950  3850 950
+Connection ~ 3850 950
 $EndSCHEMATC

Commit message: Finished adding components, need to add values
Parts:
- removed C?: C, symbol Device:C
- R? (x2): value R -> 5k1; footprint (none) -> Resistor_SMD:R_0603_1608Metric_Pad0.98x0.95mm_HandSolder
- R? (x3): value R -> 10k; footprint (none) -> Resistor_SMD:R_0603_1608Metric_Pad0.98x0.95mm_HandSolder
- R? (x3): value R -> 4k7; footprint (none) -> Resistor_SMD:R_0603_1608Metric_Pad0.98x0.95mm_HandSolder
- R?: value R -> 2k2; footprint (none) -> Resistor_SMD:R_0603_1608Metric_Pad0.98x0.95mm_HandSolder
- R?: value R -> 5k23; footprint (none) -> Resistor_SMD:R_0603_1608Metric_Pad0.98x0.95mm_HandSolder
- R?: value R -> 32k; footprint (none) -> Resistor_SMD:R_0603_1608Metric_Pad0.98x0.95mm_HandSolder
- TH?: value Thermistor_NTC -> Thermistor_NTC 10K; footprint (none) -> Resistor_SMD:R_0805_2012Metric_Pad1.20x1.40mm_HandSolder
Connections:
- wire segments 46 -> 45
Other:
- moved on the sheet: C?, L?

Commit message: Update, 21st August
Parts:
- C?: value C -> 1u; footprint (none) -> Capacitor_SMD:C_0603_1608Metric_Pad1.08x0.95mm_HandSolder
- C?: value C -> 47n; footprint (none) -> Capacitor_SMD:C_0603_1608Metric_Pad1.08x0.95mm_HandSolder
- C? (x2): value C -> 22u; footprint (none) -> Capacitor_SMD:C_0603_1608Metric_Pad1.08x0.95mm_HandSolder
- C?: value C -> 10u; footprint (none) -> Capacitor_SMD:C_0603_1608Metric_Pad1.08x0.95mm_HandSolder
- C?: value C -> 4u7; footprint (none) -> Capacitor_SMD:C_0603_1608Metric_Pad1.08x0.95mm_HandSolder
- C?: value CP -> 220u; footprint (none) -> Capacitor_Tantalum_SMD:CP_EIA-3528-12_Kemet-T_Pad1.50x2.35mm_HandSolder
- C? (x2): value C -> 0u1; footprint (none) -> Capacitor_SMD:C_0603_1608Metric_Pad1.08x0.95mm_HandSolder
- L?: value L -> 2u2
Changed lines of the file:
@@
 AR Path="/613B204B/613BC23D" Ref="C?"  Part="1"
 F 0 "C?" H 3965 1146 50  0000 L CNN
-F 1 "C" H 3965 1055 50  0000 L CNN
-F 2 "" H 3888 950 50  0001 C CNN
-F 3 "test" H 3550 1100 50  0000 L CNN
+F 1 "1u" H 3965 1055 50  0000 L CNN
+F 2 "Capacitor_SMD:C_0603_1608Metric_Pad1.08x0.95mm_HandSolder" H 3888 950 50  0001 C CNN
+F 3 "https://www.mouser.co.uk/ProductDetail/Taiyo-Yuden/LMK107B7105KAHT?qs=CNQs48zzdnpelxTWRrWvpA%3D%3D" H 3550 1100 50  0001 L CNN
 	1    3850 1100
 	1    0    0    -1
@@
 AR Path="/613B204B/613BC2C6" Ref="C?"  Part="1"
 F 0 "C?" H 5365 1146 50  0000 L CNN
-F 1 "C" H 5365 1055 50  0000 L CNN
-F 2 "" H 5288 950 50  0001 C CNN
-F 3 "~" H 5250 1100 50  0001 C CNN
+F 1 "47n" H 5365 1055 50  0000 L CNN
+F 2 "Capacitor_SMD:C_0603_1608Metric_Pad1.08x0.95mm_HandSolder" H 5288 950 50  0001 C CNN
+F 3 "https://www.mouser.co.uk/ProductDetail/Samsung-Electro-Mechanics/CL10B473KO8NNNC?qs=X6jEic%2FHinAEbu%2FfpWZrPQ%3D%3D" H 5250 1100 50  0001 C CNN
 	1    5250 1100
 	1    0    0    -1
@@
 AR Path="/613B204B/613BC2D0" Ref="L?"  Part="1"
 F 0 "L?" V 5940 1300 50  0000 C CNN
-F 1 "L" V 5849 1300 50  0000 C CNN
+F 1 "2u2" V 5849 1300 50  0000 C CNN
 F 2 "" H 5750 1300 50  0001 C CNN
-F 3 "~" H 5750 1300 50  0001 C CNN
+F 3 "https://www.mouser.co.uk/ProductDetail/Bourns/SRP0312-2R2K?qs=OlC7AqGiEDm3h2uD5NkxPQ%3D%3D" H 5750 1300 50  0001 C CNN
 	1    5750 1300
 	0    -1   -1   0
@@
 AR Path="/613B204B/613BC2E0" Ref="C?"  Part="1"
 F 0 "C?" H 6365 1696 50  0000 L CNN
-F 1 "C" H 6365 1605 50  0000 L CNN
-F 2 "" H 6288 1500 50  0001 C CNN
-F 3 "~" H 6250 1650 50  0001 C CNN
+F 1 "22u" H 6365 1605 50  0000 L CNN
+F 2 "Capacitor_SMD:C_0603_1608Metric_Pad1.08x0.95mm_HandSolder" H 6288 1500 50  0001 C CNN
+F 3 "https://www.mouser.co.uk/ProductDetail/Samsung-Electro-Mechanics/CL10A226MP8NRNC?qs=xZ%2FP%252Ba9zWqbykJJ6x%252BsWhA%3D%3D" H 6250 1650 50  0001 C CNN
 	1    6250 1650
 	1    0    0    -1
@@
 AR Path="/613B204B/613BC328" Ref="C?"  Part="1"
 F 0 "C?" H 5965 2446 50  0000 L CNN
-F 1 "C" H 5965 2355 50  0000 L CNN
-F 2 "" H 5888 2250 50  0001 C CNN
-F 3 "~" H 5850 2400 50  0001 C CNN
+F 1 "10u" H 5965 2355 50  0000 L CNN
+F 2 "Capacitor_SMD:C_0603_1608Metric_Pad1.08x0.95mm_HandSolder" H 5888 2250 50  0001 C CNN
+F 3 "https://www.mouser.co.uk/ProductDetail/Taiyo-Yuden/JMK107ABJ106KA-T?qs=lkMpTOwszhd28fybYDECfg%3D%3D" H 5850 2400 50  0001 C CNN
 	1    5850 2400
 	1    0    0    -1
@@
 AR Path="/613B204B/613BC337" Ref="C?"  Part="1"
 F 0 "C?" H 5365 2546 50  0000 L CNN
-F 1 "C" H 5365 2455 50  0000 L CNN
-F 2 "" H 5288 2350 50  0001 C CNN
-F 3 "~" H 5250 2500 50  0001 C CNN
+F 1 "4u7" H 5365 2455 50  0000 L CNN
+F 2 "Capacitor_SMD:C_0603_1608Metric_Pad1.08x0.95mm_HandSolder" H 5288 2350 50  0001 C CNN
+F 3 "https://www.mouser.co.uk/ProductDetail/Samsung-Electro-Mechanics/CL10A475KQ8NNWC?qs=EvNa9vf1TdZbxyCJBSuGUg%3D%3D" H 5250 2500 50  0001 C CNN
 	1    5250 2500
 	1    0    0    -1
@@
 P 3850 1550
 F 0 "C?" H 3965 1596 50  0000 L CNN
-F 1 "C" H 3965 1505 50  0000 L CNN
-F 2 "" H 3888 1400 50  0001 C CNN
-F 3 "~" H 3850 1550 50  0001 C CNN
+F 1 "22u" H 3965 1505 50  0000 L CNN
+F 2 "Capacitor_SMD:C_0603_1608Metric_Pad1.08x0.95mm_HandSolder" H 3888 1400 50  0001 C CNN
+F 3 "https://www.mouser.co.uk/ProductDetail/Samsung-Electro-Mechanics/CL10A226MP8NRNC?qs=xZ%2FP%252Ba9zWqbykJJ6x%252BsWhA%3D%3D" H 3850 1550 50  0001 C CNN
 	1    3850 1550
 	1    0    0    -1
@@
 P 6850 1650
 F 0 "C?" H 6968 1696 50  0000 L CNN
-F 1 "CP" H 6968 1605 50  0000 L CNN
-F 2 "" H 6888 1500 50  0001 C CNN
-F 3 "~" H 6850 1650 50  0001 C CNN
+F 1 "220u" H 6968 1605 50  0000 L CNN
+F 2 "Capacitor_Tantalum_SMD:CP_EIA-3528-12_Kemet-T_Pad1.50x2.35mm_HandSolder" H 6888 1500 50  0001 C CNN
+F 3 "https://www.mouser.co.uk/ProductDetail/AVX/F930J227MBA?qs=sGAEpiMZZMtZ1n0r9vR22dQtzANU%252BEXpnQ1Vtzj%2FLbk%3D" H 6850 1650 50  0001 C CNN
 	1    6850 1650
 	1    0    0    -1
@@
 P 8150 1900
 F 0 "C?" H 8265 1946 50  0000 L CNN
-F 1 "C" H 8265 1855 50  0000 L CNN
-F 2 "" H 8188 1750 50  0001 C CNN
+F 1 "0u1" H 8265 1855 50  0000 L CNN
+F 2 "Capacitor_SMD:C_0603_1608Metric_Pad1.08x0.95mm_HandSolder" H 8188 1750 50  0001 C CNN
 F 3 "~" H 8150 1900 50  0001 C CNN
 	1    8150 1900
@@
 P 9050 1900
 F 0 "C?" H 9165 1946 50  0000 L CNN
-F 1 "C" H 9165 1855 50  0000 L CNN
-F 2 "" H 9088 1750 50  0001 C CNN
+F 1 "0u1" H 9165 1855 50  0000 L CNN
+F 2 "Capacitor_SMD:C_0603_1608Metric_Pad1.08x0.95mm_HandSolder" H 9088 1750 50  0001 C CNN
 F 3 "~" H 9050 1900 50  0001 C CNN
 	1    9050 1900

Commit message: Added footprints to most components
Parts:
- D1: renamed from D?; footprint (none) -> LED_SMD:LED_0603_1608Metric_Pad1.05x0.95mm_HandSolder
- J1: renamed from J?; footprint (none) -> Connector_USB:USB_C_Receptacle_HRO_TYPE-C-31-M-12
- L1: renamed from L?; footprint (none) -> GPS Hardware:IND_SRP0312-2R2K
- gave numbers to parts that had none: 25

Commit message: Added all footprints
Hopefully they are correct :)
Parts:
- added TP1: Battery +, TestPoint:TestPoint_Pad_4.0x4.0mm, symbol Connector:TestPoint
- added TP2: Battery -, TestPoint:TestPoint_Pad_4.0x4.0mm, symbol Connector:TestPoint
- U1, U2: footprint (none) -> GPS Hardware:IC_ESD122DMXR
- U3: footprint (none) -> GPS Hardware:QFN50P400X400X100-25N
Connections:
- net labels removed: +BATT, -BATT
Changed lines of the file:
@@
 F 0 "U3" H 4700 3250 50  0000 C CNN
 F 1 "BQ24295" H 4700 3150 50  0000 C CNN
-F 2 "" H 4750 2400 50  0001 C CNN
+F 2 "GPS Hardware:QFN50P400X400X100-25N" H 4750 2400 50  0001 C CNN
 F 3 "https://www.mouser.co.uk/ProductDetail/Texas-Instruments/BQ24295RGER?qs=igp4D3uu33JuaPeRfsSg2w%3D%3D" H 4750 2400 50  0001 C CNN
 	1    4700 2000
@@
 F 0 "U2" H 2900 2175 50  0000 C CNN
 F 1 "ESD122DMX" H 2900 2084 50  0000 C CNN
-F 2 "" H 2900 1850 50  0001 C CNN
+F 2 "GPS Hardware:IC_ESD122DMXR" H 2900 1850 50  0001 C CNN
 F 3 "https://www.mouser.co.uk/ProductDetail/Texas-Instruments/ESD122DMXR?qs=%2Fha2pyFaduihn3aKw32kKFOpmmjnpuflw4tqhxDwaDnOkPWXZway8Q%3D%3D" H 2900 1850 50  0001 C CNN
 	1    2900 1800
@@
 F 0 "U1" H 2900 1475 50  0000 C CNN
 F 1 "ESD122DMX" H 2900 1384 50  0000 C CNN
-F 2 "" H 2900 1150 50  0001 C CNN
+F 2 "GPS Hardware:IC_ESD122DMXR" H 2900 1150 50  0001 C CNN
 F 3 "https://www.mouser.co.uk/ProductDetail/Texas-Instruments/ESD122DMXR?qs=%2Fha2pyFaduihn3aKw32kKFOpmmjnpuflw4tqhxDwaDnOkPWXZway8Q%3D%3D" H 2900 1150 50  0001 C CNN
 	1    2900 1100
@@
 	5900 2000 5450 2000
 $Comp
-L power:+BATT #PWR?
-U 1 1 613BC316
-P 6100 2250
-AR Path="/613BC316" Ref="#PWR?"  Part="1"
-AR Path="/613B204B/613BC316" Ref="#PWR0113"  Part="1"
-F 0 "#PWR0113" H 6100 2100 50  0001 C CNN
-F 1 "+BATT" V 6115 2378 50  0000 L CNN
-F 2 "" H 6100 2250 50  0001 C CNN
-F 3 "" H 6100 2250 50  0001 C CNN
-	1    6100 2250
-	0    1    1    0
-$EndComp
-$Comp
-L power:-BATT #PWR?
-U 1 1 613BC31C
-P 6100 2550
-AR Path="/613BC31C" Ref="#PWR?"  Part="1"
-AR Path="/613B204B/613BC31C" Ref="#PWR0114"  Part="1"
-F 0 "#PWR0114" H 6100 2400 50  0001 C CNN
-F 1 "-BATT" V 6115 2678 50  0000 L CNN
-F 2 "" H 6100 2550 50  0001 C CNN
-F 3 "" H 6100 2550 50  0001 C CNN
-	1    6100 2550
-	0    1    1    0
-$EndComp
-$Comp
 L power:GND #PWR?
 U 1 1 613BC322
@@
 	0    -1   -1   0
 $EndComp
+$Comp
+L Connector:TestPoint TP1
+U 1 1 6123F0EC
+P 6100 2250
+F 0 "TP1" V 6054 2438 50  0000 L CNN
+F 1 "Battery +" V 6145 2438 50  0000 L CNN
+F 2 "TestPoint:TestPoint_Pad_4.0x4.0mm" H 6300 2250 50  0001 C CNN
+F 3 "~" H 6300 2250 50  0001 C CNN
+	1    6100 2250
+	0    1    1    0
+$EndComp
+$Comp
+L Connector:TestPoint TP2
+U 1 1 61240DDF
+P 6100 2550
+F 0 "TP2" V 6054 2738 50  0000 L CNN
+F 1 "Battery -" V 6145 2738 50  0000 L CNN
+F 2 "TestPoint:TestPoint_Pad_4.0x4.0mm" H 6300 2550 50  0001 C CNN
+F 3 "~" H 6300 2550 50  0001 C CNN
+	1    6100 2550
+	0    1    1    0
+$EndComp
 $EndSCHEMATC
