File: KiCad/GPS Hardware/Power.sch (KiCad schematic (older format))
At the start: 30 parts, among them J1 USB_C_Receptacle_USB2.0, U1 ESD122DMX, U2 ESD122DMX, U3 BQ24295, U4 LM3480-3.3

Commit message: Update to laptop
Parts:
- removed U2: ESD122DMX, GPS Hardware:IC_ESD122DMXR, symbol GPS~Hardware:ESD122DMX
- R1, R10, R2: footprint Resistor_SMD:R_0603_1608Metric_Pad0.98x0.95mm_HandSolder -> Resistor_SMD:R_0402_1005Metric_Pad0.72x0.64mm_HandSolder
Changed lines of the file:
@@
-$Comp
-L GPS~Hardware:ESD122DMX U?
-U 1 1 613BC231
-P 2900 1800
-AR Path="/613BC231" Ref="U?"  Part="1"
-AR Path="/613B204B/613BC231" Ref="U2"  Part="1"
-F 0 "U2" H 2900 2175 50  0000 C CNN
-F 1 "ESD122DMX" H 2900 2084 50  0000 C CNN
-F 2 "GPS Hardware:IC_ESD122DMXR" H 2900 1850 50  0001 C CNN
-F 3 "https://www.mouser.co.uk/ProductDetail/Texas-Instruments/ESD122DMXR?qs=%2Fha2pyFaduihn3aKw32kKFOpmmjnpuflw4tqhxDwaDnOkPWXZway8Q%3D%3D" H 2900 1850 50  0001 C CNN
-	1    2900 1800
-	1    0    0    -1
-$EndComp
 $Comp
 L GPS~Hardware:ESD122DMX U?
@@
 Text GLabel 1800 1500 2    50   Output ~ 0
 D-
+Text GLabel 2600 950  0    50   BiDi ~ 0
+D+
 Text GLabel 2600 1050 0    50   BiDi ~ 0
-D+
-Text GLabel 2600 1750 0    50   BiDi ~ 0
-D+
-Text GLabel 2600 950  0    50   BiDi ~ 0
-D-
-Text GLabel 2600 1650 0    50   BiDi ~ 0
 D-
 Text GLabel 4250 1800 0    50   Input ~ 0
@@
 F 3 "" H 3200 1250 50  0001 C CNN
 	1    3200 1250
-	1    0    0    -1
-$EndComp
-$Comp
-L power:GND #PWR?
-U 1 1 613BC270
-P 3200 1950
-AR Path="/613BC270" Ref="#PWR?"  Part="1"
-AR Path="/613B204B/613BC270" Ref="#PWR0104"  Part="1"
-F 0 "#PWR0104" H 3200 1700 50  0001 C CNN
-F 1 "GND" H 3205 1777 50  0000 C CNN
-F 2 "" H 3200 1950 50  0001 C CNN
-F 3 "" H 3200 1950 50  0001 C CNN
-	1    3200 1950
 	1    0    0    -1
 $EndComp
@@
 F 0 "R10" H 5670 2846 50  0000 L CNN
 F 1 "5k23" V 5600 2700 50  0000 L CNN
-F 2 "Resistor_SMD:R_0603_1608Metric_Pad0.98x0.95mm_HandSolder" V 5530 2800 50  0001 C CNN
+F 2 "Resistor_SMD:R_0402_1005Metric_Pad0.72x0.64mm_HandSolder" V 5530 2800 50  0001 C CNN
 F 3 "~" H 5600 2800 50  0001 C CNN
 	1    5600 2800
@@
 F 0 "R1" V 1800 1150 50  0000 C CNN
 F 1 "5k1" V 1900 1150 50  0000 C CNN
-F 2 "Resistor_SMD:R_0603_1608Metric_Pad0.98x0.95mm_HandSolder" V 1830 1150 50  0001 C CNN
+F 2 "Resistor_SMD:R_0402_1005Metric_Pad0.72x0.64mm_HandSolder" V 1830 1150 50  0001 C CNN
 F 3 "~" H 1900 1150 50  0001 C CNN
 	1    1900 1150
@@
 F 0 "R2" V 2000 1250 50  0000 C CNN
 F 1 "5k1" V 1900 1250 50  0000 C CNN
-F 2 "Resistor_SMD:R_0603_1608Metric_Pad0.98x0.95mm_HandSolder" V 1830 1250 50  0001 C CNN
+F 2 "Resistor_SMD:R_0402_1005Metric_Pad0.72x0.64mm_HandSolder" V 1830 1250 50  0001 C CNN
 F 3 "~" H 1900 1250 50  0001 C CNN
 	1    1900 1250

Commit message: Update (again :+1:  )
Parts:
- R3, R4, R5: footprint Resistor_SMD:R_0603_1608Metric_Pad0.98x0.95mm_HandSolder -> Resistor_SMD:R_0402_1005Metric_Pad0.72x0.64mm_HandSolder
Changed lines of the file:
@@
 F 0 "R3" H 3480 2554 50  0000 R CNN
 F 1 "4k7" V 3550 2650 50  0000 R CNN
-F 2 "Resistor_SMD:R_0603_1608Metric_Pad0.98x0.95mm_HandSolder" V 3480 2600 50  0001 C CNN
+F 2 "Resistor_SMD:R_0402_1005Metric_Pad0.72x0.64mm_HandSolder" V 3480 2600 50  0001 C CNN
 F 3 "~" H 3550 2600 50  0001 C CNN
 	1    3550 2600
@@
 F 0 "R5" H 3980 2554 50  0000 R CNN
 F 1 "4k7" V 4050 2650 50  0000 R CNN
-F 2 "Resistor_SMD:R_0603_1608Metric_Pad0.98x0.95mm_HandSolder" V 3980 2600 50  0001 C CNN
+F 2 "Resistor_SMD:R_0402_1005Metric_Pad0.72x0.64mm_HandSolder" V 3980 2600 50  0001 C CNN
 F 3 "~" H 4050 2600 50  0001 C CNN
 	1    4050 2600
@@
 F 0 "R4" H 3870 2646 50  0000 L CNN
 F 1 "4k7" V 3800 2550 50  0000 L CNN
-F 2 "Resistor_SMD:R_0603_1608Metric_Pad0.98x0.95mm_HandSolder" V 3730 2600 50  0001 C CNN
+F 2 "Resistor_SMD:R_0402_1005Metric_Pad0.72x0.64mm_HandSolder" V 3730 2600 50  0001 C CNN
 F 3 "~" H 3800 2600 50  0001 C CNN
 	1    3800 2600

Commit message: Update
Parts:
- removed TP1: Battery +, TestPoint:TestPoint_Pad_4.0x4.0mm, symbol Connector:TestPoint
- removed TP2: Battery -, TestPoint:TestPoint_Pad_4.0x4.0mm, symbol Connector:TestPoint
- added J5: B2B-XH-A(LF)(SN), JST_B2B-XH-A(LF)(SN), symbol GPS~Hardware:B2B-XH-A(LF)(SN)
- C6: footprint Capacitor_SMD:C_0603_1608Metric_Pad1.08x0.95mm_HandSolder -> Capacitor_SMD:C_0402_1005Metric_Pad0.74x0.62mm_HandSolder
Changed lines of the file:
@@
 F 0 "C6" H 6365 1696 50  0000 L CNN
 F 1 "22u" H 6365 1605 50  0000 L CNN
-F 2 "Capacitor_SMD:C_0603_1608Metric_Pad1.08x0.95mm_HandSolder" H 6288 1500 50  0001 C CNN
+F 2 "Capacitor_SMD:C_0402_1005Metric_Pad0.74x0.62mm_HandSolder" H 6288 1500 50  0001 C CNN
 F 3 "https://www.mouser.co.uk/ProductDetail/Samsung-Electro-Mechanics/CL10A226MP8NRNC?qs=xZ%2FP%252Ba9zWqbykJJ6x%252BsWhA%3D%3D" H 6250 1650 50  0001 C CNN
 	1    6250 1650
@@
 L power:GND #PWR?
 U 1 1 613BC322
-P 6100 2550
+P 6100 2350
 AR Path="/613BC322" Ref="#PWR?"  Part="1"
 AR Path="/613B204B/613BC322" Ref="#PWR0115"  Part="1"
-F 0 "#PWR0115" H 6100 2300 50  0001 C CNN
-F 1 "GND" H 6105 2377 50  0000 C CNN
-F 2 "" H 6100 2550 50  0001 C CNN
-F 3 "" H 6100 2550 50  0001 C CNN
-	1    6100 2550
+F 0 "#PWR0115" H 6100 2100 50  0001 C CNN
+F 1 "GND" H 6105 2177 50  0000 C CNN
+F 2 "" H 6100 2350 50  0001 C CNN
+F 3 "" H 6100 2350 50  0001 C CNN
+	1    6100 2350
 	1    0    0    -1
 $EndComp
@@
 $EndComp
 $Comp
-L Connector:TestPoint TP1
-U 1 1 6123F0EC
-P 6100 2250
-F 0 "TP1" V 6054 2438 50  0000 L CNN
-F 1 "Battery +" V 6145 2438 50  0000 L CNN
-F 2 "TestPoint:TestPoint_Pad_4.0x4.0mm" H 6300 2250 50  0001 C CNN
-F 3 "~" H 6300 2250 50  0001 C CNN
-	1    6100 2250
-	0    1    1    0
-$EndComp
-$Comp
-L Connector:TestPoint TP2
-U 1 1 61240DDF
-P 6100 2550
-F 0 "TP2" V 6054 2738 50  0000 L CNN
-F 1 "Battery -" V 6145 2738 50  0000 L CNN
-F 2 "TestPoint:TestPoint_Pad_4.0x4.0mm" H 6300 2550 50  0001 C CNN
-F 3 "~" H 6300 2550 50  0001 C CNN
-	1    6100 2550
-	0    1    1    0
+L GPS~Hardware:B2B-XH-A(LF)(SN) J5
+U 1 1 61376EBD
+P 6500 2250
+F 0 "J5" H 6730 2246 50  0000 L CNN
+F 1 "B2B-XH-A(LF)(SN)" H 6730 2155 50  0000 L CNN
+F 2 "JST_B2B-XH-A(LF)(SN)" H 6500 2250 50  0001 L BNN
+F 3 "" H 6500 2250 50  0001 L BNN
+F 4 "7.0 mm" H 6500 2250 50  0001 L BNN "MAXIMUM_PACKAGE_HEIGHT"
+F 5 "1.0" H 6500 2250 50  0001 L BNN "PARTREV"
+F 6 "Manufacturer Recommendations" H 6500 2250 50  0001 L BNN "STANDARD"
+F 7 "JST Sales" H 6500 2250 50  0001 L BNN "MANUFACTURER"
+	1    6500 2250
+	1    0    0    -1
 $EndComp
 $EndSCHEMATC

Commit message: Update
Parts:
- C5: footprint Capacitor_SMD:C_0603_1608Metric_Pad1.08x0.95mm_HandSolder -> Capacitor_SMD:C_0402_1005Metric_Pad0.74x0.62mm_HandSolder
Changed lines of the file:
@@
 F 0 "C5" H 5965 2446 50  0000 L CNN
 F 1 "10u" H 5965 2355 50  0000 L CNN
-F 2 "Capacitor_SMD:C_0603_1608Metric_Pad1.08x0.95mm_HandSolder" H 5888 2250 50  0001 C CNN
+F 2 "Capacitor_SMD:C_0402_1005Metric_Pad0.74x0.62mm_HandSolder" H 5888 2250 50  0001 C CNN
 F 3 "https://www.mouser.co.uk/ProductDetail/Taiyo-Yuden/JMK107ABJ106KA-T?qs=lkMpTOwszhd28fybYDECfg%3D%3D" H 5850 2400 50  0001 C CNN
 	1    5850 2400

Commit message: Updated the sim choice to a push-push type, and generated the final gerber files
Parts:
- C1, C2, C3, C4, C5, C6, C8, C9: symbol Device:C -> GPS-Hardware-rescue:C-Device
- C7: symbol Device:CP -> GPS-Hardware-rescue:CP-Device
- D1: symbol Device:LED -> GPS-Hardware-rescue:LED-Device
- J1: symbol Connector:USB_C_Receptacle_USB2.0 -> GPS-Hardware-rescue:USB_C_Receptacle_USB2.0-Connector
- L1: symbol Device:L -> GPS-Hardware-rescue:L-Device
- R1, R10, R11, R2, R3, R4, R5, R6, R7, R8, R9: symbol Device:R -> GPS-Hardware-rescue:R-Device
- TH1: symbol Device:Thermistor_NTC -> GPS-Hardware-rescue:Thermistor_NTC-Device
- U4: symbol Regulator_Linear:LM3480-3.3 -> GPS-Hardware-rescue:LM3480-3.3-Regulator_Linear
Changed lines of the file:
@@
 $EndComp
 $Comp
-L Connector:USB_C_Receptacle_USB2.0 J?
+L GPS-Hardware-rescue:USB_C_Receptacle_USB2.0-Connector J?
 U 1 1 613BC22B
 P 1150 1550
@@
 $EndComp
 $Comp
-L Device:C C?
+L GPS-Hardware-rescue:C-Device C?
 U 1 1 613BC23D
 P 3850 1100
@@
 NoConn ~ 1750 2150
 $Comp
-L power:GND #PWR?
+L GPS-Hardware-rescue:GND-power #PWR?
 U 1 1 613BC25E
 P 1150 2450
@@
 $EndComp
 $Comp
-L power:GND #PWR?
+L GPS-Hardware-rescue:GND-power #PWR?
 U 1 1 613BC264
 P 5150 3050
@@
 $EndComp
 $Comp
-L power:GND #PWR?
+L GPS-Hardware-rescue:GND-power #PWR?
 U 1 1 613BC26A
 P 3200 1250
@@
 $EndComp
 $Comp
-L Device:R R?
+L GPS-Hardware-rescue:R-Device R?
 U 1 1 613BC276
 P 4100 2100
@@
 $EndComp
 $Comp
-L power:GND #PWR?
+L GPS-Hardware-rescue:GND-power #PWR?
 U 1 1 613BC27C
 P 3950 2100
@@
 $EndComp
 $Comp
-L Device:R R?
+L GPS-Hardware-rescue:R-Device R?
 U 1 1 613BC282
 P 4100 2200
@@
 $EndComp
 $Comp
-L power:GND #PWR?
+L GPS-Hardware-rescue:GND-power #PWR?
 U 1 1 613BC288
 P 3950 2200
@@
 $EndComp
 $Comp
-L Device:R R?
+L GPS-Hardware-rescue:R-Device R?
 U 1 1 613BC290
 P 3550 2600
@@
 SDA_Power
 $Comp
-L Device:R R?
+L GPS-Hardware-rescue:R-Device R?
 U 1 1 613BC298
 P 4050 2600
@@
 	4250 3000 4050 3000
 $Comp
-L Device:R R?
+L GPS-Hardware-rescue:R-Device R?
 U 1 1 613BC2A2
 P 3800 2600
@@
 	3800 2450 3550 2450
 $Comp
-L power:+3.3V #PWR?
+L GPS-Hardware-rescue:+3.3V-power #PWR?
 U 1 1 613BC2B4
 P 3800 2450
@@
 $EndComp
 $Comp
-L power:GND #PWR?
+L GPS-Hardware-rescue:GND-power #PWR?
 U 1 1 613BC2BA
 P 2050 1150
@@
 $EndComp
 $Comp
-L power:GND #PWR?
+L GPS-Hardware-rescue:GND-power #PWR?
 U 1 1 613BC2C0
 P 2050 1250
@@
 $EndComp
 $Comp
-L Device:C C?
+L GPS-Hardware-rescue:C-Device C?
 U 1 1 613BC2C6
 P 5250 1100
@@
 $EndComp
 $Comp
-L Device:L L?
+L GPS-Hardware-rescue:L-Device L?
 U 1 1 613BC2D0
 P 5750 1300
@@
 $EndComp
 $Comp
-L Device:C C?
+L GPS-Hardware-rescue:C-Device C?
 U 1 1 613BC2E0
 P 6250 1650
@@
 $EndComp
 $Comp
-L power:GND #PWR?
+L GPS-Hardware-rescue:GND-power #PWR?
 U 1 1 613BC2F0
 P 6250 1800
@@
 SYS
 $Comp
-L power:GND #PWR?
+L GPS-Hardware-rescue:GND-power #PWR?
 U 1 1 613BC2F9
 P 850 2450
@@
 SYS
 $Comp
-L Device:LED D?
+L GPS-Hardware-rescue:LED-Device D?
 U 1 1 613BC300
 P 5700 1900
@@
 	5550 1900 5450 1900
 $Comp
-L Device:R R?
+L GPS-Hardware-rescue:R-Device R?
 U 1 1 613BC308
 P 5300 1900
@@
 	5900 2000 5450 2000
 $Comp
-L power:GND #PWR?
+L GPS-Hardware-rescue:GND-power #PWR?
 U 1 1 613BC322
 P 6100 2350
@@
 $EndComp
 $Comp
-L Device:C C?
+L GPS-Hardware-rescue:C-Device C?
 U 1 1 613BC328
 P 5850 2400
@@
 	5850 2250 5150 2250
 $Comp
-L power:GND #PWR?
+L GPS-Hardware-rescue:GND-power #PWR?
 U 1 1 613BC331
 P 5850 2550
@@
 $EndComp
 $Comp
-L Device:C C?
+L GPS-Hardware-rescue:C-Device C?
 U 1 1 613BC337
 P 5250 2500
@@
 $EndComp
 $Comp
-L power:GND #PWR?
+L GPS-Hardware-rescue:GND-power #PWR?
 U 1 1 613BC33D
 P 5250 2650
@@
 Connection ~ 5250 2350
 $Comp
-L Device:R R?
+L GPS-Hardware-rescue:R-Device R?
 U 1 1 613BC347
 P 5600 2800
@@
 $EndComp
 $Comp
-L Device:R R?
+L GPS-Hardware-rescue:R-Device R?
 U 1 1 613BC34D
 P 5600 3100
@@
 $EndComp
 $Comp
-L Device:Thermistor_NTC TH?
+L GPS-Hardware-rescue:Thermistor_NTC-Device TH?
 U 1 1 613BC353
 P 6000 3100
@@
 	5600 2950 6000 2950
 $Comp
-L power:GND #PWR?
+L GPS-Hardware-rescue:GND-power #PWR?
 U 1 1 613BC35C
 P 5600 3250
@@
 $EndComp
 $Comp
-L power:GND #PWR?
+L GPS-Hardware-rescue:GND-power #PWR?
 U 1 1 613BC362
 P 6000 3250
@@
 NoConn ~ 4250 2300
 $Comp
-L Device:C C2
+L GPS-Hardware-rescue:C-Device C2
 U 1 1 6140FB1F
 P 3850 1550
@@
 $EndComp
 $Comp
-L power:GND #PWR0120
+L GPS-Hardware-rescue:GND-power #PWR0120
 U 1 1 61411635
 P 3850 1700
@@
 $EndComp
 $Comp
-L power:GND #PWR0121
+L GPS-Hardware-rescue:GND-power #PWR0121
 U 1 1 614120E2
 P 3850 1250
@@
 	3850 1400 4250 1400
 $Comp
-L Device:CP C7
+L GPS-Hardware-rescue:CP-Device C7
 U 1 1 6142C46C
 P 6850 1650
@@
 $EndComp
 $Comp
-L power:GND #PWR0122
+L GPS-Hardware-rescue:GND-power #PWR0122
 U 1 1 6142CFD4
 P 6850 1800
@@
 Different capacitor values for low impedance at a range of frequencies
 $Comp
-L Regulator_Linear:LM3480-3.3 U4
+L GPS-Hardware-rescue:LM3480-3.3-Regulator_Linear U4
 U 1 1 6145B119
 P 8600 1750
@@
 $EndComp
 $Comp
-L Device:C C8
+L GPS-Hardware-rescue:C-Device C8
 U 1 1 6146363C
 P 8150 1900
@@
 $EndComp
 $Comp
-L Device:C C9
+L GPS-Hardware-rescue:C-Device C9
 U 1 1 614640B3
 P 9050 1900
@@
 Connection ~ 8150 1750
 $Comp
-L power:+3V3 #PWR0123
+L GPS-Hardware-rescue:+3V3-power #PWR0123
 U 1 1 6146807E
 P 9250 1750
@@
 Connection ~ 9050 1750
 $Comp
-L power:GND #PWR0124
+L GPS-Hardware-rescue:GND-power #PWR0124
 U 1 1 6146B115
 P 8150 2050
@@
 $EndComp
 $Comp
-L power:GND #PWR0125
+L GPS-Hardware-rescue:GND-power #PWR0125
 U 1 1 6146BB0D
 P 9050 2050
@@
 $EndComp
 $Comp
-L power:GND #PWR0126
+L GPS-Hardware-rescue:GND-power #PWR0126
 U 1 1 6146F41C
 P 8600 2050
@@
 Connection ~ 6850 1500
 $Comp
-L Device:R R?
+L GPS-Hardware-rescue:R-Device R?
 U 1 1 613BC252
 P 1900 1150
@@
 $EndComp
 $Comp
-L Device:R R?
+L GPS-Hardware-rescue:R-Device R?
 U 1 1 613BC258
 P 1900 1250
@@
 $EndComp
 $Comp
-L Device:R R?
+L GPS-Hardware-rescue:R-Device R?
 U 1 1 613BC310
 P 5300 2000

Commit message: Changed resistor values for LEDs
Parts:
- R8: value 2k2 -> 250
Changed lines of the file:
@@
 AR Path="/613B204B/613BC308" Ref="R8"  Part="1"
 F 0 "R8" V 5200 1900 50  0000 C CNN
-F 1 "2k2" V 5300 1900 50  0000 C CNN
+F 1 "250" V 5300 1900 50  0000 C CNN
 F 2 "Resistor_SMD:R_0402_1005Metric_Pad0.72x0.64mm_HandSolder" V 5230 1900 50  0001 C CNN
 F 3 "~" H 5300 1900 50  0001 C CNN
