File: KiCad/GPS Hardware/_autosave-Cellular and GPS.sch (KiCad schematic (older format))
At the start: 31 parts, among them J3 Conn_Coaxial, Q1 BC847, U10 ublox_SAM-M8Q, U7 74AVC2T245GU-Q100X, U8 SARA-U201, U9 NCP662SQ33T1G

Commit message: Update
Parts:
- C31: renamed from C?; footprint Capacitor_SMD:C_0603_1608Metric_Pad1.08x0.95mm_HandSolder -> Capacitor_SMD:C_0402_1005Metric_Pad0.74x0.62mm_HandSolder
- J4: renamed from J?; footprint GCT_SIM8051-6-0-14-01-X-REVD -> GPS Hardware:GCT_SIM8051-6-0-14-01-X-REVD
- gave numbers to parts that had none: 8
Changed lines of the file:
@@
 $EndComp
 $Comp
-L GPS~Hardware:SIM8051-6-0-14-01-X-REVD J?
+L GPS~Hardware:SIM8051-6-0-14-01-X-REVD J4
 U 1 1 612F619C
 P 9100 2550
-F 0 "J?" H 9200 2917 50  0000 C CNN
+F 0 "J4" H 9200 2917 50  0000 C CNN
 F 1 "SIM8051-6-0-14-01-X-REVD" H 9200 2826 50  0000 C CNN
-F 2 "GCT_SIM8051-6-0-14-01-X-REVD" H 9100 2550 50  0001 L BNN
+F 2 "GPS Hardware:GCT_SIM8051-6-0-14-01-X-REVD" H 9100 2550 50  0001 L BNN
 F 3 "" H 9100 2550 50  0001 L BNN
 F 4 "GCT" H 9100 2550 50  0001 L BNN "MANUFACTURER"
@@
 $EndComp
 $Comp
-L power:GND #PWR?
+L power:GND #PWR0114
 U 1 1 61320761
 P 8000 3050
-F 0 "#PWR?" H 8000 2800 50  0001 C CNN
+F 0 "#PWR0114" H 8000 2800 50  0001 C CNN
 F 1 "GND" H 8005 2877 50  0000 C CNN
 F 2 "" H 8000 3050 50  0001 C CNN
@@
 $EndComp
 $Comp
-L power:GND #PWR?
+L power:GND #PWR0128
 U 1 1 61320767
 P 8350 3050
-F 0 "#PWR?" H 8350 2800 50  0001 C CNN
+F 0 "#PWR0128" H 8350 2800 50  0001 C CNN
 F 1 "GND" H 8355 2877 50  0000 C CNN
 F 2 "" H 8350 3050 50  0001 C CNN
@@
 $EndComp
 $Comp
-L power:GND #PWR?
+L power:GND #PWR0129
 U 1 1 6132076D
 P 8700 3050
-F 0 "#PWR?" H 8700 2800 50  0001 C CNN
+F 0 "#PWR0129" H 8700 2800 50  0001 C CNN
 F 1 "GND" H 8705 2877 50  0000 C CNN
 F 2 "" H 8700 3050 50  0001 C CNN
@@
 $EndComp
 $Comp
-L power:GND #PWR?
+L power:GND #PWR0133
 U 1 1 61320773
 P 8000 2050
-F 0 "#PWR?" H 8000 1800 50  0001 C CNN
+F 0 "#PWR0133" H 8000 1800 50  0001 C CNN
 F 1 "GND" H 8005 1877 50  0000 C CNN
 F 2 "" H 8000 2050 50  0001 C CNN
@@
 $EndComp
 $Comp
-L power:GND #PWR?
+L power:GND #PWR0157
 U 1 1 61320779
 P 8350 2050
-F 0 "#PWR?" H 8350 1800 50  0001 C CNN
+F 0 "#PWR0157" H 8350 1800 50  0001 C CNN
 F 1 "GND" H 8355 1877 50  0000 C CNN
 F 2 "" H 8350 2050 50  0001 C CNN
@@
 $EndComp
 $Comp
-L power:GND #PWR?
+L power:GND #PWR0158
 U 1 1 6132077F
 P 8700 2050
-F 0 "#PWR?" H 8700 1800 50  0001 C CNN
+F 0 "#PWR0158" H 8700 1800 50  0001 C CNN
 F 1 "GND" H 8705 1877 50  0000 C CNN
 F 2 "" H 8700 2050 50  0001 C CNN
@@
 RST
 $Comp
-L Device:D_TVS D?
+L Device:D_TVS D3
 U 1 1 61320797
 P 8000 2900
-F 0 "D?" V 7954 2980 50  0000 L CNN
+F 0 "D3" V 7954 2980 50  0000 L CNN
 F 1 "PESD0402" V 8045 2980 50  0000 L CNN
 F 2 "Capacitor_SMD:C_0402_1005Metric_Pad0.74x0.62mm_HandSolder" H 8000 2900 50  0001 C CNN
@@
 $EndComp
 $Comp
-L Device:D_TVS D?
+L Device:D_TVS D5
 U 1 1 6132079D
 P 8700 2900
-F 0 "D?" V 8654 2980 50  0000 L CNN
+F 0 "D5" V 8654 2980 50  0000 L CNN
 F 1 "PESD0402" V 8745 2980 50  0000 L CNN
 F 2 "Capacitor_SMD:C_0402_1005Metric_Pad0.74x0.62mm_HandSolder" H 8700 2900 50  0001 C CNN
@@
 $EndComp
 $Comp
-L Device:C C?
+L Device:C C28
 U 1 1 613207A3
 P 8350 2200
-F 0 "C?" H 8465 2246 50  0000 L CNN
+F 0 "C28" H 8465 2246 50  0000 L CNN
 F 1 "47p" H 8465 2155 50  0000 L CNN
 F 2 "Capacitor_SMD:C_0402_1005Metric_Pad0.74x0.62mm_HandSolder" H 8388 2050 50  0001 C CNN
@@
 $EndComp
 $Comp
-L Device:C C?
+L Device:C C29
 U 1 1 613207A9
 P 8700 2200
-F 0 "C?" H 8815 2246 50  0000 L CNN
+F 0 "C29" H 8815 2246 50  0000 L CNN
 F 1 "47p" H 8815 2155 50  0000 L CNN
 F 2 "Capacitor_SMD:C_0402_1005Metric_Pad0.74x0.62mm_HandSolder" H 8738 2050 50  0001 C CNN
@@
 $EndComp
 $Comp
-L Device:D_TVS D?
+L Device:D_TVS D4
 U 1 1 613207AF
 P 8350 2900
-F 0 "D?" V 8304 2980 50  0000 L CNN
+F 0 "D4" V 8304 2980 50  0000 L CNN
 F 1 "PESD0402" V 8395 2980 50  0000 L CNN
 F 2 "Capacitor_SMD:C_0402_1005Metric_Pad0.74x0.62mm_HandSolder" H 8350 2900 50  0001 C CNN
@@
 $EndComp
 $Comp
-L Device:C C?
+L Device:C C27
 U 1 1 613207B5
 P 8000 2200
-F 0 "C?" H 8115 2246 50  0000 L CNN
+F 0 "C27" H 8115 2246 50  0000 L CNN
 F 1 "47p" H 8115 2155 50  0000 L CNN
 F 2 "Capacitor_SMD:C_0402_1005Metric_Pad0.74x0.62mm_HandSolder" H 8038 2050 50  0001 C CNN
@@
 VSIM
 $Comp
-L power:GND #PWR?
+L power:GND #PWR0159
 U 1 1 61330E52
 P 9900 2150
-F 0 "#PWR?" H 9900 1900 50  0001 C CNN
+F 0 "#PWR0159" H 9900 1900 50  0001 C CNN
 F 1 "GND" H 9905 1977 50  0000 C CNN
 F 2 "" H 9900 2150 50  0001 C CNN
@@
 $EndComp
 $Comp
-L power:GND #PWR?
+L power:GND #PWR0160
 U 1 1 61330E58
 P 10200 2150
-F 0 "#PWR?" H 10200 1900 50  0001 C CNN
+F 0 "#PWR0160" H 10200 1900 50  0001 C CNN
 F 1 "GND" H 10205 1977 50  0000 C CNN
 F 2 "" H 10200 2150 50  0001 C CNN
@@
 $EndComp
 $Comp
-L power:GND #PWR?
+L power:GND #PWR0161
 U 1 1 61330E5E
 P 10550 2150
-F 0 "#PWR?" H 10550 1900 50  0001 C CNN
+F 0 "#PWR0161" H 10550 1900 50  0001 C CNN
 F 1 "GND" H 10555 1977 50  0000 C CNN
 F 2 "" H 10550 2150 50  0001 C CNN
@@
 Connection ~ 9900 2450
 $Comp
-L Device:D_TVS D?
+L Device:D_TVS D6
 U 1 1 61330E66
 P 9900 2300
-F 0 "D?" V 9854 2380 50  0000 L CNN
+F 0 "D6" V 9854 2380 50  0000 L CNN
 F 1 "PESD0402" V 9945 2380 50  0000 L CNN
 F 2 "Capacitor_SMD:C_0402_1005Metric_Pad0.74x0.62mm_HandSolder" H 9900 2300 50  0001 C CNN
@@
 $EndComp
 $Comp
-L Device:C C?
+L Device:C C31
 U 1 1 61330E6C
 P 10550 2300
-F 0 "C?" H 10665 2346 50  0000 L CNN
+F 0 "C31" H 10665 2346 50  0000 L CNN
 F 1 "0u1" H 10665 2255 50  0000 L CNN
-F 2 "Capacitor_SMD:C_0603_1608Metric_Pad1.08x0.95mm_HandSolder" H 10588 2150 50  0001 C CNN
+F 2 "Capacitor_SMD:C_0402_1005Metric_Pad0.74x0.62mm_HandSolder" H 10588 2150 50  0001 C CNN
 F 3 "~" H 10550 2300 50  0001 C CNN
 	1    10550 2300
@@
 Connection ~ 10200 2450
 $Comp
-L Device:C C?
+L Device:C C30
 U 1 1 61330E75
 P 10200 2300
-F 0 "C?" H 10315 2346 50  0000 L CNN
+F 0 "C30" H 10315 2346 50  0000 L CNN
 F 1 "47p" H 10315 2255 50  0000 L CNN
 F 2 "Capacitor_SMD:C_0402_1005Metric_Pad0.74x0.62mm_HandSolder" H 10238 2150 50  0001 C CNN
@@
 $EndComp
 $Comp
-L power:GND #PWR?
+L power:GND #PWR0162
 U 1 1 61331880
 P 9600 2650
-F 0 "#PWR?" H 9600 2400 50  0001 C CNN
+F 0 "#PWR0162" H 9600 2400 50  0001 C CNN
 F 1 "GND" H 9605 2477 50  0000 C CNN
 F 2 "" H 9600 2650 50  0001 C CNN
