File: KiCad/GPS Hardware/_autosave-Cellular and GPS.sch (KiCad schematic (older format))
At the start: 30 parts, among them J3 Conn_Coaxial, J4 SIM8051-6-0-14-01-X-REVD, Q1 BC847, Q2 BC847, Q3 BSS84, U10 ublox_SAM-M8Q, U7 74AVC2T245GU-Q100X, U8 SARA-U201

Commit message: Updated the sim choice to a push-push type, and generated the final gerber files
Parts:
- removed J4: SIM8051-6-0-14-01-X-REVD, GPS Hardware:GCT_SIM8051-6-0-14-01-X-REVD, symbol GPS~Hardware:SIM8051-6-0-14-01-X-REVD
- added J5: SIM8065-6-1-14-01-A_REVA1, GCT_SIM8065-6-1-14-01-A_REVA1, symbol GPS~Hardware:SIM8065-6-1-14-01-A_REVA1
- C18, C19, C20, C21, C22, C23: symbol Device:C -> GPS-Hardware-rescue:C-Device
- C24: renamed from C25; symbol Device:C -> GPS-Hardware-rescue:C-Device
- C25: renamed from C31; symbol Device:C -> GPS-Hardware-rescue:C-Device
- C26: renamed from C27; symbol Device:C -> GPS-Hardware-rescue:C-Device
- C27: renamed from C30; symbol Device:C -> GPS-Hardware-rescue:C-Device
- C28: renamed from C29; symbol Device:C -> GPS-Hardware-rescue:C-Device
- C29: renamed from C28; symbol Device:C -> GPS-Hardware-rescue:C-Device
- D2: symbol Device:LED -> GPS-Hardware-rescue:LED-Device
- D3, D5: symbol Device:D_TVS -> GPS-Hardware-rescue:D_TVS-Device
- D4: renamed from D6; symbol Device:D_TVS -> GPS-Hardware-rescue:D_TVS-Device
- D6: renamed from D4; symbol Device:D_TVS -> GPS-Hardware-rescue:D_TVS-Device
- J4: renamed from J3; symbol Connector:Conn_Coaxial -> GPS-Hardware-rescue:Conn_Coaxial-Connector
- Q1, Q2: symbol Transistor_BJT:BC847 -> GPS-Hardware-rescue:BC847-Transistor_BJT
- Q3: symbol Transistor_FET:BSS84 -> GPS-Hardware-rescue:BSS84-Transistor_FET
- R16, R17, R18, R19, R20: symbol Device:R -> GPS-Hardware-rescue:R-Device
- U7: renamed from U8; symbol RF_GSM:SARA-U201 -> GPS-Hardware-rescue:SARA-U201-RF_GSM
- U8: renamed from U10; symbol RF_GPS:ublox_SAM-M8Q -> GPS-Hardware-rescue:ublox_SAM-M8Q-RF_GPS
- renumbered U7 to U6
Connections:
- wire segments 45 -> 50
- no-connect marks 23 -> 24
Other:
- moved on the sheet: C25, C26, C27, C28, C29, D3, D4, D5, D6
