File: KiCad/GPS Hardware/GPS Hardware.kicad_pcb (KiCad board)
At the start: 2 copper layers, 77 parts, among them J1 USB_C_Receptacle_USB2.0, J2 Conn_2Rows-07Pins, J3 Conn_Coaxial, J4 SIM7050-6-0-00-X_REVC, Q1 BC847, U1 ESD122DMX, U10 ublox_SAM-M8Q, U2 ESD122DMX, U3 BQ24295, U4 LM3480-3.3, U5 ATmega328-AU, U6 SN74AVC4T774PW, U7 74AVC2T245GU-Q100X, U8 SARA-U201, U9 NCP662SQ33T1G, Y1 Crystal_GND24

Commit message: Started pcb layout
Parts:
- J1: moved to B.Cu
- moved C21 99.9 mm to (112.4, 73.6), turned to 90 degrees
- moved C19 96.4 mm to (116.5, 73.2), turned to 90 degrees
- moved J1 89.9 mm to (106.1, 63.6)
- moved C20 86.0 mm to (113.6, 73.6), turned to 90 degrees
- moved C18 82.1 mm to (114.9, 73.6), turned to 90 degrees
- moved C7 77.1 mm to (119.0, 72.2), turned to 90 degrees
- moved R18 76.8 mm to (141.8, 106.7), turned to 180 degrees
- moved R17 48.1 mm to (142.7, 104.1), turned to 270 degrees
- moved U10 20.1 mm to (180.0, 80.0)
- moved U8 17.4 mm to (123.5, 83.2)
- moved J3 16.2 mm to (105.6, 79.9)
Other:
- board outline added: 100 x 40 mm
- copper layers 2 -> 4

Commit message: Update
Parts:
- C1, C2, C3, C4: footprint Capacitor_SMD:C_0603_1608Metric_Pad1.08x0.95mm_HandSolder -> Capacitor_SMD:C_0402_1005Metric_Pad0.74x0.62mm_HandSolder; moved to B.Cu
- C27: value 0u1 -> 47p; footprint Capacitor_SMD:C_0603_1608Metric_Pad1.08x0.95mm_HandSolder -> Capacitor_SMD:C_0402_1005Metric_Pad0.74x0.62mm_HandSolder; moved to B.Cu
- C28, C29, C30, C5, C6, C8, C9, D1, D3, D4, D5, D6, L1, R11, R16, R5, R9, TH1, TP1, TP2, U1, U2, U3, U4, U5, U6, U9: moved to B.Cu
- C31: value 47p -> 0u1; moved to B.Cu
- J2: value Conn_2Rows-07Pins -> Conn_01x06_Male; moved to B.Cu
- J4: value SIM7050-6-0-00-X_REVC -> SIM8051-6-0-14-01-X-REVD; footprint GPS Hardware:GCT_SIM7050-6-0-00-X_REVC -> GPS Hardware:GCT_SIM8051-6-0-14-01-X-REVD; moved to B.Cu
- R1, R2, R6, R7, R8: footprint Resistor_SMD:R_0603_1608Metric_Pad0.98x0.95mm_HandSolder -> Resistor_SMD:R_0402_1005Metric_Pad0.72x0.64mm_HandSolder; moved to B.Cu
- Y1: value Crystal_GND24 -> Crystal; moved to B.Cu
- moved C25 124.4 mm to (177.2, 88.8), turned to 180 degrees
- moved J2 110.9 mm to (149.5, 64.0)
- moved D5 109.9 mm to (135.4, 61.6), turned to 90 degrees
- moved C27 108.5 mm to (125.9, 75.8), turned to 270 degrees
- moved C29 104.8 mm to (134.3, 61.6), turned to 270 degrees
- moved Y1 100.5 mm to (152.4, 69.6)
- moved C31 99.2 mm to (123.4, 75.8), turned to 270 degrees
- moved R16 98.9 mm to (147.1, 86.6)
- moved R1 96.8 mm to (105.0, 71.1)
- moved U5 96.5 mm to (154.1, 83.8), turned to 270 degrees
- moved U2 95.3 mm to (108.5, 69.8), turned to 90 degrees
- moved U1 94.3 mm to (106.9, 69.8), turned to 270 degrees
- moved D2 94.1 mm to (133.6, 101.3)
- moved TP1 93.9 mm to (97.0, 68.7)
- moved R7 93.5 mm to (104.0, 77.3)
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Connections:
- C27 pad 1: VSIM -> RST
- C28 pad 1: VSIM -> CLK
- C29 pad 1: RST -> IO
- C30 pad 1: IO -> VSIM
- C31 pad 1: CLK -> VSIM
- D3 pad 1: VSIM -> GND
- D3 pad 2: GND -> RST
- D4 pad 2: RST -> CLK
- D6 pad 1: GND -> VSIM
- D6 pad 2: CLK -> GND
- J3 pad 2: (no net) -> GND
- U1 pad 1: D+ -> D-
- U1 pad 2: D- -> D+
- U2 pad 1: D+ -> D-
- U2 pad 2: D- -> D+
- Y1 pad 2: GND -> Net-(C15-Pad1)

Commit message: Update for PC
Parts:
- C10, C14, C15, C16, C17, R10, R12, R13, R14, R15, R3, R4: moved to B.Cu
- C11, C12, C13: footprint Capacitor_SMD:C_0603_1608Metric_Pad1.08x0.95mm_HandSolder -> Capacitor_SMD:C_0402_1005Metric_Pad0.74x0.62mm_HandSolder; moved to B.Cu
- C31: footprint Capacitor_SMD:C_0402_1005Metric_Pad0.74x0.62mm_HandSolder -> Capacitor_SMD:C_0603_1608Metric_Pad1.08x0.95mm_HandSolder
- R1, R2: footprint Resistor_SMD:R_0402_1005Metric_Pad0.72x0.64mm_HandSolder -> Resistor_SMD:R_0603_1608Metric_Pad0.98x0.95mm_HandSolder
- moved R14 117.4 mm to (143.7, 63.6), turned to 180 degrees
- moved R13 113.4 mm to (143.7, 65.1), turned to 180 degrees
- moved R12 109.9 mm to (155.1, 64.0)
- moved C15 105.4 mm to (148.0, 73.4), turned to 180 degrees
- moved C13 103.5 mm to (152.7, 77.8), turned to 180 degrees
- moved C14 102.5 mm to (157.1, 73.8)
- moved C12 101.0 mm to (154.9, 77.8), turned to 180 degrees
- moved C16 98.5 mm to (135.6, 78.8), turned to 180 degrees
- moved R15 96.6 mm to (147.1, 81.9)
- moved C17 96.5 mm to (146.2, 77.6), turned to 90 degrees
- moved C11 91.6 mm to (155.7, 89.7), turned to 180 degrees
- moved C10 89.3 mm to (152.9, 92.0), turned to 270 degrees
- moved R10 82.3 mm to (104.6, 87.1)
- moved R3 76.8 mm to (147.1, 83.4), turned to 180 degrees
- moved R4 70.5 mm to (147.1, 84.9)
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Other:
- net class Default: via_drill 0.4 -> 0.3
- board text added: "Designed by the great owen97779"

Commit message: Update for PC again
Parts:
- moved D1 5.97 mm to (110.4, 85.5)
- moved R9 5.94 mm to (110.3, 84.0)
- moved U1 2.03 mm to (109.2, 88.5), turned to 0 degrees
- moved R2 0.79 mm to (104.6, 89.0), turned to 270 degrees
- moved U2 0.57 mm to (106.9, 90.4), turned to 180 degrees
- moved R8 0.43 mm to (107.4, 84.5)
Routing:
- net D-: track 0.00 -> 16.1 mm, vias 0 -> 2
- net D+: track 0.00 -> 14.2 mm, vias 0 -> 3
Other:
- rule via_min_drill: 0.3 -> 0.2
Changed lines of the file:
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@@
     (thickness 1.6)
     (drawings 7)
-    (tracks 0)
+    (tracks 36)
     (zones 0)
     (modules 77)
@@
     (via_drill 0.3)
     (via_min_size 0.4)
-    (via_min_drill 0.3)
-    (user_via 0.45 0.3)
+    (via_min_drill 0.2)
+    (user_via 0.45 0.2)
     (uvia_size 0.2)
     (uvia_drill 0.1)
@@
     (pad_to_mask_clearance 0)
     (aux_axis_origin 0 0)
-    (visible_elements 7FFFFFDF)
+    (visible_elements 7FFF7FDF)
     (pcbplotparams
       (layerselection 0x010fc_ffffffff)
@@
   )
   (module Resistor_SMD:R_0603_1608Metric_Pad0.98x0.95mm_HandSolder (layer B.Cu)
-    (at 105.4025 88.97)
+    (at 104.6175 88.99 270)
     (descr "Resistor SMD 0603 (1608 Metric), square (rectangular) end terminal, IPC_7351 nominal with elongated pad for handsoldering. (Body size source: IPC-SM-782 page 72, https://www.pcb-3d.com/wordpress/wp-content/uploads/ipc-sm-782a_amendment_1_and_2.pdf), generated with kicad-footprint-generator")
     (tags "resistor handsolder")
     (attr smd)
-    (fp_text reference R2 (at 0 1.43) (layer B.SilkS)
+    (fp_text reference R2 (at 0 1.43 90) (layer B.SilkS)
       (effects (font (size 1 1) (thickness 0.15)) (justify mirror))
     )
-    (fp_text value 5k1 (at 0 -1.43) (layer B.Fab)
+    (fp_text value 5k1 (at 0 -1.43 90) (layer B.Fab)
       (effects (font (size 1 1) (thickness 0.15)) (justify mirror))
     )
-    (fp_text user %R (at 0 0) (layer B.Fab)
+    (fp_text user %R (at 0 0 90) (layer B.Fab)
       (effects (font (size 0.4 0.4) (thickness 0.06)) (justify mirror))
     )
@@
     (fp_line (start 1.65 0.73) (end 1.65 -0.73) (layer B.CrtYd) (width 0.05))
     (fp_line (start 1.65 -0.73) (end -1.65 -0.73) (layer B.CrtYd) (width 0.05))
-    (pad 2 smd roundrect (at 0.9125 0) (size 0.975 0.95) (layers B.Cu B.Paste B.Mask) (roundrect_rratio 0.25)
+    (pad 2 smd roundrect (at 0.9125 0 270) (size 0.975 0.95) (layers B.Cu B.Paste B.Mask) (roundrect_rratio 0.25)
       (net 27 "Net-(J1-PadB5)"))
-    (pad 1 smd roundrect (at -0.9125 0) (size 0.975 0.95) (layers B.Cu B.Paste B.Mask) (roundrect_rratio 0.25)
+    (pad 1 smd roundrect (at -0.9125 0 270) (size 0.975 0.95) (layers B.Cu B.Paste B.Mask) (roundrect_rratio 0.25)
       (net 1 GND))
     (model ${KISYS3DMOD}/Resistor_SMD.3dshapes/R_0603_1608Metric.wrl
@@
   )
   (module Resistor_SMD:R_0402_1005Metric_Pad0.72x0.64mm_HandSolder (layer B.Cu)
-    (at 107.55 84.8675 90)
+    (at 107.36 84.4775 90)
     (descr "Resistor SMD 0402 (1005 Metric), square (rectangular) end terminal, IPC_7351 nominal with elongated pad for handsoldering. (Body size source: IPC-SM-782 page 72, https://www.pcb-3d.com/wordpress/wp-content/uploads/ipc-sm-782a_amendment_1_and_2.pdf), generated with kicad-footprint-generator")
     (tags "resistor handsolder")
@@
   )
   (module "GPS Hardware:IC_ESD122DMXR" (layer B.Cu)
-    (at 109 90.5 90)
-    (fp_text reference U1 (at 0.062 0.9524 270) (layer B.SilkS)
+    (at 109.22 88.48)
+    (fp_text reference U1 (at 0.062 0.9524 180) (layer B.SilkS)
       (effects (font (size 0.24 0.24) (thickness 0.15)) (justify mirror))
     )
-    (fp_text value ESD122DMX (at 1.2812 -0.9476 270) (layer B.Fab)
+    (fp_text value ESD122DMX (at 1.2812 -0.9476 180) (layer B.Fab)
       (effects (font (size 0.24 0.24) (thickness 0.15)) (justify mirror))
     )
@@
       (xy 0.001093 0.450396) (xy 0.000616 0.447822) (xy 0.000274 0.445226) (xy 0.000069 0.442617)
       (xy 0 0.44)) (layer B.Mask) (width 0.01))
-    (pad 3 smd rect (at 0.15 0.34 90) (size 0.2 0.2) (layers B.Cu)
+    (pad 3 smd rect (at 0.15 0.34) (size 0.2 0.2) (layers B.Cu)
       (net 1 GND))
-    (pad 2 smd rect (at 0.15 -0.34 90) (size 0.2 0.2) (layers B.Cu)
+    (pad 2 smd rect (at 0.15 -0.34) (size 0.2 0.2) (layers B.Cu)
       (net 25 D+))
-    (pad 1 smd rect (at -0.15 0 90) (size 0.2 0.2) (layers B.Cu)
+    (pad 1 smd rect (at -0.15 0) (size 0.2 0.2) (layers B.Cu)
       (net 24 D-))
   )
   (module "GPS Hardware:IC_ESD122DMXR" (layer B.Cu)
-    (at 107.436 90.5 270)
-    (fp_text reference U2 (at 0.062 0.9524 270) (layer B.SilkS)
+    (at 106.88 90.36 180)
+    (fp_text reference U2 (at 0.062 0.9524 180) (layer B.SilkS)
       (effects (font (size 0.24 0.24) (thickness 0.15)) (justify mirror))
     )
-    (fp_text value ESD122DMX (at 1.2812 -0.9476 270) (layer B.Fab)
+    (fp_text value ESD122DMX (at 1.2812 -0.9476 180) (layer B.Fab)
       (effects (font (size 0.24 0.24) (thickness 0.15)) (justify mirror))
     )
@@
       (xy 0.001093 0.450396) (xy 0.000616 0.447822) (xy 0.000274 0.445226) (xy 0.000069 0.442617)
       (xy 0 0.44)) (layer B.Mask) (width 0.01))
-    (pad 3 smd rect (at 0.15 0.34 270) (size 0.2 0.2) (layers B.Cu)
+    (pad 3 smd rect (at 0.15 0.34 180) (size 0.2 0.2) (layers B.Cu)
       (net 1 GND))
-    (pad 2 smd rect (at 0.15 -0.34 270) (size 0.2 0.2) (layers B.Cu)
+    (pad 2 smd rect (at 0.15 -0.34 180) (size 0.2 0.2) (layers B.Cu)
       (net 25 D+))
-    (pad 1 smd rect (at -0.15 0 270) (size 0.2 0.2) (layers B.Cu)
+    (pad 1 smd rect (at -0.15 0 180) (size 0.2 0.2) (layers B.Cu)
       (net 24 D-))
   )
@@
   )
   (module Resistor_SMD:R_0603_1608Metric_Pad0.98x0.95mm_HandSolder (layer B.Cu)
-    (at 116.0855 85.39)
+    (at 110.2975 84.04)
     (descr "Resistor SMD 0603 (1608 Metric), square (rectangular) end terminal, IPC_7351 nominal with elongated pad for handsoldering. (Body size source: IPC-SM-782 page 72, https://www.pcb-3d.com/wordpress/wp-content/uploads/ipc-sm-782a_amendment_1_and_2.pdf), generated with kicad-footprint-generator")
     (tags "resistor handsolder")
@@
   )
   (module LED_SMD:LED_0603_1608Metric_Pad1.05x0.95mm_HandSolder (layer B.Cu)
-    (at 116.123 87.168)
+    (at 110.39 85.5)
     (descr "LED SMD 0603 (1608 Metric), square (rectangular) end terminal, IPC_7351 nominal, (Body size source: http://www.tortai-tech.com/upload/download/2011102023233369053.pdf), generated with kicad-footprint-generator")
     (tags "LED handsolder")
@@
   (gr_line (start 100 100) (end 200 100) (layer Edge.Cuts) (width 0.15))
   (gr_line (start 100 100) (end 100 60) (layer Edge.Cuts) (width 0.15))
+  (via (at 108.49 83.08) (size 0.45) (drill 0.2) (layers F.Cu B.Cu) (net 25))
+  (segment (start 109.090001 90.104001) (end 109.090001 89.400001) (width 0.25) (layer B.Cu) (net 24))
+  (segment (start 109.026 90.168002) (end 109.090001 90.104001) (width 0.25) (layer B.Cu) (net 24))
+  (segment (start 109.026 92.375) (end 109.026 90.168002) (width 0.25) (layer B.Cu) (net 24))
+  (via (at 107.86 88.21) (size 0.45) (drill 0.2) (layers F.Cu B.Cu) (net 24))
+  (segment (start 109.050001 89.400001) (end 107.86 88.21) (width 0.25) (layer B.Cu) (net 24))
+  (segment (start 109.090001 89.400001) (end 109.050001 89.400001) (width 0.25) (layer B.Cu) (net 24))
+  (segment (start 107.86 89.974002) (end 107.86 88.21) (width 0.25) (layer B.Cu) (net 24))
+  (segment (start 108.050001 90.164003) (end 107.86 89.974002) (width 0.25) (layer B.Cu) (net 24))
+  (segment (start 108.050001 91.861999) (end 108.050001 90.164003) (width 0.25) (layer B.Cu) (net 24))
+  (segment (start 108.026 91.886) (end 108.050001 91.861999) (width 0.25) (layer B.Cu) (net 24))
+  (segment (start 108.026 92.375) (end 108.026 91.886) (width 0.25) (layer B.Cu) (net 24))
+  (segment (start 107.86 83.16) (end 107.86 83.16) (width 0.25) (layer In1.Cu) (net 24))
+  (via (at 107.86 83.08) (size 0.45) (drill 0.2) (layers F.Cu B.Cu) (net 24))
+  (segment (start 107.86 88.21) (end 107.86 83.08) (width 0.25) (layer In1.Cu) (net 24))
+  (segment (start 107.949 82.672802) (end 107.949 82.07) (width 0.25) (layer B.Cu) (net 24))
+  (segment (start 107.86 82.761802) (end 107.949 82.672802) (width 0.25) (layer B.Cu) (net 24))
+  (segment (start 107.86 83.08) (end 107.86 82.761802) (width 0.25) (layer B.Cu) (net 24))
+  (segment (start 107.155001 90.124999) (end 107.155001 90.339999) (width 0.25) (layer B.Cu) (net 24))
+  (segment (start 107.305998 89.974002) (end 107.155001 90.124999) (width 0.25) (layer B.Cu) (net 24))
+  (segment (start 107.86 89.974002) (end 107.305998 89.974002) (width 0.25) (layer B.Cu) (net 24))
+  (via (at 107.5 90.81) (size 0.45) (drill 0.2) (layers F.Cu B.Cu) (net 25))
+  (segment (start 107.526 90.836) (end 107.5 90.81) (width 0.25) (layer B.Cu) (net 25))
+  (segment (start 107.526 92.375) (end 107.526 90.836) (width 0.25) (layer B.Cu) (net 25))
+  (segment (start 107.6 90.81) (end 108.57 89.84) (width 0.25) (layer In1.Cu) (net 25))
+  (segment (start 107.5 90.81) (end 107.6 90.81) (width 0.25) (layer In1.Cu) (net 25))
+  (segment (start 108.526 89.884) (end 108.57 89.84) (width 0.25) (layer B.Cu) (net 25))
+  (segment (start 108.526 92.375) (end 108.526 89.884) (width 0.25) (layer B.Cu) (net 25))
+  (segment (start 108.449 82.720802) (end 108.449 82.07) (width 0.25) (layer B.Cu) (net 25))
+  (segment (start 108.49 82.761802) (end 108.449 82.720802) (width 0.25) (layer B.Cu) (net 25))
+  (segment (start 108.49 83.08) (end 108.49 82.761802) (width 0.25) (layer B.Cu) (net 25))
+  (via (at 108.54 89.84) (size 0.45) (drill 0.2) (layers F.Cu B.Cu) (net 25))
+  (segment (start 108.54 83.13) (end 108.49 83.08) (width 0.25) (layer In1.Cu) (net 25))
+  (segment (start 108.54 89.84) (end 108.54 83.13) (width 0.25) (layer In1.Cu) (net 25))
+  (segment (start 106.754999 90.81) (end 106.73 90.785001) (width 0.25) (layer B.Cu) (net 25))
+  (segment (start 107.5 90.81) (end 106.754999 90.81) (width 0.25) (layer B.Cu) (net 25))
 )

Commit message: Update to laptop
Parts:
- removed U2: ESD122DMX, GPS Hardware:IC_ESD122DMXR
- R1, R10, R2: footprint Resistor_SMD:R_0603_1608Metric_Pad0.98x0.95mm_HandSolder -> Resistor_SMD:R_0402_1005Metric_Pad0.72x0.64mm_HandSolder
- moved R10 11.3 mm to (113.7, 80.4)
- moved TH1 10.3 mm to (103.2, 78.2), turned to 180 degrees
- moved R11 5.24 mm to (114.3, 82.6), turned to 270 degrees
- moved R9 2.86 mm to (110.5, 86.9)
- moved R2 2.27 mm to (106.7, 90.0)
- moved U1 1.87 mm to (108.2, 90.0), turned to 180 degrees
- moved R1 1.76 mm to (109.5, 90.0), turned to 270 degrees
- moved R6 0.80 mm to (103.3, 80.7)
- moved C2 0.62 mm to (110.9, 81.8), turned to 270 degrees
- moved C4 0.54 mm to (112.0, 81.0), turned to 270 degrees
- moved R7 0.41 mm to (103.9, 79.7)
- moved D1 0.17 mm to (110.5, 85.4)
- moved R8 0.10 mm to (107.5, 84.5)
Connections:
- U1 pad 1: D- -> D+
- U1 pad 2: D+ -> D-
Routing:
- net Net-(R9-Pad1): track 0.00 -> 9.96 mm, vias 0 -> 2
- net VBUS: track 0.00 -> 6.12 mm, vias 0 -> 5
- net Net-(C4-Pad1): track 0.00 -> 3.49 mm
- net Net-(R10-Pad2): track 0.00 -> 3.41 mm
- net Net-(D1-Pad1): track 0.00 -> 2.28 mm
- net Net-(R6-Pad1): track 0.00 -> 2.04 mm
- net Net-(R8-Pad2): track 0.00 -> 1.96 mm
- net Net-(J1-PadA5): track 0.00 -> 1.83 mm
- net Net-(J1-PadB5): track 0.00 -> 1.83 mm
- net Net-(R7-Pad2): track 0.00 -> 1.32 mm
- net D+: track 14.2 -> 15.3 mm, vias 3 -> 4
- net (no net): vias 0 -> 2
- added copper zone on In2.Cu, net VBUS
Other:
- rule trace_min: 0.2 -> 0.15

Commit message: Update to laptop
Parts:
- moved R9 2.93 mm to (113.4, 86.9)
- moved D1 2.90 mm to (113.4, 85.4)
- moved R6 0.68 mm to (103.9, 80.7)
- moved R8 0.36 mm to (107.2, 84.8)
- moved C1 0.33 mm to (110.2, 83.3)
- moved R1 0.20 mm to (109.2, 90.0)
- moved C2 0.11 mm to (110.8, 81.7)
Routing:
- net Net-(R9-Pad1): track 9.96 -> 0.00 mm, vias 2 -> 0
- net VBUS: track 6.12 -> 0.06 mm, vias 5 -> 0
- net Net-(D1-Pad1): track 2.28 -> 0.00 mm
- net Net-(C2-Pad1): track 0.00 -> 1.31 mm
- net D+: track 15.3 -> 14.4 mm, vias 4 -> 2
- net Net-(R6-Pad1): track 2.04 -> 1.36 mm
- net Net-(J1-PadA5): track 1.83 -> 2.43 mm
- net D-: track 16.1 -> 15.7 mm, vias 2 -> 0
- added copper zone on B.Cu, net Net-(C3-Pad2)
- added copper zone on B.Cu, net VBUS
- removed copper zone on In2.Cu, net VBUS

Commit message: Update once again
Parts:
- moved TH1 8.52 mm to (103.7, 69.7), turned to 90 degrees
- moved C10 7.57 mm to (160.4, 93.2)
- moved C13 7.57 mm to (160.2, 79.0)
- moved C12 7.57 mm to (162.4, 79.0)
- moved C14 7.57 mm to (164.6, 75.0)
- moved C22 7.57 mm to (162.2, 93.2)
- moved R16 7.57 mm to (154.5, 87.8)
- moved R5 7.57 mm to (168.6, 82.2)
- moved U5 7.57 mm to (161.6, 85.0)
- moved U6 7.57 mm to (148.9, 81.7)
- moved C11 7.57 mm to (163.2, 90.9)
- moved C15 7.57 mm to (155.5, 74.6)
- moved C23 7.57 mm to (168.3, 94.1)
- moved R15 7.57 mm to (154.6, 83.1)
- moved R3 7.57 mm to (154.6, 84.6)
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Connections:
- U6 pad 11: RTS_Cellular -> RX_Cellular
- U6 pad 12: CTS_Cellular -> TX_Cellular
- U6 pad 13: RX_Cellular -> CTS_Cellular
- U6 pad 14: TX_Cellular -> RTS_Cellular
- U6 pad 3: RX -> CTS
- U6 pad 4: TX -> RTS
- U6 pad 5: RTS -> RX
- U6 pad 6: CTS -> TX
- U6 pad 7: +3V3 -> GND
- U6 pad 8: GND -> +3V3
Routing:
- net Net-(R10-Pad2): track 3.57 -> 31.6 mm, vias 0 -> 2
- net RTS_Cellular: track 0.00 -> 27.2 mm, vias 0 -> 1
- net CTS_Cellular: track 0.00 -> 25.9 mm, vias 0 -> 1
- net TX_Cellular: track 0.00 -> 24.5 mm, vias 0 -> 1
- net Net-(R9-Pad1): track 0.00 -> 23.8 mm, vias 0 -> 2
- net RX_Cellular: track 0.00 -> 23.3 mm, vias 0 -> 1
- net IO: track 0.00 -> 21.8 mm, vias 0 -> 1
- net Net-(D1-Pad1): track 0.00 -> 12.7 mm, vias 0 -> 2
- net CLK: track 0.00 -> 6.88 mm, vias 0 -> 1
- net RST: track 0.00 -> 6.65 mm, vias 0 -> 1
- net VSIM: track 0.00 -> 1.88 mm, vias 0 -> 1
- net SYS: vias 0 -> 8
- added copper zone on B.Cu, net SYS
- added copper zone on F.Cu, net SYS
- added copper zone on B.Cu, net VSIM

Commit message: Update (again :+1:  )
Parts:
- C16, C17: footprint Capacitor_SMD:C_0603_1608Metric_Pad1.08x0.95mm_HandSolder -> Capacitor_SMD:C_0402_1005Metric_Pad0.74x0.62mm_HandSolder
- R15, R16, R3, R4, R5: footprint Resistor_SMD:R_0603_1608Metric_Pad0.98x0.95mm_HandSolder -> Resistor_SMD:R_0402_1005Metric_Pad0.72x0.64mm_HandSolder
- moved R5 40.2 mm to (128.5, 78.9), turned to 90 degrees
- moved R14 28.7 mm to (142.1, 92.0), turned to 270 degrees
- moved C17 27.9 mm to (120.5, 88.0), turned to 270 degrees
- moved R3 27.7 mm to (127.5, 79.0), turned to 90 degrees
- moved C12 27.5 mm to (134.9, 80.5)
- moved C13 27.5 mm to (132.8, 80.5)
- moved C11 27.4 mm to (135.8, 92.1)
- moved U5 27.4 mm to (134.2, 86.3)
- moved R13 27.0 mm to (143.6, 92.0), turned to 270 degrees
- moved R15 27.0 mm to (127.8, 86.0)
- moved R4 26.8 mm to (127.8, 87.6)
- moved R16 26.8 mm to (127.8, 89.1)
- moved U6 25.4 mm to (123.8, 85.2), turned to 270 degrees
- moved C16 24.5 mm to (120.7, 89.7)
- moved J2 24.4 mm to (142.5, 86.2), turned to 90 degrees
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Routing:
- net RTS_Cellular: track 27.2 -> 1.69 mm
- net CTS_Cellular: track 25.9 -> 1.50 mm
- net TX_Cellular: track 24.5 -> 1.59 mm
- net RX_Cellular: track 23.3 -> 1.95 mm
- net CTS: track 0.00 -> 8.42 mm, vias 0 -> 2
- net RTS: track 0.00 -> 7.36 mm, vias 0 -> 2
- net RX: track 0.00 -> 7.01 mm, vias 0 -> 2
- net TX: track 0.00 -> 5.82 mm, vias 0 -> 2
- net SDA_Power: track 0.00 -> 1.00 mm, vias 0 -> 1
- net SCL_Power: track 0.00 -> 0.89 mm, vias 0 -> 1
- net Net-(J1-PadB5): track 1.83 -> 2.40 mm
- net INT_Power: track 0.00 -> 0.56 mm, vias 0 -> 1
- net +1V8: vias 0 -> 1
- removed copper zone on B.Cu, net SYS
- removed copper zone on F.Cu, net SYS
