File: KiCad/GPS Hardware/GPS Hardware.kicad_pcb (KiCad board)
At the start: 4 copper layers, 50 x 50 mm, 76 parts, among them J1 USB_C_Receptacle_USB2.0, J2 Conn_01x06_Male, J3 Conn_Coaxial, J4 SIM8051-6-0-14-01-X-REVD, Q1 BC847, U1 ESD122DMX, U10 ublox_SAM-M8Q, U3 BQ24295, U4 LM3480-3.3, U5 ATmega328-AU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

Commit message: Update to laptop
Yay
Parts:
- moved TH1 16.9 mm to (117.0, 66.7), turned to 90 degrees
- moved C19 3.34 mm to (104.2, 81.9), turned to 180 degrees
- moved C5 2.11 mm to (103.5, 76.8)
- moved R18 1.64 mm to (129.0, 101.5)
- moved C20 1.56 mm to (107.7, 80.4)
- moved C21 1.50 mm to (106.6, 80.4)
- moved R17 1.46 mm to (125.6, 101.5)
- moved C18 0.77 mm to (110.8, 81.0), turned to 0 degrees
- moved R19 0.30 mm to (130.4, 99.6)
- moved D2 0.20 mm to (127.3, 99.6)
- moved Q1 0.19 mm to (123.6, 99.5)
- turned R16 to 90 degrees
- turned U10 to 90 degrees
Routing:
- net CTS: track 0.00 -> 49.1 mm
- net RTS: track 0.00 -> 45.1 mm
- net TX: track 0.00 -> 41.2 mm
- net RX: track 0.00 -> 40.9 mm
- net RESET_Cellular: track 0.00 -> 32.2 mm
- net Net-(C15-Pad1): track 0.00 -> 17.0 mm
- net +1V8: track 0.00 -> 8.47 mm
- net Net-(C14-Pad2): track 0.00 -> 7.17 mm
- net RX_Cellular: track 0.00 -> 3.95 mm
- net TX_Cellular: track 0.00 -> 3.76 mm
- net CTS_Cellular: track 0.00 -> 3.58 mm
- net RTS_Cellular: track 0.00 -> 3.39 mm
- net Net-(R14-Pad2): track 0.00 -> 3.31 mm
- net SCK: track 0.00 -> 3.08 mm
- net MISO: track 0.00 -> 3.04 mm
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- added copper zone on F.Cu, net Net-(C3-Pad2)
- added copper zone on F.Cu, net Net-(C5-Pad1)

Commit message: Update
Parts:
- removed TP1: Battery +, TestPoint:TestPoint_Pad_4.0x4.0mm
- removed TP2: Battery -, TestPoint:TestPoint_Pad_4.0x4.0mm
- added J5: B2B-XH-A(LF)(SN), GPS Hardware:JST_B2B-XH-A(LF)(SN), B.Cu at (103.5, 77.2)
- C6: footprint Capacitor_SMD:C_0603_1608Metric_Pad1.08x0.95mm_HandSolder -> Capacitor_SMD:C_0402_1005Metric_Pad0.74x0.62mm_HandSolder
- moved TH1 14.0 mm to (103.9, 71.7), turned to 180 degrees
- moved C4 6.23 mm to (113.1, 73.3)
- moved R19 5.60 mm to (136.0, 99.6)
- moved Q1 5.58 mm to (129.2, 99.6)
- moved D2 5.43 mm to (132.7, 99.6)
- moved D1 4.30 mm to (116.8, 71.4)
- moved R9 4.08 mm to (113.0, 69.3)
- moved R10 3.21 mm to (112.5, 71.7), turned to 90 degrees
- moved R8 3.05 mm to (114.2, 71.5)
- moved R17 2.96 mm to (125.6, 98.5)
- moved R18 2.43 mm to (126.6, 101.0), turned to 270 degrees
- moved C18 2.24 mm to (108.7, 80.4), turned to 90 degrees
- moved C5 1.51 mm to (105.0, 76.4)
- moved C6 1.17 mm to (109.0, 76.7)
- moved C1 1.13 mm to (110.9, 70.4)
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Routing:
- net SCL_Power: track 1.75 -> 82.1 mm, vias 0 -> 2
- net SDA_Power: track 1.84 -> 79.5 mm, vias 0 -> 2
- net INT_Power: track 0.00 -> 63.2 mm, vias 0 -> 2
- net RESET: track 1.72 -> 48.2 mm, vias 0 -> 2
- net RESET_Cellular: track 32.2 -> 0.00 mm
- net RX: track 40.9 -> 50.2 mm
- net Net-(R9-Pad1): track 0.00 -> 9.28 mm, vias 0 -> 2
- net TX: track 41.2 -> 50.3 mm
- net RTS: track 45.1 -> 51.7 mm
- net CTS: track 49.1 -> 54.8 mm
- net Net-(C4-Pad1): track 0.00 -> 3.28 mm
- net Net-(C3-Pad1): track 0.00 -> 1.27 mm
- net Net-(R6-Pad1): track 1.58 -> 2.53 mm
- net Net-(R7-Pad2): track 1.66 -> 2.60 mm
- net Net-(R10-Pad2): track 0.00 -> 0.93 mm, vias 0 -> 2
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
Commit message: Test
Commit
Parts:
- moved C10 5.76 mm to (159.7, 98.9)
Changed lines of the file:
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@@
   )
   (module Capacitor_SMD:C_0603_1608Metric_Pad1.08x0.95mm_HandSolder (layer F.Cu)
-    (at 160.425 93.2125 90)
+    (at 159.67 98.9225 90)
     (descr "Capacitor SMD 0603 (1608 Metric), square (rectangular) end terminal, IPC_7351 nominal with elongated pad for handsoldering. (Body size source: IPC-SM-782 page 76, https://www.pcb-3d.com/wordpress/wp-content/uploads/ipc-sm-782a_amendment_1_and_2.pdf), generated with kicad-footprint-generator")
     (tags "capacitor handsolder")

Commit message: Update for today
Just added a couple sim power lines to see how it will affect the 3v3 plane
Parts:
- moved C9 8.71 mm to (129.3, 78.6), turned to 0 degrees
- moved C8 8.57 mm to (123.4, 79.6)
- moved U4 8.57 mm to (125.9, 79.7)
- turned U10 to 0 degrees
Routing:
- net VSIM: track 0.00 -> 26.1 mm, vias 0 -> 2
- net RST: track 0.00 -> 16.1 mm, vias 0 -> 2
- net CLK: track 0.00 -> 0.64 mm, vias 0 -> 1
- net IO: track 0.00 -> 0.37 mm, vias 0 -> 1

Commit message: Update
Parts:
- C19, C5: footprint Capacitor_SMD:C_0603_1608Metric_Pad1.08x0.95mm_HandSolder -> Capacitor_SMD:C_0402_1005Metric_Pad0.74x0.62mm_HandSolder
- J5: moved to F.Cu
- U1: moved to B.Cu
- moved C29 6.50 mm to (134.1, 73.9)
- moved D5 6.48 mm to (135.1, 73.9)
- moved C19 6.26 mm to (110.3, 80.4), turned to 90 degrees
- moved C8 3.94 mm to (119.5, 79.7)
- moved U4 3.94 mm to (122.0, 79.8)
- moved C9 3.94 mm to (125.3, 78.7)
- moved U1 3.85 mm to (107.9, 65.5)
- moved C7 2.40 mm to (114.7, 79.8), turned to 0 degrees
- moved J5 1.78 mm to (102.7, 78.8)
- moved L1 1.72 mm to (113.8, 76.0), turned to 270 degrees
- moved C5 1.44 mm to (106.3, 77.0)
- moved C18 0.66 mm to (109.3, 80.4)
- moved C20 0.66 mm to (108.3, 80.4)
- moved C21 0.66 mm to (107.3, 80.4)
- moved R2 0.63 mm to (105.1, 69.0)
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Routing:
- net CLK: track 0.64 -> 41.6 mm, vias 1 -> 2
- net IO: track 0.37 -> 22.3 mm, vias 1 -> 2
- net RST: track 16.1 -> 26.0 mm
- net INT_Power: track 63.2 -> 55.6 mm
- net Net-(R9-Pad1): track 9.28 -> 4.87 mm
- net Net-(J1-PadB5): track 1.78 -> 0.00 mm
- net SDA_Power: track 79.5 -> 80.5 mm
- net Net-(R8-Pad2): track 0.00 -> 0.13 mm, vias 0 -> 1

Commit message: Update
Parts:
- U1: moved to F.Cu
- moved U1 3.83 mm to (108.3, 69.3)
Routing:
- net INT_Power: track 55.6 -> 62.0 mm
- net Net-(R8-Pad2): track 0.13 -> 1.81 mm
- net D-: track 4.89 -> 5.93 mm
- net SCL_Power: track 82.5 -> 83.1 mm
- net GND: track 0.00 -> 0.42 mm, vias 1 -> 2

Commit message: Update to laptop
Parts:
- R11: footprint Resistor_SMD:R_0603_1608Metric_Pad0.98x0.95mm_HandSolder -> Resistor_SMD:R_0402_1005Metric_Pad0.72x0.64mm_HandSolder
- moved U7 30.6 mm to (134.3, 93.2)
- moved R11 12.2 mm to (104.3, 70.2), turned to 180 degrees
- moved C8 5.43 mm to (124.9, 79.6)
- moved U4 5.43 mm to (127.4, 79.6)
- moved C9 4.71 mm to (129.9, 79.6), turned to 270 degrees
- moved D1 1.28 mm to (115.7, 72.1)
- moved R8 0.66 mm to (113.5, 71.7), turned to 90 degrees
- moved C11 0.23 mm to (134.3, 80.8)
- turned U10 to 270 degrees
Routing:
- net Net-(R10-Pad2): track 0.93 -> 15.6 mm, vias 2 -> 3
- net +3V3: track 0.00 -> 8.11 mm, vias 0 -> 7
- net Net-(R8-Pad2): track 1.81 -> 8.46 mm, vias 1 -> 2
- net GND: track 0.42 -> 4.86 mm, vias 2 -> 17
- net SYS: track 0.00 -> 3.31 mm
- net Net-(D1-Pad1): track 0.00 -> 1.38 mm
- net Net-(R9-Pad1): track 4.87 -> 3.53 mm
- added copper zone on F.Cu, net +3V3
- added copper zone on In1.Cu, net GND

Commit message: Update
Parts:
- moved U7 0.70 mm to (134.2, 92.5)
- moved C13 0.24 mm to (146.3, 83.4)
- moved C12 0.24 mm to (146.3, 81.2)
Routing:
- net GND: track 4.86 -> 6.98 mm, vias 17 -> 18
- net +3V3: track 8.11 -> 8.61 mm
