File: KiCad/GPS Hardware/_autosave-GPS Hardware.kicad_pcb (KiCad board)
At the start: 4 copper layers, 50 x 50 mm, 74 parts, among them J1 USB_C_Receptacle_USB2.0, J2 Conn_01x06_Male, J3 Conn_Coaxial, J4 SIM8051-6-0-14-01-X-REVD, J5 B2B-XH-A(LF)(SN), Q1 BC847, Q2 BC847, Q3 BSS84, U1 ESD122DMX, U10 ublox_SAM-M8Q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

Commit message: Update to laptop
Parts:
- moved C31 2.09 mm to (118.8, 63.5), turned to 90 degrees
- moved C30 2.03 mm to (120.8, 63.6), turned to 90 degrees
- moved R2 0.88 mm to (104.2, 68.9)
- moved R11 0.86 mm to (103.4, 70.2)
- moved D6 0.37 mm to (119.9, 63.6), turned to 90 degrees
- moved R6 0.18 mm to (103.4, 73.3)
- moved R7 0.18 mm to (103.4, 74.3)
- moved TH1 0.17 mm to (103.9, 71.9)
Routing:
- net Net-(R9-Pad1): track 3.53 -> 10.00 mm
- net GND: track 6.98 -> 13.0 mm, vias 18 -> 22
- net Net-(J3-Pad1): track 3.82 -> 0.03 mm
- net Net-(Q1-Pad1): track 0.00 -> 3.30 mm
- net Net-(R17-Pad1): track 0.00 -> 2.06 mm
- net Net-(D2-Pad1): track 0.00 -> 1.64 mm
- net Net-(D2-Pad2): track 0.00 -> 1.54 mm
- net VSIM: track 25.9 -> 26.9 mm
- net SCL_Power: track 83.1 -> 84.0 mm
- net INT_Power: track 62.0 -> 62.7 mm
- net SDA_Power: track 80.8 -> 81.5 mm
