File: KiCad/GPS Prototype 2/Cellular and GPS.sch (KiCad schematic (older format))
At the start: 30 parts, among them J3 Conn_Coaxial, J4 SIM8065-6-1-14-01-A_REVA1, Q1 BC847, Q2 BC847, Q3 BSS84, U10 ublox_SAM-M8Q, U7 74AVC2T245GU-Q100X, U8 SARA-U201

Commit message: updated
Parts:
- C18, C19, C20, C21, C22, C23: footprint Capacitor_SMD:C_0402_1005Metric_Pad0.74x0.62mm_HandSolder -> Capacitor_SMD:C_0805_2012Metric
- R16, R20: footprint Resistor_SMD:R_0402_1005Metric_Pad0.72x0.64mm_HandSolder -> Resistor_SMD:R_0805_2012Metric
- R17, R18, R19: footprint Resistor_SMD:R_0603_1608Metric_Pad0.98x0.95mm_HandSolder -> Resistor_SMD:R_0805_2012Metric
Changed lines of the file:
@@
 F 0 "R16" H 1770 2746 50  0000 L CNN
 F 1 "100k" H 1770 2655 50  0000 L CNN
-F 2 "Resistor_SMD:R_0402_1005Metric_Pad0.72x0.64mm_HandSolder" V 1630 2700 50  0001 C CNN
+F 2 "Resistor_SMD:R_0805_2012Metric" V 1630 2700 50  0001 C CNN
 F 3 "~" H 1700 2700 50  0001 C CNN
 	1    1700 2700
@@
 F 0 "C18" H 1965 1396 50  0000 L CNN
 F 1 "10n" H 1965 1305 50  0000 L CNN
-F 2 "Capacitor_SMD:C_0402_1005Metric_Pad0.74x0.62mm_HandSolder" H 1888 1200 50  0001 C CNN
+F 2 "Capacitor_SMD:C_0805_2012Metric" H 1888 1200 50  0001 C CNN
 F 3 "~" H 1850 1350 50  0001 C CNN
 	1    1850 1350
@@
 F 0 "C19" H 2265 1396 50  0000 L CNN
 F 1 "0u1" H 2265 1305 50  0000 L CNN
-F 2 "Capacitor_SMD:C_0402_1005Metric_Pad0.74x0.62mm_HandSolder" H 2188 1200 50  0001 C CNN
+F 2 "Capacitor_SMD:C_0805_2012Metric" H 2188 1200 50  0001 C CNN
 F 3 "~" H 2150 1350 50  0001 C CNN
 	1    2150 1350
@@
 F 0 "C20" H 2565 1396 50  0000 L CNN
 F 1 "56p" H 2565 1305 50  0000 L CNN
-F 2 "Capacitor_SMD:C_0402_1005Metric_Pad0.74x0.62mm_HandSolder" H 2488 1200 50  0001 C CNN
+F 2 "Capacitor_SMD:C_0805_2012Metric" H 2488 1200 50  0001 C CNN
 F 3 "~" H 2450 1350 50  0001 C CNN
 	1    2450 1350
@@
 F 0 "C21" H 2865 1396 50  0000 L CNN
 F 1 "15p" H 2865 1305 50  0000 L CNN
-F 2 "Capacitor_SMD:C_0402_1005Metric_Pad0.74x0.62mm_HandSolder" H 2788 1200 50  0001 C CNN
+F 2 "Capacitor_SMD:C_0805_2012Metric" H 2788 1200 50  0001 C CNN
 F 3 "~" H 2750 1350 50  0001 C CNN
 	1    2750 1350
@@
 F 0 "C22" H 3415 5896 50  0000 L CNN
 F 1 "0u1" H 3415 5805 50  0000 L CNN
-F 2 "Capacitor_SMD:C_0402_1005Metric_Pad0.74x0.62mm_HandSolder" H 3338 5700 50  0001 C CNN
+F 2 "Capacitor_SMD:C_0805_2012Metric" H 3338 5700 50  0001 C CNN
 F 3 "~" H 3300 5850 50  0001 C CNN
 	1    3300 5850
@@
 F 0 "C23" H 4065 5796 50  0000 L CNN
 F 1 "0u1" H 4065 5705 50  0000 L CNN
-F 2 "Capacitor_SMD:C_0402_1005Metric_Pad0.74x0.62mm_HandSolder" H 3988 5600 50  0001 C CNN
+F 2 "Capacitor_SMD:C_0805_2012Metric" H 3988 5600 50  0001 C CNN
 F 3 "~" H 3950 5750 50  0001 C CNN
 	1    3950 5750
@@
 F 0 "R17" H 3970 2896 50  0000 L CNN
 F 1 "10k" V 3900 2800 50  0000 L CNN
-F 2 "Resistor_SMD:R_0603_1608Metric_Pad0.98x0.95mm_HandSolder" V 3830 2850 50  0001 C CNN
+F 2 "Resistor_SMD:R_0805_2012Metric" V 3830 2850 50  0001 C CNN
 F 3 "~" H 3900 2850 50  0001 C CNN
 	1    3900 2850
@@
 F 0 "R18" H 4170 3046 50  0000 L CNN
 F 1 "47k" V 4100 2950 50  0000 L CNN
-F 2 "Resistor_SMD:R_0603_1608Metric_Pad0.98x0.95mm_HandSolder" V 4030 3000 50  0001 C CNN
+F 2 "Resistor_SMD:R_0805_2012Metric" V 4030 3000 50  0001 C CNN
 F 3 "~" H 4100 3000 50  0001 C CNN
 	1    4100 3000
@@
 F 0 "R19" H 4520 2246 50  0000 L CNN
 F 1 "250" V 4450 2150 50  0000 L CNN
-F 2 "Resistor_SMD:R_0603_1608Metric_Pad0.98x0.95mm_HandSolder" V 4380 2200 50  0001 C CNN
+F 2 "Resistor_SMD:R_0805_2012Metric" V 4380 2200 50  0001 C CNN
 F 3 "~" H 4450 2200 50  0001 C CNN
 	1    4450 2200
@@
 F 0 "R20" H 5220 3646 50  0000 L CNN
 F 1 "47k" H 5220 3555 50  0000 L CNN
-F 2 "Resistor_SMD:R_0402_1005Metric_Pad0.72x0.64mm_HandSolder" V 5080 3600 50  0001 C CNN
+F 2 "Resistor_SMD:R_0805_2012Metric" V 5080 3600 50  0001 C CNN
 F 3 "~" H 5150 3600 50  0001 C CNN
 	1    5150 3600
