File: KiCad/GPS Prototype 2/MCU.sch (KiCad schematic (older format))
At the start: 16 parts, among them J2 Conn_01x06_Male, U5 ATmega328-AU, U6 SN74AVC4T774PW, Y1 Crystal

Commit message: updated
Parts:
- removed J2: Conn_01x06_Male, Connector_PinHeader_1.00mm:PinHeader_2x03_P1.00mm_Vertical_SMD, symbol GPS-Hardware-rescue:Conn_01x06_Male-Connector
- added J2: TSM-103-01-L-DV-P-TR, SAMTEC_TSM-103-01-L-DV-P-TR, symbol GPS~Hardware:TSM-103-01-L-DV-P-TR
- C10, C11, C12, C13, C16, C17: footprint Capacitor_SMD:C_0402_1005Metric_Pad0.74x0.62mm_HandSolder -> Capacitor_SMD:C_0805_2012Metric
- C14, C15: footprint Capacitor_SMD:C_0603_1608Metric_Pad1.08x0.95mm_HandSolder -> Capacitor_SMD:C_0805_2012Metric
- R12, R13, R14, R15: footprint Resistor_SMD:R_0402_1005Metric_Pad0.72x0.64mm_HandSolder -> Resistor_SMD:R_0805_2012Metric
- U6: footprint GPS Hardware:SOP65P640X120-16N -> SOP65P640X120-16N
Changed lines of the file:
@@
 F 0 "C10" H 2065 2246 50  0000 L CNN
 F 1 "0u1" H 2065 2155 50  0000 L CNN
-F 2 "Capacitor_SMD:C_0402_1005Metric_Pad0.74x0.62mm_HandSolder" H 1988 2050 50  0001 C CNN
+F 2 "Capacitor_SMD:C_0805_2012Metric" H 1988 2050 50  0001 C CNN
 F 3 "~" H 1950 2200 50  0001 C CNN
 	1    1950 2200
@@
 F 0 "C14" H 4515 2396 50  0000 L CNN
 F 1 "22p" H 4515 2305 50  0000 L CNN
-F 2 "Capacitor_SMD:C_0603_1608Metric_Pad1.08x0.95mm_HandSolder" H 4438 2200 50  0001 C CNN
+F 2 "Capacitor_SMD:C_0805_2012Metric" H 4438 2200 50  0001 C CNN
 F 3 "https://www.mouser.co.uk/ProductDetail/KEMET/C0603C220J1HACTU?qs=W0yvOO0ixfF6hDt%252BXfnhnA%3D%3D" H 4400 2350 50  0001 C CNN
 	1    4400 2350
@@
 F 0 "C15" H 4515 2996 50  0000 L CNN
 F 1 "22p" H 4515 2905 50  0000 L CNN
-F 2 "Capacitor_SMD:C_0603_1608Metric_Pad1.08x0.95mm_HandSolder" H 4438 2800 50  0001 C CNN
+F 2 "Capacitor_SMD:C_0805_2012Metric" H 4438 2800 50  0001 C CNN
 F 3 "https://www.mouser.co.uk/ProductDetail/KEMET/C0603C220J1HACTU?qs=W0yvOO0ixfF6hDt%252BXfnhnA%3D%3D" H 4400 2950 50  0001 C CNN
 	1    4400 2950
@@
 F 0 "R15" H 4070 3796 50  0000 L CNN
 F 1 "10k" V 4000 3700 50  0000 L CNN
-F 2 "Resistor_SMD:R_0402_1005Metric_Pad0.72x0.64mm_HandSolder" V 3930 3750 50  0001 C CNN
+F 2 "Resistor_SMD:R_0805_2012Metric" V 3930 3750 50  0001 C CNN
 F 3 "~" H 4000 3750 50  0001 C CNN
 	1    4000 3750
@@
 F 0 "R12" V 3650 2150 50  0000 C CNN
 F 1 "330" V 3700 2300 50  0000 C CNN
-F 2 "Resistor_SMD:R_0402_1005Metric_Pad0.72x0.64mm_HandSolder" V 3630 2300 50  0001 C CNN
+F 2 "Resistor_SMD:R_0805_2012Metric" V 3630 2300 50  0001 C CNN
 F 3 "~" H 3700 2300 50  0001 C CNN
 	1    3700 2300
@@
 F 0 "R13" V 3650 2250 50  0000 C CNN
 F 1 "330" V 3700 2400 50  0000 C CNN
-F 2 "Resistor_SMD:R_0402_1005Metric_Pad0.72x0.64mm_HandSolder" V 3630 2400 50  0001 C CNN
+F 2 "Resistor_SMD:R_0805_2012Metric" V 3630 2400 50  0001 C CNN
 F 3 "~" H 3700 2400 50  0001 C CNN
 	1    3700 2400
@@
 F 0 "R14" V 3650 2350 50  0000 C CNN
 F 1 "330" V 3700 2500 50  0000 C CNN
-F 2 "Resistor_SMD:R_0402_1005Metric_Pad0.72x0.64mm_HandSolder" V 3630 2500 50  0001 C CNN
+F 2 "Resistor_SMD:R_0805_2012Metric" V 3630 2500 50  0001 C CNN
 F 3 "~" H 3700 2500 50  0001 C CNN
 	1    3700 2500
@@
 F 0 "C11" H 2665 1096 50  0000 L CNN
 F 1 "0u1" H 2665 1005 50  0000 L CNN
-F 2 "Capacitor_SMD:C_0402_1005Metric_Pad0.74x0.62mm_HandSolder" H 2588 900 50  0001 C CNN
+F 2 "Capacitor_SMD:C_0805_2012Metric" H 2588 900 50  0001 C CNN
 F 3 "~" H 2550 1050 50  0001 C CNN
 	1    2550 1050
@@
 F 0 "C12" H 3015 1096 50  0000 L CNN
 F 1 "0u1" H 3015 1005 50  0000 L CNN
-F 2 "Capacitor_SMD:C_0402_1005Metric_Pad0.74x0.62mm_HandSolder" H 2938 900 50  0001 C CNN
+F 2 "Capacitor_SMD:C_0805_2012Metric" H 2938 900 50  0001 C CNN
 F 3 "~" H 2900 1050 50  0001 C CNN
 	1    2900 1050
@@
 F 0 "C13" H 3365 1096 50  0000 L CNN
 F 1 "0u1" H 3365 1005 50  0000 L CNN
-F 2 "Capacitor_SMD:C_0402_1005Metric_Pad0.74x0.62mm_HandSolder" H 3288 900 50  0001 C CNN
+F 2 "Capacitor_SMD:C_0805_2012Metric" H 3288 900 50  0001 C CNN
 F 3 "~" H 3250 1050 50  0001 C CNN
 	1    3250 1050
@@
 F 0 "C17" H 7715 2146 50  0000 L CNN
 F 1 "0u1" H 7715 2055 50  0000 L CNN
-F 2 "Capacitor_SMD:C_0402_1005Metric_Pad0.74x0.62mm_HandSolder" H 7638 1950 50  0001 C CNN
+F 2 "Capacitor_SMD:C_0805_2012Metric" H 7638 1950 50  0001 C CNN
 F 3 "~" H 7600 2100 50  0001 C CNN
 	1    7600 2100
@@
 F 0 "C16" H 7165 2246 50  0000 L CNN
 F 1 "0u1" H 7165 2155 50  0000 L CNN
-F 2 "Capacitor_SMD:C_0402_1005Metric_Pad0.74x0.62mm_HandSolder" H 7088 2050 50  0001 C CNN
+F 2 "Capacitor_SMD:C_0805_2012Metric" H 7088 2050 50  0001 C CNN
 F 3 "~" H 7050 2200 50  0001 C CNN
 	1    7050 2200
@@
 $EndComp
 $Comp
-L GPS-Hardware-rescue:Conn_01x06_Male-Connector J2
-U 1 1 612547C1
-P 4150 1300
-AR Path="/612547C1" Ref="J2"  Part="1"
-AR Path="/613BCFBA/612547C1" Ref="J2"  Part="1"
-F 0 "J2" H 4258 1681 50  0000 C CNN
-F 1 "Conn_01x06_Male" H 4258 1590 50  0000 C CNN
-F 2 "Connector_PinHeader_1.00mm:PinHeader_2x03_P1.00mm_Vertical_SMD" H 4150 1300 50  0001 C CNN
-F 3 "~" H 4150 1300 50  0001 C CNN
-	1    4150 1300
-	1    0    0    -1
-$EndComp
-$Comp
 L GPS-Hardware-rescue:+3V3-power #PWR0135
 U 1 1 61218E15
-P 4350 1200
-F 0 "#PWR0135" H 4350 1050 50  0001 C CNN
-F 1 "+3V3" V 4365 1328 50  0000 L CNN
-F 2 "" H 4350 1200 50  0001 C CNN
-F 3 "" H 4350 1200 50  0001 C CNN
-	1    4350 1200
+P 6000 1000
+F 0 "#PWR0135" H 6000 850 50  0001 C CNN
+F 1 "+3V3" V 6015 1128 50  0000 L CNN
+F 2 "" H 6000 1000 50  0001 C CNN
+F 3 "" H 6000 1000 50  0001 C CNN
+	1    6000 1000
 	0    1    1    0
 $EndComp
@@
 L GPS-Hardware-rescue:GND-power #PWR0132
 U 1 1 611EA8CA
-P 4350 1400
-F 0 "#PWR0132" H 4350 1150 50  0001 C CNN
-F 1 "GND" V 4355 1272 50  0000 R CNN
-F 2 "" H 4350 1400 50  0001 C CNN
-F 3 "" H 4350 1400 50  0001 C CNN
-	1    4350 1400
+P 6000 1100
+F 0 "#PWR0132" H 6000 850 50  0001 C CNN
+F 1 "GND" V 6005 972 50  0000 R CNN
+F 2 "" H 6000 1100 50  0001 C CNN
+F 3 "" H 6000 1100 50  0001 C CNN
+	1    6000 1100
 	0    -1   -1   0
 $EndComp
-Text GLabel 4350 1500 2    50   Output ~ 0
+Text GLabel 5000 1200 0    50   Output ~ 0
 MOSI
-Text GLabel 4350 1600 2    50   Output ~ 0
+Text GLabel 6000 1200 2    50   Output ~ 0
 RESET
-Text GLabel 4350 1100 2    50   Output ~ 0
+Text GLabel 5000 1000 0    50   Output ~ 0
 SCK
-Text GLabel 4350 1300 2    50   Output ~ 0
+Text GLabel 5000 1100 0    50   Output ~ 0
 MISO
 $Comp
@@
 F 0 "U6" H 6250 3820 50  0000 C CNN
 F 1 "SN74AVC4T774PW" H 6250 3729 50  0000 C CNN
-F 2 "GPS Hardware:SOP65P640X120-16N" H 6250 2750 50  0001 L BNN
+F 2 "SOP65P640X120-16N" H 6250 2750 50  0001 L BNN
 F 3 "" H 6250 2750 50  0001 L BNN
 	1    6250 2750
@@
 Wire Wire Line
 	5200 2450 5200 2650
+$Comp
+L GPS~Hardware:TSM-103-01-L-DV-P-TR J2
+U 1 1 6226FA65
+P 5500 1100
+F 0 "J2" H 5500 1467 50  0000 C CNN
+F 1 "TSM-103-01-L-DV-P-TR" H 5500 1376 50  0000 C CNN
+F 2 "SAMTEC_TSM-103-01-L-DV-P-TR" H 5500 1100 50  0001 L BNN
+F 3 "" H 5500 1100 50  0001 L BNN
+F 4 "SAMTEC" H 5500 1100 50  0001 L BNN "MANUFACTURER"
+	1    5500 1100
+	1    0    0    -1
+$EndComp
 $EndSCHEMATC
