File: KiCad/GPS Hardware/GPS Prototype 2 - ESP32/Power.sch (KiCad schematic (older format))
At the start: 27 parts, among them J1 USB_C_Receptacle_USB2.0, J5 B2B-XH-A(LF)(SN), U3 BQ24295, U4 LM3480-3.3

Commit message: Update to Uni computers
Finish esp32 connections.
Connections:
- wire segments 45 -> 46
Changed lines of the file:
@@
 	1    0    0    -1
 $EndComp
+Wire Wire Line
+	3450 2800 3550 2800
+Connection ~ 3550 2800
 $EndSCHEMATC

Commit message: Update
Parts:
- C7: symbol GPS-Hardware-rescue:CP-Device -> GPS-Hardware-rescue:CP-Device-GPS-Hardware-rescue
- D1: symbol GPS-Hardware-rescue:LED-Device -> GPS-Hardware-rescue:LED-Device-GPS-Hardware-rescue
- J1: symbol GPS-Hardware-rescue:USB_C_Receptacle_USB2.0-Connector -> GPS-Hardware-rescue:USB_C_Receptacle_USB2.0-Connector-GPS-Hardware-rescue
- L1: symbol GPS-Hardware-rescue:L-Device -> GPS-Hardware-rescue:L-Device-GPS-Hardware-rescue
- TH1: symbol GPS-Hardware-rescue:Thermistor_NTC-Device -> GPS-Hardware-rescue:Thermistor_NTC-Device-GPS-Hardware-rescue
- U4: symbol GPS-Hardware-rescue:LM3480-3.3-Regulator_Linear -> GPS-Hardware-rescue:LM3480-3.3-Regulator_Linear-GPS-Hardware-rescue
Changed lines of the file:
@@
 $EndComp
 $Comp
-L GPS-Hardware-rescue:USB_C_Receptacle_USB2.0-Connector J?
+L GPS-Hardware-rescue:USB_C_Receptacle_USB2.0-Connector-GPS-Hardware-rescue J?
 U 1 1 613BC22B
 P 1150 1550
@@
 NoConn ~ 1750 2150
 $Comp
-L GPS-Hardware-rescue:GND-power #PWR?
+L GPS-Hardware-rescue:GND-power-GPS-Hardware-rescue #PWR?
 U 1 1 613BC25E
 P 1150 2450
@@
 $EndComp
 $Comp
-L GPS-Hardware-rescue:GND-power #PWR?
+L GPS-Hardware-rescue:GND-power-GPS-Hardware-rescue #PWR?
 U 1 1 613BC264
 P 5150 3050
@@
 $EndComp
 $Comp
-L GPS-Hardware-rescue:GND-power #PWR?
+L GPS-Hardware-rescue:GND-power-GPS-Hardware-rescue #PWR?
 U 1 1 613BC27C
 P 3950 2100
@@
 $EndComp
 $Comp
-L GPS-Hardware-rescue:GND-power #PWR?
+L GPS-Hardware-rescue:GND-power-GPS-Hardware-rescue #PWR?
 U 1 1 613BC288
 P 3950 2200
@@
 	3800 2450 3550 2450
 $Comp
-L GPS-Hardware-rescue:+3.3V-power #PWR?
+L GPS-Hardware-rescue:+3.3V-power-GPS-Hardware-rescue #PWR?
 U 1 1 613BC2B4
 P 3800 2450
@@
 $EndComp
 $Comp
-L GPS-Hardware-rescue:GND-power #PWR?
+L GPS-Hardware-rescue:GND-power-GPS-Hardware-rescue #PWR?
 U 1 1 613BC2BA
 P 2050 1150
@@
 $EndComp
 $Comp
-L GPS-Hardware-rescue:GND-power #PWR?
+L GPS-Hardware-rescue:GND-power-GPS-Hardware-rescue #PWR?
 U 1 1 613BC2C0
 P 2050 1250
@@
 $EndComp
 $Comp
-L GPS-Hardware-rescue:L-Device L?
+L GPS-Hardware-rescue:L-Device-GPS-Hardware-rescue L?
 U 1 1 613BC2D0
 P 5750 1300
@@
 $EndComp
 $Comp
-L GPS-Hardware-rescue:GND-power #PWR?
+L GPS-Hardware-rescue:GND-power-GPS-Hardware-rescue #PWR?
 U 1 1 613BC2F0
 P 6250 1800
@@
 SYS
 $Comp
-L GPS-Hardware-rescue:GND-power #PWR?
+L GPS-Hardware-rescue:GND-power-GPS-Hardware-rescue #PWR?
 U 1 1 613BC2F9
 P 850 2450
@@
 SYS
 $Comp
-L GPS-Hardware-rescue:LED-Device D?
+L GPS-Hardware-rescue:LED-Device-GPS-Hardware-rescue D?
 U 1 1 613BC300
 P 5700 1900
@@
 	5900 2000 5450 2000
 $Comp
-L GPS-Hardware-rescue:GND-power #PWR?
+L GPS-Hardware-rescue:GND-power-GPS-Hardware-rescue #PWR?
 U 1 1 613BC322
 P 6100 2350
@@
 	5850 2250 5150 2250
 $Comp
-L GPS-Hardware-rescue:GND-power #PWR?
+L GPS-Hardware-rescue:GND-power-GPS-Hardware-rescue #PWR?
 U 1 1 613BC331
 P 5850 2550
@@
 $EndComp
 $Comp
-L GPS-Hardware-rescue:GND-power #PWR?
+L GPS-Hardware-rescue:GND-power-GPS-Hardware-rescue #PWR?
 U 1 1 613BC33D
 P 5250 2650
@@
 $EndComp
 $Comp
-L GPS-Hardware-rescue:Thermistor_NTC-Device TH?
+L GPS-Hardware-rescue:Thermistor_NTC-Device-GPS-Hardware-rescue TH?
 U 1 1 613BC353
 P 6000 3100
@@
 	5600 2950 6000 2950
 $Comp
-L GPS-Hardware-rescue:GND-power #PWR?
+L GPS-Hardware-rescue:GND-power-GPS-Hardware-rescue #PWR?
 U 1 1 613BC35C
 P 5600 3250
@@
 $EndComp
 $Comp
-L GPS-Hardware-rescue:GND-power #PWR?
+L GPS-Hardware-rescue:GND-power-GPS-Hardware-rescue #PWR?
 U 1 1 613BC362
 P 6000 3250
@@
 $EndComp
 $Comp
-L GPS-Hardware-rescue:GND-power #PWR0120
+L GPS-Hardware-rescue:GND-power-GPS-Hardware-rescue #PWR0120
 U 1 1 61411635
 P 3850 1700
@@
 $EndComp
 $Comp
-L GPS-Hardware-rescue:GND-power #PWR0121
+L GPS-Hardware-rescue:GND-power-GPS-Hardware-rescue #PWR0121
 U 1 1 614120E2
 P 3850 1250
@@
 	3850 1400 4250 1400
 $Comp
-L GPS-Hardware-rescue:CP-Device C7
+L GPS-Hardware-rescue:CP-Device-GPS-Hardware-rescue C7
 U 1 1 6142C46C
 P 6850 1650
@@
 $EndComp
 $Comp
-L GPS-Hardware-rescue:GND-power #PWR0122
+L GPS-Hardware-rescue:GND-power-GPS-Hardware-rescue #PWR0122
 U 1 1 6142CFD4
 P 6850 1800
@@
 Different capacitor values for low impedance at a range of frequencies
 $Comp
-L GPS-Hardware-rescue:LM3480-3.3-Regulator_Linear U4
+L GPS-Hardware-rescue:LM3480-3.3-Regulator_Linear-GPS-Hardware-rescue U4
 U 1 1 6145B119
 P 8600 1750
@@
 Connection ~ 8150 1750
 $Comp
-L GPS-Hardware-rescue:+3V3-power #PWR0123
+L GPS-Hardware-rescue:+3V3-power-GPS-Hardware-rescue #PWR0123
 U 1 1 6146807E
 P 9250 1750
@@
 Connection ~ 9050 1750
 $Comp
-L GPS-Hardware-rescue:GND-power #PWR0124
+L GPS-Hardware-rescue:GND-power-GPS-Hardware-rescue #PWR0124
 U 1 1 6146B115
 P 8150 2050
@@
 $EndComp
 $Comp
-L GPS-Hardware-rescue:GND-power #PWR0125
+L GPS-Hardware-rescue:GND-power-GPS-Hardware-rescue #PWR0125
 U 1 1 6146BB0D
 P 9050 2050
@@
 $EndComp
 $Comp
-L GPS-Hardware-rescue:GND-power #PWR0126
+L GPS-Hardware-rescue:GND-power-GPS-Hardware-rescue #PWR0126
 U 1 1 6146F41C
 P 8600 2050

Commit message: Update to Laptop
Still a lot more to go
Parts:
- removed C8: 0u1, Capacitor_SMD:C_1206_3216Metric_Pad1.33x1.80mm_HandSolder, symbol GPS-Hardware-rescue:C-Device
- removed U4: LM3480-3.3, Package_TO_SOT_SMD:SOT-23, symbol GPS-Hardware-rescue:LM3480-3.3-Regulator_Linear-GPS-Hardware-rescue
- added C12: 100u, Capacitor_Tantalum_SMD:CP_EIA-6032-15_Kemet-U_Pad2.25x2.35mm_HandSolder, symbol Device:CP
- added C8: 10u, Capacitor_SMD:C_1206_3216Metric_Pad1.33x1.80mm_HandSolder, symbol Device:C
- added D7: SP712-02HTG, GPS Hardware:SOT95P237X115-3N, symbol GPS~Hardware:SP712-02HTG
- added U2: MIC5209-4.2YS-TR, Package_TO_SOT_SMD:SOT-223, symbol GPS~Hardware:MIC5209-4.2YS-TR
Connections:
- wire segments 46 -> 47
Changed lines of the file:
@@
 	3550 2750 3550 2800
-Wire Wire Line
-	3300 4700 3200 4700
 Wire Wire Line
 	3800 2750 3800 2900
@@
 Text Notes 7500 950  0    50   ~ 0
 Different capacitor values for low impedance at a range of frequencies
-$Comp
-L GPS-Hardware-rescue:LM3480-3.3-Regulator_Linear-GPS-Hardware-rescue U4
-U 1 1 6145B119
-P 8600 1750
-F 0 "U4" H 8600 1992 50  0000 C CNN
-F 1 "LM3480-3.3" H 8600 1901 50  0000 C CNN
-F 2 "Package_TO_SOT_SMD:SOT-23" H 8600 1975 50  0001 C CIN
-F 3 "http://www.ti.com/lit/ds/symlink/lm3480.pdf" H 8600 1750 50  0001 C CNN
-	1    8600 1750
-	1    0    0    -1
-$EndComp
-$Comp
-L GPS-Hardware-rescue:C-Device C8
-U 1 1 6146363C
-P 8150 1900
-F 0 "C8" H 8265 1946 50  0000 L CNN
-F 1 "0u1" H 8265 1855 50  0000 L CNN
-F 2 "Capacitor_SMD:C_1206_3216Metric_Pad1.33x1.80mm_HandSolder" H 8188 1750 50  0001 C CNN
-F 3 "~" H 8150 1900 50  0001 C CNN
-	1    8150 1900
-	1    0    0    -1
-$EndComp
-$Comp
-L GPS-Hardware-rescue:C-Device C9
-U 1 1 614640B3
-P 9050 1900
-F 0 "C9" H 9165 1946 50  0000 L CNN
-F 1 "0u1" H 9165 1855 50  0000 L CNN
-F 2 "Capacitor_SMD:C_1206_3216Metric_Pad1.33x1.80mm_HandSolder" H 9088 1750 50  0001 C CNN
-F 3 "~" H 9050 1900 50  0001 C CNN
-	1    9050 1900
-	1    0    0    -1
-$EndComp
-Wire Wire Line
-	8150 1750 8300 1750
-Wire Wire Line
-	8900 1750 9050 1750
-Text GLabel 8000 1750 0    50   Input ~ 0
-VCC
-Wire Wire Line
-	8000 1750 8150 1750
-Connection ~ 8150 1750
-$Comp
-L GPS-Hardware-rescue:+3V3-power-GPS-Hardware-rescue #PWR0123
-U 1 1 6146807E
-P 9250 1750
-F 0 "#PWR0123" H 9250 1600 50  0001 C CNN
-F 1 "+3V3" V 9265 1878 50  0000 L CNN
-F 2 "" H 9250 1750 50  0001 C CNN
-F 3 "" H 9250 1750 50  0001 C CNN
-	1    9250 1750
-	0    1    1    0
-$EndComp
-Wire Wire Line
-	9050 1750 9250 1750
-Connection ~ 9050 1750
-$Comp
-L GPS-Hardware-rescue:GND-power-GPS-Hardware-rescue #PWR0124
-U 1 1 6146B115
-P 8150 2050
-F 0 "#PWR0124" H 8150 1800 50  0001 C CNN
-F 1 "GND" H 8155 1877 50  0000 C CNN
-F 2 "" H 8150 2050 50  0001 C CNN
-F 3 "" H 8150 2050 50  0001 C CNN
-	1    8150 2050
-	1    0    0    -1
-$EndComp
-$Comp
-L GPS-Hardware-rescue:GND-power-GPS-Hardware-rescue #PWR0125
-U 1 1 6146BB0D
-P 9050 2050
-F 0 "#PWR0125" H 9050 1800 50  0001 C CNN
-F 1 "GND" H 9055 1877 50  0000 C CNN
-F 2 "" H 9050 2050 50  0001 C CNN
-F 3 "" H 9050 2050 50  0001 C CNN
-	1    9050 2050
-	1    0    0    -1
-$EndComp
-$Comp
-L GPS-Hardware-rescue:GND-power-GPS-Hardware-rescue #PWR0126
-U 1 1 6146F41C
-P 8600 2050
-F 0 "#PWR0126" H 8600 1800 50  0001 C CNN
-F 1 "GND" H 8605 1877 50  0000 C CNN
-F 2 "" H 8600 2050 50  0001 C CNN
-F 3 "" H 8600 2050 50  0001 C CNN
-	1    8600 2050
-	1    0    0    -1
-$EndComp
 Wire Wire Line
 	3750 950  3850 950
@@
 	3450 2800 3550 2800
 Connection ~ 3550 2800
+$Comp
+L GPS~Hardware:MIC5209-4.2YS-TR U2
+U 1 1 62C71F30
+P 9250 1700
+F 0 "U2" H 9250 2042 50  0000 C CNN
+F 1 "MIC5209-4.2YS-TR" H 9250 1951 50  0000 C CNN
+F 2 "Package_TO_SOT_SMD:SOT-223" H 9250 1950 50  0001 C CNN
+F 3 "" H 9250 1950 50  0001 C CNN
+	1    9250 1700
+	1    0    0    -1
+$EndComp
+Text GLabel 8150 1600 0    50   Input ~ 0
+VCC
+$Comp
+L GPS-Hardware-rescue:C-Device C9
+U 1 1 62C749FD
+P 8600 1750
+F 0 "C9" H 8715 1796 50  0000 L CNN
+F 1 "0u1" H 8715 1705 50  0000 L CNN
+F 2 "Capacitor_SMD:C_1206_3216Metric_Pad1.33x1.80mm_HandSolder" H 8638 1600 50  0001 C CNN
+F 3 "~" H 8600 1750 50  0001 C CNN
+	1    8600 1750
+	1    0    0    -1
+$EndComp
+$Comp
+L Device:C C8
+U 1 1 62C75DFE
+P 8300 1750
+F 0 "C8" H 8415 1796 50  0000 L CNN
+F 1 "10u" H 8415 1705 50  0000 L CNN
+F 2 "Capacitor_SMD:C_1206_3216Metric_Pad1.33x1.80mm_HandSolder" H 8338 1600 50  0001 C CNN
+F 3 "~" H 8300 1750 50  0001 C CNN
+	1    8300 1750
+	1    0    0    -1
+$EndComp
+Wire Wire Line
+	8150 1600 8300 1600
+Connection ~ 8300 1600
+Wire Wire Line
+	8300 1600 8600 1600
+Connection ~ 8600 1600
+Wire Wire Line
+	8600 1600 8950 1600
+$Comp
+L GPS-Hardware-rescue:GND-power-GPS-Hardware-rescue #PWR01
+U 1 1 62C7760C
+P 8300 1900
+F 0 "#PWR01" H 8300 1650 50  0001 C CNN
+F 1 "GND" H 8305 1727 50  0000 C CNN
+F 2 "" H 8300 1900 50  0001 C CNN
+F 3 "" H 8300 1900 50  0001 C CNN
+	1    8300 1900
+	1    0    0    -1
+$EndComp
+$Comp
+L GPS-Hardware-rescue:GND-power-GPS-Hardware-rescue #PWR02
+U 1 1 62C78084
+P 8600 1900
+F 0 "#PWR02" H 8600 1650 50  0001 C CNN
+F 1 "GND" H 8605 1727 50  0000 C CNN
+F 2 "" H 8600 1900 50  0001 C CNN
+F 3 "" H 8600 1900 50  0001 C CNN
+	1    8600 1900
+	1    0    0    -1
+$EndComp
+$Comp
+L GPS-Hardware-rescue:GND-power-GPS-Hardware-rescue #PWR04
+U 1 1 62C78719
+P 9250 2000
+F 0 "#PWR04" H 9250 1750 50  0001 C CNN
+F 1 "GND" H 9255 1827 50  0000 C CNN
+F 2 "" H 9250 2000 50  0001 C CNN
+F 3 "" H 9250 2000 50  0001 C CNN
+	1    9250 2000
+	1    0    0    -1
+$EndComp
+$Comp
+L Device:CP C12
+U 1 1 62C799C9
+P 9700 1750
+F 0 "C12" H 9818 1796 50  0000 L CNN
+F 1 "100u" H 9818 1705 50  0000 L CNN
+F 2 "Capacitor_Tantalum_SMD:CP_EIA-6032-15_Kemet-U_Pad2.25x2.35mm_HandSolder" H 9738 1600 50  0001 C CNN
+F 3 "https://www.mouser.co.uk/ProductDetail/Kyocera-AVX/TPSC107K010R0150?qs=sGAEpiMZZMsh%252B1woXyUXj5%252BF0nMD%252BKFrWBHmduck3mw%3D" H 9700 1750 50  0001 C CNN
+	1    9700 1750
+	1    0    0    -1
+$EndComp
+Wire Wire Line
+	9550 1600 9700 1600
+$Comp
+L GPS-Hardware-rescue:GND-power-GPS-Hardware-rescue #PWR05
+U 1 1 62C7B6B6
+P 9700 1900
+F 0 "#PWR05" H 9700 1650 50  0001 C CNN
+F 1 "GND" H 9705 1727 50  0000 C CNN
+F 2 "" H 9700 1900 50  0001 C CNN
+F 3 "" H 9700 1900 50  0001 C CNN
+	1    9700 1900
+	1    0    0    -1
+$EndComp
+$Comp
+L GPS-Hardware-rescue:+3V3-power-GPS-Hardware-rescue #PWR06
+U 1 1 62C7BADA
+P 9900 1600
+F 0 "#PWR06" H 9900 1450 50  0001 C CNN
+F 1 "+3V3" V 9915 1728 50  0000 L CNN
+F 2 "" H 9900 1600 50  0001 C CNN
+F 3 "" H 9900 1600 50  0001 C CNN
+	1    9900 1600
+	0    1    1    0
+$EndComp
+Wire Wire Line
+	9700 1600 9900 1600
+Connection ~ 9700 1600
+$Comp
+L GPS-Hardware-rescue:GND-power-GPS-Hardware-rescue #PWR03
+U 1 1 62C84CE9
+P 8950 1800
+F 0 "#PWR03" H 8950 1550 50  0001 C CNN
+F 1 "GND" H 8955 1627 50  0000 C CNN
+F 2 "" H 8950 1800 50  0001 C CNN
+F 3 "" H 8950 1800 50  0001 C CNN
+	1    8950 1800
+	1    0    0    -1
+$EndComp
+Wire Wire Line
+	8950 1700 8950 1800
+Text GLabel 2200 1550 0    50   Input ~ 0
+D+
+Text GLabel 2200 1650 0    50   Input ~ 0
+D-
+$Comp
+L GPS-Hardware-rescue:GND-power-GPS-Hardware-rescue #PWR0123
+U 1 1 62C7F4C3
+P 3400 1550
+F 0 "#PWR0123" H 3400 1300 50  0001 C CNN
+F 1 "GND" H 3405 1377 50  0000 C CNN
+F 2 "" H 3400 1550 50  0001 C CNN
+F 3 "" H 3400 1550 50  0001 C CNN
+	1    3400 1550
+	0    -1   -1   0
+$EndComp
+$Comp
+L GPS~Hardware:SP712-02HTG D7
+U 1 1 62CA71B2
+P 2200 1550
+F 0 "D7" H 2800 1815 50  0000 C CNN
+F 1 "SP712-02HTG" H 2800 1724 50  0000 C CNN
+F 2 "GPS Hardware:SOT95P237X115-3N" H 3250 1650 50  0001 L CNN
+F 3 "https://www.littelfuse.com/~/media/electronics/datasheets/tvs_diode_arrays/littelfuse_tvs_diode_array_sp712_datasheet.pdf.pdf" H 3250 1550 50  0001 L CNN
+F 4 "ESD Suppressors / TVS Diodes SP712 12V 20A 30kV SOT23-3L" H 3250 1450 50  0001 L CNN "Description"
+F 5 "1.15" H 3250 1350 50  0001 L CNN "Height"
+F 6 "576-SP712-02HTG" H 3250 1250 50  0001 L CNN "Mouser Part Number"
+F 7 "https://www.mouser.co.uk/ProductDetail/Littelfuse/SP712-02HTG?qs=GBLSl2AkiruqudcLsbr7vw%3D%3D" H 3250 1150 50  0001 L CNN "Mouser Price/Stock"
+F 8 "LITTELFUSE" H 3250 1050 50  0001 L CNN "Manufacturer_Name"
+F 9 "SP712-02HTG" H 3250 950 50  0001 L CNN "Manufacturer_Part_Number"
+	1    2200 1550
+	1    0    0    -1
+$EndComp
 $EndSCHEMATC
