File: KiCad/GPS Hardware/GPS Prototype 2 - ESP32/GPS Hardware.kicad_pcb (KiCad board)
At the start: 4 copper layers, 130 x 60 mm, 70 parts, among them J1 USB_C_Receptacle_USB2.0, J2 Conn_01x04_Male, J3 Conn_Coaxial, J4 Conn_01x05_Male, J5 B2B-XH-A(LF)(SN), J6 SIM8065-6-1-14-01-A_REVA1, J7 Conn_01x08_Male, Q1 BC847, Q2 BC847, Q3 BSS84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

Commit message: update
Parts:
- moved S2 72.2 mm to (23.8, 117.2), turned to 0 degrees
- moved R4 70.9 mm to (21.4, 123.0), turned to 180 degrees
- moved R3 69.5 mm to (20.6, 127.0), turned to 0 degrees
- moved C11 65.7 mm to (136.9, 147.2), turned to 270 degrees
- moved J2 63.4 mm to (22.5, 134.8), turned to 0 degrees
- moved R13 63.2 mm to (31.1, 118.0), turned to 270 degrees
- moved J4 57.2 mm to (40.1, 114.9), turned to 90 degrees
- moved U1 47.7 mm to (123.8, 139.8), turned to 180 degrees
- moved J7 41.4 mm to (59.6, 117.6), turned to 0 degrees
- moved C9 26.2 mm to (162.3, 139.1), turned to 270 degrees
- moved C8 22.3 mm to (166.1, 139.1), turned to 270 degrees
- moved R5 21.1 mm to (65.0, 131.2), turned to 90 degrees
- moved S1 18.4 mm to (59.8, 134.6), turned to 270 degrees
- moved C10 18.3 mm to (55.0, 139.0), turned to 270 degrees
- moved R12 11.5 mm to (64.9, 138.0), turned to 270 degrees
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Routing:
- net PWR_Cellular: track 87.5 -> 0.00 mm
- net RTS: track 56.7 -> 0.00 mm
- net CTS: track 56.7 -> 0.00 mm
- net TX: track 54.1 -> 0.00 mm
- net RX: track 52.1 -> 0.00 mm
- net VSIM: track 0.00 -> 47.5 mm
- net RST: track 0.00 -> 40.8 mm
- net CLK: track 0.00 -> 38.3 mm
- net /MCU Schematic/SENS_VN: track 35.7 -> 0.00 mm
- net +1V8: track 35.4 -> 0.00 mm
- net IO: track 0.00 -> 34.1 mm
- net /MCU Schematic/SENS_VP: track 32.0 -> 0.00 mm
- net SDA_Power: track 31.3 -> 0.00 mm, vias 1 -> 0
- net /MCU Schematic/IO14: track 22.9 -> 0.00 mm
- net /MCU Schematic/IO33: track 22.9 -> 0.00 mm
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
Commit message: Update
Parts:
- removed Q3: BSS84, Package_TO_SOT_SMD:SOT-323_SC-70
- removed R20: 47k, Resistor_SMD:R_1206_3216Metric_Pad1.30x1.75mm_HandSolder
- added D3: LED, LED_SMD:LED_1206_3216Metric_Pad1.42x1.75mm_HandSolder, F.Cu at (167.2, 93.7)
- added R14: 100k, Resistor_SMD:R_1206_3216Metric_Pad1.30x1.75mm_HandSolder, F.Cu at (175.8, 96.6)
- added R15: 1k, Resistor_SMD:R_1206_3216Metric_Pad1.30x1.75mm_HandSolder, F.Cu at (163.9, 93.6)
- Q2: value BC847 -> 2N7002
- R19: value 250 -> 820
- R8: moved to B.Cu
- moved R8 79.1 mm to (142.8, 126.2)
- moved C11 69.1 mm to (185.5, 98.2), turned to 180 degrees
- moved U1 62.6 mm to (179.1, 110.4), turned to 270 degrees
- moved R16 44.9 mm to (185.8, 122.6), turned to 90 degrees
- moved C12 43.1 mm to (164.9, 101.0), turned to 90 degrees
- moved U2 40.6 mm to (156.8, 100.4), turned to 90 degrees
- moved C9 38.7 mm to (150.3, 102.3), turned to 90 degrees
- moved C14 23.7 mm to (108.0, 129.8), turned to 180 degrees
- moved C17 22.4 mm to (117.0, 104.5)
- moved R17 22.2 mm to (119.7, 115.9)
- moved R9 22.1 mm to (136.4, 126.3)
- moved U8 22.1 mm to (131.7, 110.0)
- moved R18 22.1 mm to (119.7, 120.4)
- moved J3 22.1 mm to (135.0, 93.2)
- moved C21 21.8 mm to (143.9, 101.5)
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Connections:
- C13 pad 1: VCC_GPS -> +3V3
- C14 pad 1: VCC_GPS -> +3V3
- C23 pad 1: VCC_GPS -> +3V3
- C25 pad 1: VCC_GPS -> +3V3
- J2 pad 2: RX_MCU -> GND
- J2 pad 3: TX_MCU -> RX_MCU
- J2 pad 4: GND -> TX_MCU
- J7 pad 3: /MCU Schematic/IO27 -> Net-(J7-Pad3)
- Q2 pad 1: GPIO2 -> RESET_Cellular
- U1 pad 12: /MCU Schematic/IO27 -> EXTINT
- U10 pad 17: VCC_GPS -> +3V3
- U10 pad 2: VCC_GPS -> +3V3
- U10 pad 3: VCC_GPS -> +3V3
- U7 pad 10: VCC_GPS -> +3V3
- U7 pad 7: VCC_GPS -> +3V3
- U8 pad 18: RESET_Cellular -> Net-(Q2-Pad3)
- U8 pad 23: GPIO2 -> Net-(U8-Pad23)
Routing:
- net VSIM: track 47.5 -> 0.00 mm
- net RST: track 40.8 -> 0.00 mm
- net CLK: track 38.3 -> 0.00 mm
- net IO: track 34.1 -> 0.00 mm
- net VCC_GPS: track 3.94 -> 0.00 mm
- net SCL_Power: track 1.34 -> 0.00 mm
