File: KiCad/GPS Hardware/GPS Prototype 2 - ESP32/MCU.sch (KiCad schematic (older format))
At the start: 12 parts, among them J2 Conn_01x04_Male, J4 Conn_01x13_Male, U1 ESP32-WROOM-32D, U6 SN74AVC4T774PW

Commit message: Update to Uni computers
Finish esp32 connections.
Changed lines of the file:
@@
 	1    0    0    -1
 $EndComp
-Text GLabel 5600 5850 2    50   Input ~ 0
+Text GLabel 5600 5950 2    50   Input ~ 0
 RX
-Text GLabel 5600 5950 2    50   Output ~ 0
+Text GLabel 5600 5850 2    50   Output ~ 0
 TX
 Text GLabel 5600 6050 2    50   Output ~ 0

Commit message: Update
Parts:
- C10: symbol Device:C -> GPS-Hardware-rescue:C-Device
- J2: symbol Connector:Conn_01x04_Male -> GPS-Hardware-rescue:Conn_01x04_Male-Connector
- J4: symbol Connector:Conn_01x13_Male -> GPS-Hardware-rescue:Conn_01x13_Male-Connector
- R12, R13: symbol Device:R -> GPS-Hardware-rescue:R-Device
- U1: symbol RF_Module:ESP32-WROOM-32D -> GPS-Hardware-rescue:ESP32-WROOM-32D-RF_Module
Changed lines of the file:
@@
 $EndDescr
 $Comp
-L GPS-Hardware-rescue:+1V8-power #PWR0142
+L GPS-Hardware-rescue:+1V8-power-GPS-Hardware-rescue #PWR0142
 U 1 1 6149F6C9
 P 7150 2050
@@
 $EndComp
 $Comp
-L GPS-Hardware-rescue:+3V3-power #PWR0143
+L GPS-Hardware-rescue:+3V3-power-GPS-Hardware-rescue #PWR0143
 U 1 1 6149E56B
 P 7700 1950
@@
 $EndComp
 $Comp
-L GPS-Hardware-rescue:GND-power #PWR0144
+L GPS-Hardware-rescue:GND-power-GPS-Hardware-rescue #PWR0144
 U 1 1 6149DEBA
 P 6950 3450
@@
 $EndComp
 $Comp
-L GPS-Hardware-rescue:GND-power #PWR0145
+L GPS-Hardware-rescue:GND-power-GPS-Hardware-rescue #PWR0145
 U 1 1 6149C4AF
 P 5550 2250
@@
 $EndComp
 $Comp
-L GPS-Hardware-rescue:GND-power #PWR0146
+L GPS-Hardware-rescue:GND-power-GPS-Hardware-rescue #PWR0146
 U 1 1 6149BDCB
 P 5550 2350
@@
 $EndComp
 $Comp
-L GPS-Hardware-rescue:GND-power #PWR0147
+L GPS-Hardware-rescue:GND-power-GPS-Hardware-rescue #PWR0147
 U 1 1 6149B341
 P 5550 2550
@@
 	5550 2650 5200 2650
 $Comp
-L GPS-Hardware-rescue:+3V3-power #PWR0148
+L GPS-Hardware-rescue:+3V3-power-GPS-Hardware-rescue #PWR0148
 U 1 1 6149A2FD
 P 5200 2250
@@
 	7050 2050 6950 2050
 $Comp
-L GPS-Hardware-rescue:GND-power #PWR0110
+L GPS-Hardware-rescue:GND-power-GPS-Hardware-rescue #PWR0110
 U 1 1 612DF9B5
 P 7050 2350
@@
 $EndComp
 $Comp
-L GPS-Hardware-rescue:GND-power #PWR0149
+L GPS-Hardware-rescue:GND-power-GPS-Hardware-rescue #PWR0149
 U 1 1 612E15CE
 P 7600 2250
@@
 	5200 2450 5200 2650
 $Comp
-L RF_Module:ESP32-WROOM-32D U1
+L GPS-Hardware-rescue:ESP32-WROOM-32D-RF_Module U1
 U 1 1 6297038E
 P 5000 6050
@@
 INT_Power
 $Comp
-L Device:R R12
+L GPS-Hardware-rescue:R-Device R12
 U 1 1 62994EBE
 P 4100 4700
@@
 	4100 4850 4400 4850
 $Comp
-L GPS-Hardware-rescue:+3V3-power #PWR0103
+L GPS-Hardware-rescue:+3V3-power-GPS-Hardware-rescue #PWR0103
 U 1 1 62997A00
 P 4100 4550
@@
 $EndComp
 $Comp
-L Device:C C10
+L GPS-Hardware-rescue:C-Device C10
 U 1 1 62998D4D
 P 4100 5000
@@
 Connection ~ 4100 4850
 $Comp
-L GPS-Hardware-rescue:GND-power #PWR0127
+L GPS-Hardware-rescue:GND-power-GPS-Hardware-rescue #PWR0127
 U 1 1 6299A333
 P 4100 5150
@@
 	3800 4850 4100 4850
 $Comp
-L GPS-Hardware-rescue:GND-power #PWR0130
+L GPS-Hardware-rescue:GND-power-GPS-Hardware-rescue #PWR0130
 U 1 1 629A2C88
 P 3800 5250
@@
 $EndComp
 $Comp
-L Device:R R13
+L GPS-Hardware-rescue:R-Device R13
 U 1 1 629A3E5B
 P 5850 4700
@@
 $EndComp
 $Comp
-L GPS-Hardware-rescue:+3V3-power #PWR0131
+L GPS-Hardware-rescue:+3V3-power-GPS-Hardware-rescue #PWR0131
 U 1 1 629A44F3
 P 5850 4550
@@
 	5850 4850 5600 4850
 $Comp
-L GPS-Hardware-rescue:GND-power #PWR0132
+L GPS-Hardware-rescue:GND-power-GPS-Hardware-rescue #PWR0132
 U 1 1 629A8081
 P 6100 5250
@@
 RX_MCU
 $Comp
-L Connector:Conn_01x04_Male J2
+L GPS-Hardware-rescue:Conn_01x04_Male-Connector J2
 U 1 1 629C2CA6
 P 7800 4900
+AR Path="/629C2CA6" Ref="J2"  Part="1"
+AR Path="/613BCFBA/629C2CA6" Ref="J2"  Part="1"
 F 0 "J2" H 7908 5181 50  0000 C CNN
 F 1 "Conn_01x04_Male" H 7908 5090 50  0000 C CNN
@@
 RX_MCU
 $Comp
-L GPS-Hardware-rescue:+3V3-power #PWR0134
+L GPS-Hardware-rescue:+3V3-power-GPS-Hardware-rescue #PWR0134
 U 1 1 629C44E6
 P 8000 4800
@@
 $EndComp
 $Comp
-L GPS-Hardware-rescue:GND-power #PWR0135
+L GPS-Hardware-rescue:GND-power-GPS-Hardware-rescue #PWR0135
 U 1 1 629C538E
 P 8000 5100
@@
 SENS_VN
 $Comp
-L Connector:Conn_01x13_Male J4
+L GPS-Hardware-rescue:Conn_01x13_Male-Connector J4
 U 1 1 629CB424
 P 8750 5400
@@
 	1    0    0    -1
 $EndComp
+Text Label 8950 5000 0    50   ~ 0
+IO2
 Text Label 8950 4800 0    50   ~ 0
-IO2
+IO4
 Text Label 8950 4900 0    50   ~ 0
-IO4
-Text Label 8950 5000 0    50   ~ 0
 IO5
-Text Label 8950 5100 0    50   ~ 0
+Text Label 8950 5300 0    50   ~ 0
 IO12
 Text Label 8950 5200 0    50   ~ 0
 IO13
-Text Label 8950 5300 0    50   ~ 0
+Text Label 8950 5400 0    50   ~ 0
 IO14
-Text Label 8950 5400 0    50   ~ 0
+Text Label 8950 5100 0    50   ~ 0
 IO15
 Text Label 8950 5500 0    50   ~ 0
 IO27
+Text Label 8950 5700 0    50   ~ 0
+IO32
 Text Label 8950 5600 0    50   ~ 0
-IO32
-Text Label 8950 5700 0    50   ~ 0
 IO33
-Text Label 8950 5800 0    50   ~ 0
-IO35
-Text Label 8950 5900 0    50   ~ 0
-SENS_VP
-Text Label 8950 6000 0    50   ~ 0
-SENS_VN
 $Comp
 L GPS-Hardware-rescue:C-Device C11
@@
 $EndComp
 $Comp
-L GPS-Hardware-rescue:GND-power #PWR0136
+L GPS-Hardware-rescue:GND-power-GPS-Hardware-rescue #PWR0136
 U 1 1 629D3A1B
 P 5300 4350
@@
 $EndComp
 $Comp
-L GPS-Hardware-rescue:+3V3-power #PWR0137
+L GPS-Hardware-rescue:+3V3-power-GPS-Hardware-rescue #PWR0137
 U 1 1 629D4CF8
 P 5000 4350
@@
 Connection ~ 5000 4350
 $Comp
-L GPS-Hardware-rescue:GND-power #PWR0138
+L GPS-Hardware-rescue:GND-power-GPS-Hardware-rescue #PWR0138
 U 1 1 629D772D
 P 5000 7450
@@
 $EndComp
 $Comp
-L GPS-Hardware-rescue:+3V3-power #PWR0139
+L GPS-Hardware-rescue:+3V3-power-GPS-Hardware-rescue #PWR0139
 U 1 1 629DE412
 P 2800 4850
@@
 $EndComp
 $Comp
-L GPS-Hardware-rescue:GND-power #PWR0140
+L GPS-Hardware-rescue:GND-power-GPS-Hardware-rescue #PWR0140
 U 1 1 629DF21B
 P 2800 5250
@@
 $EndComp
 $Comp
-L GPS-Hardware-rescue:+3V3-power #PWR0141
+L GPS-Hardware-rescue:+3V3-power-GPS-Hardware-rescue #PWR0141
 U 1 1 629DFCA1
 P 7100 4850
@@
 $EndComp
 $Comp
-L GPS-Hardware-rescue:GND-power #PWR0164
+L GPS-Hardware-rescue:GND-power-GPS-Hardware-rescue #PWR0164
 U 1 1 629E0C0A
 P 7100 5250
@@
 	1    0    0    -1
 $EndComp
+Text Label 8950 5800 0    50   ~ 0
+IO35
+Text Label 8950 5900 0    50   ~ 0
+SENS_VN
+Text Label 8950 6000 0    50   ~ 0
+SENS_VP
 $EndSCHEMATC

Commit message: Update to Laptop
Still a lot more to go
Parts:
- removed J4: Conn_01x13_Male, Connector_PinHeader_2.54mm:PinHeader_1x13_P2.54mm_Vertical, symbol GPS-Hardware-rescue:Conn_01x13_Male-Connector
- added J4: Conn_01x05_Male, Connector_PinHeader_2.54mm:PinHeader_1x05_P2.54mm_Vertical_SMD_Pin1Left, symbol Connector:Conn_01x05_Male
- added J7: Conn_01x08_Male, Connector_PinHeader_2.54mm:PinHeader_1x08_P2.54mm_Vertical_SMD_Pin1Left, symbol Connector:Conn_01x08_Male
- J2: footprint Connector_PinHeader_2.54mm:PinHeader_1x04_P2.54mm_Vertical -> Connector_PinHeader_2.54mm:PinHeader_1x04_P2.54mm_Vertical_SMD_Pin1Left
Changed lines of the file:
@@
 Text GLabel 5600 6150 2    50   Input ~ 0
 CTS
-Text GLabel 5600 6450 2    50   Input ~ 0
+Text GLabel 5600 6550 2    50   Input ~ 0
 RESET_Cellular
-Text GLabel 5600 6550 2    50   Output ~ 0
+Text GLabel 5600 6450 2    50   Output ~ 0
 PWR_Cellular
 NoConn ~ 4400 6050
@@
 F 0 "J2" H 7908 5181 50  0000 C CNN
 F 1 "Conn_01x04_Male" H 7908 5090 50  0000 C CNN
-F 2 "Connector_PinHeader_2.54mm:PinHeader_1x04_P2.54mm_Vertical" H 7800 4900 50  0001 C CNN
+F 2 "Connector_PinHeader_2.54mm:PinHeader_1x04_P2.54mm_Vertical_SMD_Pin1Left" H 7800 4900 50  0001 C CNN
 F 3 "~" H 7800 4900 50  0001 C CNN
 	1    7800 4900
 	1    0    0    -1
 $EndComp
-Text GLabel 8000 4900 2    50   Input ~ 0
+Text GLabel 8000 5000 2    50   Input ~ 0
 TX_MCU
-Text GLabel 8000 5000 2    50   Output ~ 0
+Text GLabel 8000 4900 2    50   Output ~ 0
 RX_MCU
 $Comp
@@
 Text Label 4400 5150 2    50   ~ 0
 SENS_VN
-$Comp
-L GPS-Hardware-rescue:Conn_01x13_Male-Connector J4
-U 1 1 629CB424
-P 8750 5400
-F 0 "J4" H 8858 6181 50  0000 C CNN
-F 1 "Conn_01x13_Male" H 8858 6090 50  0000 C CNN
-F 2 "Connector_PinHeader_2.54mm:PinHeader_1x13_P2.54mm_Vertical" H 8750 5400 50  0001 C CNN
-F 3 "~" H 8750 5400 50  0001 C CNN
-	1    8750 5400
-	1    0    0    -1
-$EndComp
 Text Label 8950 5000 0    50   ~ 0
 IO2
@@
 Text Label 8950 4900 0    50   ~ 0
 IO5
-Text Label 8950 5300 0    50   ~ 0
+Text Label 9750 5300 0    50   ~ 0
 IO12
 Text Label 8950 5200 0    50   ~ 0
 IO13
-Text Label 8950 5400 0    50   ~ 0
+Text Label 9750 5400 0    50   ~ 0
 IO14
 Text Label 8950 5100 0    50   ~ 0
 IO15
-Text Label 8950 5500 0    50   ~ 0
+Text Label 9750 5500 0    50   ~ 0
 IO27
-Text Label 8950 5700 0    50   ~ 0
+Text Label 9750 5700 0    50   ~ 0
 IO32
-Text Label 8950 5600 0    50   ~ 0
+Text Label 9750 5600 0    50   ~ 0
 IO33
 $Comp
@@
 	1    0    0    -1
 $EndComp
-Text Label 8950 5800 0    50   ~ 0
+Text Label 9750 5800 0    50   ~ 0
 IO35
-Text Label 8950 5900 0    50   ~ 0
+Text Label 9750 5900 0    50   ~ 0
 SENS_VN
-Text Label 8950 6000 0    50   ~ 0
+Text Label 9750 6000 0    50   ~ 0
 SENS_VP
+$Comp
+L Connector:Conn_01x08_Male J7
+U 1 1 62BC985B
+P 9550 5600
+F 0 "J7" H 9658 6081 50  0000 C CNN
+F 1 "Conn_01x08_Male" H 9658 5990 50  0000 C CNN
+F 2 "Connector_PinHeader_2.54mm:PinHeader_1x08_P2.54mm_Vertical_SMD_Pin1Left" H 9550 5600 50  0001 C CNN
+F 3 "~" H 9550 5600 50  0001 C CNN
+	1    9550 5600
+	1    0    0    -1
+$EndComp
+$Comp
+L Connector:Conn_01x05_Male J4
+U 1 1 62BD8C7B
+P 8750 5000
+F 0 "J4" H 8858 5381 50  0000 C CNN
+F 1 "Conn_01x05_Male" H 8858 5290 50  0000 C CNN
+F 2 "Connector_PinHeader_2.54mm:PinHeader_1x05_P2.54mm_Vertical_SMD_Pin1Left" H 8750 5000 50  0001 C CNN
+F 3 "~" H 8750 5000 50  0001 C CNN
+	1    8750 5000
+	1    0    0    -1
+$EndComp
 $EndSCHEMATC

Commit message: Update
Parts:
- added R14: 100k, Resistor_SMD:R_1206_3216Metric_Pad1.30x1.75mm_HandSolder, symbol Device:R
Connections:
- net labels added: EXTINT
- net labels removed: IO27
- wire segments 13 -> 15
Other:
- moved on the sheet: C10, C11, C16, C17, J2, J4, J7, R12, R13, U1
